File: pcb/jerboa.sch (KiCad schematic (older format))
At the start: 1 part

Commit message: Some work on mcu circuitry
Parts:
- added C? (x5): 100nF, symbol agg-kicad:C
- added C?: 10uF, symbol agg-kicad:C
- added C?: 1uF, symbol agg-kicad:C
- added D?: LED_GREEN, agg:0603-LED, symbol agg-kicad:LED
- added P?: SWD_TC, agg:TC2030-NL, symbol agg-kicad:SWD_TC
- added R?: 120, agg:0402, symbol agg-kicad:R
Connections:
- net labels added: 3v3, GND, NRST, SWCLK, SWDIO
- wire segments 0 -> 50
- no-connect marks 0 -> 1
Other:
- note added: "16mA max current source"
- note added: "2496810 - 100nF caps 0402"
- note added: "No DFU required"

Commit message: Begin gps schematic, assuming dcdc converter used
Parts:
- removed C? (x4): 100nF, symbol agg-kicad:C
- added C? (x4): 100nF, agg:0402, symbol agg-kicad:C
- C?: footprint (none) -> agg:0402; Farnell Value -> 2496810
Other:
- note removed: "2496810 - 100nF caps 0402"
Changed lines of the file:
@@
 F 0 "C?" H 4450 1395 50  0000 C CNN
 F 1 "100nF" H 4450 1304 50  0000 C CNN
-F 2 "" H 4400 1200 50  0001 C CNN
+F 2 "agg:0402" H 4400 1200 50  0001 C CNN
 F 3 "" H 4400 1200 50  0001 C CNN
-F 4 "Value" H 4400 1200 60  0001 C CNN "Farnell"
+F 4 "2496810" H 4400 1200 60  0001 C CNN "Farnell"
 	1    4400 1200
-	1    0    0    -1
-$EndComp
-$Comp
-L agg-kicad:C C?
-U 1 1 5A3E3F1F
-P 4200 1400
-F 0 "C?" H 4250 1595 50  0000 C CNN
-F 1 "100nF" H 4250 1504 50  0000 C CNN
-F 2 "" H 4200 1400 50  0001 C CNN
-F 3 "" H 4200 1400 50  0001 C CNN
-F 4 "Value" H 4200 1400 60  0001 C CNN "Farnell"
-	1    4200 1400
-	1    0    0    -1
-$EndComp
-$Comp
-L agg-kicad:C C?
-U 1 1 5A3E3F54
-P 4400 1600
-F 0 "C?" H 4450 1795 50  0000 C CNN
-F 1 "100nF" H 4450 1704 50  0000 C CNN
-F 2 "" H 4400 1600 50  0001 C CNN
-F 3 "" H 4400 1600 50  0001 C CNN
-F 4 "Value" H 4400 1600 60  0001 C CNN "Farnell"
-	1    4400 1600
 	1    0    0    -1
 $EndComp
@@
 	1    0    0    -1
 $EndComp
-Wire Wire Line
-	4900 1950 4900 1900
-Wire Wire Line
-	4900 1900 5000 1900
 Text Notes 4800 2000 0    60   ~ 0
 No DFU required
@@
 	7100 2800 6700 2800
 NoConn ~ 6300 5000
-$Comp
-L agg-kicad:C C?
-U 1 1 5A3F62BE
-P 5000 4850
-F 0 "C?" H 5050 5045 50  0000 C CNN
-F 1 "100nF" H 5050 4954 50  0000 C CNN
-F 2 "" H 5000 4850 50  0001 C CNN
-F 3 "" H 5000 4850 50  0001 C CNN
-F 4 "Value" H 5000 4850 60  0001 C CNN "Farnell"
-	1    5000 4850
-	0    1    1    0
-$EndComp
 Wire Wire Line
 	5000 4850 5000 4800
@@
 	5000 5000 5000 4950
 Connection ~ 5400 5000
-$Comp
-L agg-kicad:C C?
-U 1 1 5A3F712E
-P 4700 1750
-F 0 "C?" H 4750 1945 50  0000 C CNN
-F 1 "100nF" H 4750 1854 50  0000 C CNN
-F 2 "" H 4700 1750 50  0001 C CNN
-F 3 "" H 4700 1750 50  0001 C CNN
-F 4 "Value" H 4700 1750 60  0001 C CNN "Farnell"
-	1    4700 1750
-	0    1    1    0
-$EndComp
 $Comp
 L agg-kicad:GND #PWR07
@@
 Wire Wire Line
 	4700 1700 5000 1700
-Text Notes 2300 1000 0    60   ~ 0
-2496810 - 100nF caps 0402
 $Comp
 L agg-kicad:LED D?
@@
 Text Notes 7050 2150 0    60   ~ 0
 16mA max current source
+Wire Wire Line
+	4900 1900 5000 1900
+Wire Wire Line
+	4900 1950 4900 1900
+$Comp
+L agg-kicad:C C?
+U 1 1 5A4085C3
+P 4200 1400
+F 0 "C?" H 4250 1595 50  0000 C CNN
+F 1 "100nF" H 4250 1504 50  0000 C CNN
+F 2 "agg:0402" H 4200 1400 50  0001 C CNN
+F 3 "" H 4200 1400 50  0001 C CNN
+F 4 "2496810" H 4200 1400 60  0001 C CNN "Farnell"
+	1    4200 1400
+	1    0    0    -1
+$EndComp
+$Comp
+L agg-kicad:C C?
+U 1 1 5A408606
+P 4400 1600
+F 0 "C?" H 4450 1795 50  0000 C CNN
+F 1 "100nF" H 4450 1704 50  0000 C CNN
+F 2 "agg:0402" H 4400 1600 50  0001 C CNN
+F 3 "" H 4400 1600 50  0001 C CNN
+F 4 "2496810" H 4400 1600 60  0001 C CNN "Farnell"
+	1    4400 1600
+	1    0    0    -1
+$EndComp
+$Comp
+L agg-kicad:C C?
+U 1 1 5A408643
+P 4700 1750
+F 0 "C?" H 4750 1945 50  0000 C CNN
+F 1 "100nF" H 4750 1854 50  0000 C CNN
+F 2 "agg:0402" H 4700 1750 50  0001 C CNN
+F 3 "" H 4700 1750 50  0001 C CNN
+F 4 "2496810" H 4700 1750 60  0001 C CNN "Farnell"
+	1    4700 1750
+	0    1    1    0
+$EndComp
+$Comp
+L agg-kicad:C C?
+U 1 1 5A4087DD
+P 5000 4950
+F 0 "C?" H 5050 5145 50  0000 C CNN
+F 1 "100nF" H 5050 5054 50  0000 C CNN
+F 2 "agg:0402" H 5000 4950 50  0001 C CNN
+F 3 "" H 5000 4950 50  0001 C CNN
+F 4 "2496810" H 5000 4950 60  0001 C CNN "Farnell"
+	1    5000 4950
+	0    -1   -1   0
+$EndComp
 $EndSCHEMATC

Commit message: Add some component values
Parts:
- C?: footprint (none) -> agg:0402; Farnell Value -> 1327658
Changed lines of the file:
@@
 F 0 "C?" H 4250 1995 50  0000 C CNN
 F 1 "1uF" H 4250 1904 50  0000 C CNN
-F 2 "" H 4200 1800 50  0001 C CNN
+F 2 "agg:0402" H 4200 1800 50  0001 C CNN
 F 3 "" H 4200 1800 50  0001 C CNN
-F 4 "Value" H 4200 1800 60  0001 C CNN "Farnell"
+F 4 "1327658" H 4200 1800 60  0001 C CNN "Farnell"
 	1    4200 1800
 	1    0    0    -1

Commit message: Added radio circuit
Connections:
- wire segments 50 -> 36
Changed lines of the file:
@@
-EESchema Schematic File Version 4
+EESchema Schematic File Version 2
+LIBS:agg-kicad
 LIBS:jerboa-cache
-EELAYER 26 0
+EELAYER 25 0
 EELAYER END
 $Descr A4 11693 8268
@@
 	4500 1600 4550 1600
 Wire Wire Line
-	4400 1600 4150 1600
+	4150 1600 4400 1600
 Wire Wire Line
 	4200 1400 4150 1400
 Wire Wire Line
-	4150 1400 4150 1600
+	4150 1000 4150 1850
 Connection ~ 4150 1600
 Wire Wire Line
 	4400 1200 4150 1200
-Wire Wire Line
-	4150 1200 4150 1400
 Connection ~ 4150 1400
 $Comp
@@
 Wire Wire Line
 	4200 1000 4150 1000
-Wire Wire Line
-	4150 1000 4150 1200
 Connection ~ 4150 1200
 $Comp
@@
 $EndComp
 Wire Wire Line
-	4150 1850 4150 1800
-Wire Wire Line
 	4200 1800 4150 1800
 Connection ~ 4150 1800
 Wire Wire Line
-	4150 1800 4150 1600
-Wire Wire Line
-	4300 1800 4550 1800
-Wire Wire Line
-	4550 1800 4550 1600
-Wire Wire Line
-	4550 1500 4550 1600
+	4550 1800 4300 1800
+Wire Wire Line
+	4550 900  4550 1800
 Connection ~ 4550 1600
-Wire Wire Line
-	4550 1300 4550 1200
 Wire Wire Line
 	4550 1000 4300 1000
@@
 	4500 1200 4550 1200
 Connection ~ 4550 1200
-Wire Wire Line
-	4550 1200 4550 1000
 Text Label 4650 1700 0    60   ~ 0
 NRST
@@
 	4550 1300 5000 1300
 Wire Wire Line
-	4300 1400 4550 1400
+	4300 1400 5000 1400
 Wire Wire Line
 	4550 1500 5000 1500
@@
 	1    0    0    -1
 $EndComp
-Wire Wire Line
-	4550 1000 4550 900
 Connection ~ 4550 1000
-Wire Wire Line
-	4550 1300 4550 1400
 Connection ~ 4550 1300
 Connection ~ 4550 1400
-Wire Wire Line
-	4550 1400 5000 1400
-Wire Wire Line
-	4550 1400 4550 1500
 Connection ~ 4550 1500
 $Comp
@@
 $EndComp
 Wire Wire Line
-	5500 4800 5400 4800
+	5000 4800 5500 4800
 Wire Wire Line
 	5400 4800 5400 4750
@@
 	5400 5050 5400 5000
 Wire Wire Line
-	5400 5000 5500 5000
+	5000 5000 5500 5000
 Text Label 6700 4800 2    60   ~ 0
 SWDIO
@@
 Wire Wire Line
 	5000 4850 5000 4800
-Wire Wire Line
-	5000 4800 5400 4800
 Connection ~ 5400 4800
-Wire Wire Line
-	5400 5000 5000 5000
 Wire Wire Line
 	5000 5000 5000 4950
@@
 Connection ~ 4700 1700
 Wire Wire Line
-	4700 1700 4650 1700
-Wire Wire Line
-	4700 1700 5000 1700
+	4650 1700 5000 1700
 $Comp
 L agg-kicad:LED D?

Commit message: Forgot to save
Connections:
- net labels added: MCU_MISO_TO_RADIO, MCU_MOSI_TO_RADIO, MCU_NSS_TO_RADIO, MCU_SCK_TO_RADIO
- wire segments 36 -> 40
Changed lines of the file:
@@
 	1    0    0    -1
 $EndComp
-Wire Wire Line
-	5000 2400 4900 2400
-Wire Wire Line
-	4900 2400 4900 2500
 $Comp
 L agg-kicad:C C?
@@
 	1    0    0    -1
 $EndComp
-Wire Wire Line
-	4500 1600 4550 1600
-Wire Wire Line
-	4150 1600 4400 1600
-Wire Wire Line
-	4200 1400 4150 1400
-Wire Wire Line
-	4150 1000 4150 1850
-Connection ~ 4150 1600
-Wire Wire Line
-	4400 1200 4150 1200
-Connection ~ 4150 1400
 $Comp
 L agg-kicad:C C?
@@
 	1    0    0    -1
 $EndComp
-Wire Wire Line
-	4200 1000 4150 1000
-Connection ~ 4150 1200
 $Comp
 L agg-kicad:C C?
@@
 	1    0    0    -1
 $EndComp
-Wire Wire Line
-	4200 1800 4150 1800
-Connection ~ 4150 1800
-Wire Wire Line
-	4550 1800 4300 1800
-Wire Wire Line
-	4550 900  4550 1800
-Connection ~ 4550 1600
-Wire Wire Line
-	4550 1000 4300 1000
-Wire Wire Line
-	4500 1200 4550 1200
-Connection ~ 4550 1200
 Text Label 4650 1700 0    60   ~ 0
 NRST
-Wire Wire Line
-	4550 1300 5000 1300
-Wire Wire Line
-	4300 1400 5000 1400
-Wire Wire Line
-	4550 1500 5000 1500
 Text Label 5200 4900 0    60   ~ 0
 NRST
@@
 	1    0    0    -1
 $EndComp
-Connection ~ 4550 1000
-Connection ~ 4550 1300
-Connection ~ 4550 1400
-Connection ~ 4550 1500
 $Comp
 L agg-kicad:GND #PWR04
@@
 	1    0    0    -1
 $EndComp
-Wire Wire Line
-	5200 4900 5500 4900
 $Comp
 L agg-kicad:GND #PWR05
@@
 	1    0    0    -1
 $EndComp
-Wire Wire Line
-	5000 4800 5500 4800
-Wire Wire Line
-	5400 4800 5400 4750
-Wire Wire Line
-	5400 5050 5400 5000
-Wire Wire Line
-	5000 5000 5500 5000
 Text Label 6700 4800 2    60   ~ 0
 SWDIO
 Text Label 6700 4900 2    60   ~ 0
 SWCLK
-Wire Wire Line
-	6700 4800 6300 4800
-Wire Wire Line
-	6300 4900 6700 4900
 Text Label 7100 2700 2    60   ~ 0
 SWDIO
 Text Label 7100 2800 2    60   ~ 0
 SWCLK
-Wire Wire Line
-	6700 2700 7100 2700
-Wire Wire Line
-	7100 2800 6700 2800
 NoConn ~ 6300 5000
-Wire Wire Line
-	5000 4850 5000 4800
-Connection ~ 5400 4800
-Wire Wire Line
-	5000 5000 5000 4950
-Connection ~ 5400 5000
 $Comp
 L agg-kicad:GND #PWR07
@@
 	1    0    0    -1
 $EndComp
-Wire Wire Line
-	4700 1950 4700 1850
-Wire Wire Line
-	4700 1750 4700 1700
-Connection ~ 4700 1700
-Wire Wire Line
-	4650 1700 5000 1700
 $Comp
 L agg-kicad:LED D?
@@
 	1    0    0    -1
 $EndComp
-Wire Wire Line
-	6700 2200 6900 2200
 $Comp
 L agg-kicad:GND #PWR?
@@
 	1    0    0    -1
 $EndComp
-Wire Wire Line
-	7150 2400 7150 2350
-Wire Wire Line
-	7150 2250 7150 2200
-Wire Wire Line
-	7150 2200 7000 2200
 Text Notes 7050 2150 0    60   ~ 0
 16mA max current source
-Wire Wire Line
-	4900 1900 5000 1900
-Wire Wire Line
-	4900 1950 4900 1900
 $Comp
 L agg-kicad:C C?
@@
 	0    -1   -1   0
 $EndComp
+Text Label 7050 1900 0    60   ~ 0
+MCU_MISO_TO_RADIO
+Text Label 7050 1800 0    60   ~ 0
+MCU_SCK_TO_RADIO
+Text Label 7050 1700 0    60   ~ 0
+MCU_NSS_TO_RADIO
+Text Label 7050 2000 0    60   ~ 0
+MCU_MOSI_TO_RADIO
+Wire Wire Line
+	5000 2400 4900 2400
+Wire Wire Line
+	4900 2400 4900 2500
+Wire Wire Line
+	4500 1600 4550 1600
+Wire Wire Line
+	4150 1600 4400 1600
+Wire Wire Line
+	4200 1400 4150 1400
+Wire Wire Line
+	4150 1000 4150 1850
+Connection ~ 4150 1600
+Wire Wire Line
+	4400 1200 4150 1200
+Connection ~ 4150 1400
+Wire Wire Line
+	4200 1000 4150 1000
+Connection ~ 4150 1200
+Wire Wire Line
+	4200 1800 4150 1800
+Connection ~ 4150 1800
+Wire Wire Line
+	4550 1800 4300 1800
+Wire Wire Line
+	4550 900  4550 1800
+Connection ~ 4550 1600
+Wire Wire Line
+	4550 1000 4300 1000
+Wire Wire Line
+	4500 1200 4550 1200
+Connection ~ 4550 1200
+Wire Wire Line
+	4550 1300 5000 1300
+Wire Wire Line
+	4300 1400 5000 1400
+Wire Wire Line
+	4550 1500 5000 1500
+Connection ~ 4550 1000
+Connection ~ 4550 1300
+Connection ~ 4550 1400
+Connection ~ 4550 1500
+Wire Wire Line
+	5200 4900 5500 4900
+Wire Wire Line
+	5000 4800 5500 4800
+Wire Wire Line
+	5400 4800 5400 4750
+Wire Wire Line
+	5400 5050 5400 5000
+Wire Wire Line
+	5000 5000 5500 5000
+Wire Wire Line
+	6700 4800 6300 4800
+Wire Wire Line
+	6300 4900 6700 4900
+Wire Wire Line
+	6700 2700 7100 2700
+Wire Wire Line
+	7100 2800 6700 2800
+Wire Wire Line
+	5000 4850 5000 4800
+Connection ~ 5400 4800
+Wire Wire Line
+	5000 5000 5000 4950
+Connection ~ 5400 5000
+Wire Wire Line
+	4700 1950 4700 1850
+Wire Wire Line
+	4700 1750 4700 1700
+Connection ~ 4700 1700
+Wire Wire Line
+	4650 1700 5000 1700
+Wire Wire Line
+	6700 2200 6900 2200
+Wire Wire Line
+	7150 2400 7150 2350
+Wire Wire Line
+	7150 2250 7150 2200
+Wire Wire Line
+	7150 2200 7000 2200
+Wire Wire Line
+	4900 1900 5000 1900
+Wire Wire Line
+	4900 1950 4900 1900
+Wire Wire Line
+	7050 2000 6700 2000
+Wire Wire Line
+	6700 1900 7050 1900
+Wire Wire Line
+	7050 1800 6700 1800
+Wire Wire Line
+	6700 1700 7050 1700
 $EndSCHEMATC

Commit message: Schematic almost done.
Parts:
- gave numbers to parts that had none: 11
Connections:
- net labels added: RX_GPS_from_MCU, TX_GPS_from_MCU
- wire segments 40 -> 48
- no-connect marks 1 -> 19
Other:
- moved on the sheet: C101, C102, C103, C104, C105

Commit message: Added shutdown and interrupt control for Radio
Connections:
- net labels added: MCU_SHUTDOWN_TO_RADIO, MCU_nIRQ_TO_RADIO
- wire segments 48 -> 52
- no-connect marks 19 -> 17
Changed lines of the file:
@@
 NoConn ~ 6700 1300
 NoConn ~ 6700 1400
-NoConn ~ 6700 1500
-NoConn ~ 6700 1600
 NoConn ~ 6700 2300
 NoConn ~ 6700 2400
@@
 NoConn ~ 6700 3300
 NoConn ~ 6700 3500
-NoConn ~ 6700 3600
-NoConn ~ 6700 3700
 NoConn ~ 6700 4100
 Wire Wire Line
@@
 Wire Wire Line
 	1400 6150 1600 6150
+Wire Wire Line
+	1400 5550 1600 5550
+Wire Wire Line
+	1400 6300 1600 6300
+NoConn ~ 6700 3600
+NoConn ~ 6700 3700
+Text Label 7050 1500 0    60   ~ 0
+MCU_SHUTDOWN_TO_RADIO
+Text Label 7050 1600 0    60   ~ 0
+MCU_nIRQ_TO_RADIO
+Wire Wire Line
+	6700 1600 7050 1600
+Wire Wire Line
+	6700 1500 7050 1500
+Text Label 1600 5550 0    60   ~ 0
+MCU_SHUTDOWN_TO_RADIO
+Text Label 1600 6300 0    60   ~ 0
+MCU_nIRQ_TO_RADIO
 $EndSCHEMATC

Commit message: Attempt to fix symbol library problems from old kicad version
Connections:
- wire segments 52 -> 66
Changed lines of the file:
@@
-EESchema Schematic File Version 2
-LIBS:agg-kicad
+EESchema Schematic File Version 4
 LIBS:jerboa-cache
-EELAYER 25 0
+EELAYER 26 0
 EELAYER END
 $Descr A4 11693 8268
@@
 F 2 "" H 4900 2500 60  0001 C CNN
 F 3 "" H 4900 2500 60  0001 C CNN
+F 4 "Value" H 4900 2500 50  0001 C CNN "Farnell"
 	1    4900 2500
 	1    0    0    -1
@@
 	4050 1400 4000 1400
 Wire Wire Line
-	4000 1000 4000 1850
+	4000 1000 4000 1200
 Connection ~ 4000 1600
 Wire Wire Line
@@
 	4400 1800 4150 1800
 Wire Wire Line
-	4400 900  4400 1800
+	4400 900  4400 1000
 Connection ~ 4400 1600
 Wire Wire Line
@@
 	4400 1300 5000 1300
 Wire Wire Line
-	4150 1400 5000 1400
+	4150 1400 4400 1400
 Wire Wire Line
 	4400 1500 5000 1500
@@
 NRST
 Wire Wire Line
-	4650 1700 5000 1700
+	4650 1700 4700 1700
 Text Label 6850 3800 0    60   ~ 0
 TX_GPS_from_MCU
 Text Label 6850 3900 0    60   ~ 0
 RX_GPS_from_MCU
-Wire Wire Line
-	6700 3800 6850 3800
 Wire Wire Line
 	6700 3900 6850 3900
@@
 NoConn ~ 6700 4100
 Wire Wire Line
-	5000 5000 5500 5000
-Wire Wire Line
-	5000 4800 5500 4800
+	5000 5000 5400 5000
+Wire Wire Line
+	5000 4800 5400 4800
 Text Label 1600 6150 0    60   ~ 0
 MCU_NSS_TO_RADIO
@@
 Text Label 1600 6300 0    60   ~ 0
 MCU_nIRQ_TO_RADIO
+Wire Wire Line
+	4000 1600 4000 1800
+Wire Wire Line
+	4000 1400 4000 1600
+Wire Wire Line
+	4000 1200 4000 1400
+Wire Wire Line
+	4000 1800 4000 1850
+Wire Wire Line
+	4400 1600 4400 1800
+Wire Wire Line
+	4400 1200 4400 1300
+Wire Wire Line
+	4400 1000 4400 1200
+Wire Wire Line
+	4400 1300 4400 1400
+Wire Wire Line
+	4400 1400 5000 1400
+Wire Wire Line
+	4400 1400 4400 1500
+Wire Wire Line
+	4400 1500 4400 1600
+Wire Wire Line
+	5400 4800 5500 4800
+Wire Wire Line
+	5400 5000 5500 5000
+Wire Wire Line
+	4700 1700 5000 1700
+Wire Wire Line
+	6850 3800 6700 3800
 $EndSCHEMATC
