File: pcb/jerboa.sch (KiCad schematic (older format))
At the start: 27 parts, among them IC1 SL18860DC, J1 CONN_01x02, J2 CONN_01x03, P1 SWD_TC, U1 STM32L051K8U6, Y1 TCXO

Commit message: WIP: begin board layout
Parts:
- added X3: MOUNT, agg:M2.5_MOUNT, symbol agg-kicad:PART
Changed lines of the file:
@@
 $EndComp
 Connection ~ 3450 4250
+$Comp
+L agg-kicad:PART X3
+U 1 1 5B50EEE8
+P 7050 5550
+F 0 "X3" H 7578 5646 50  0000 L CNN
+F 1 "MOUNT" H 7578 5555 50  0000 L CNN
+F 2 "agg:M2.5_MOUNT" H 7050 5550 50  0001 C CNN
+F 3 "" H 7050 5550 50  0001 C CNN
+	1    7050 5550
+	1    0    0    -1
+$EndComp
 $EndSCHEMATC

Commit message: Redo si4460 matching for 169MHz
Parts:
- renumbered X3 to X1
Changed lines of the file:
@@
 EESchema Schematic File Version 4
-LIBS:jerboa-cache
 EELAYER 26 0
 EELAYER END
@@
 $EndSheet
 $Comp
-L agg-kicad:GND #PWR016
+L agg-kicad:GND #PWR0101
 U 1 1 5A3E3DF5
 P 6450 2350
-F 0 "#PWR016" H 6320 2390 50  0001 L CNN
+F 0 "#PWR0101" H 6320 2390 50  0001 L CNN
 F 1 "GND" H 6450 2250 50  0000 C CNN
 F 2 "" H 6450 2350 60  0001 C CNN
@@
 $EndComp
 $Comp
-L agg-kicad:GND #PWR012
+L agg-kicad:GND #PWR0102
 U 1 1 5A3E4029
 P 5550 1700
-F 0 "#PWR012" H 5420 1740 50  0001 L CNN
+F 0 "#PWR0102" H 5420 1740 50  0001 L CNN
 F 1 "GND" H 5550 1787 50  0000 C CNN
 F 2 "" H 5550 1700 60  0001 C CNN
@@
 NRST
 $Comp
-L agg-kicad:3v3 #PWR013
+L agg-kicad:3v3 #PWR0103
 U 1 1 5A3EFF91
 P 5950 750
-F 0 "#PWR013" H 5950 860 50  0001 L CNN
+F 0 "#PWR0103" H 5950 860 50  0001 L CNN
 F 1 "3v3" H 5950 874 50  0000 C CNN
 F 2 "" H 5950 750 60  0001 C CNN
@@
 $EndComp
 $Comp
-L agg-kicad:GND #PWR015
+L agg-kicad:GND #PWR0104
 U 1 1 5A3F2FB2
 P 6450 1800
-F 0 "#PWR015" H 6320 1840 50  0001 L CNN
+F 0 "#PWR0104" H 6320 1840 50  0001 L CNN
 F 1 "GND" H 6500 1700 50  0000 C CNN
 F 2 "" H 6450 1800 60  0001 C CNN
@@
 $EndComp
 $Comp
-L agg-kicad:GND #PWR018
+L agg-kicad:GND #PWR0105
 U 1 1 5A3F3ABE
 P 6800 4650
-F 0 "#PWR018" H 6670 4690 50  0001 L CNN
+F 0 "#PWR0105" H 6670 4690 50  0001 L CNN
 F 1 "GND" H 6800 4737 50  0000 C CNN
 F 2 "" H 6800 4650 60  0001 C CNN
@@
 $EndComp
 $Comp
-L agg-kicad:3v3 #PWR017
+L agg-kicad:3v3 #PWR0106
 U 1 1 5A3F3B9B
 P 6800 4350
-F 0 "#PWR017" H 6800 4460 50  0001 L CNN
+F 0 "#PWR0106" H 6800 4460 50  0001 L CNN
 F 1 "3v3" H 6800 4474 50  0000 C CNN
 F 2 "" H 6800 4350 60  0001 C CNN
@@
 NoConn ~ 7700 4600
 $Comp
-L agg-kicad:GND #PWR014
+L agg-kicad:GND #PWR0107
 U 1 1 5A3F7FF1
 P 6250 1800
-F 0 "#PWR014" H 6120 1840 50  0001 L CNN
+F 0 "#PWR0107" H 6120 1840 50  0001 L CNN
 F 1 "GND" H 6200 1700 50  0000 C CNN
 F 2 "" H 6250 1800 60  0001 C CNN
@@
 $EndComp
 $Comp
-L agg-kicad:GND #PWR019
+L agg-kicad:GND #PWR0108
 U 1 1 5A3EA11D
 P 8700 4150
-F 0 "#PWR019" H 8570 4190 50  0001 L CNN
+F 0 "#PWR0108" H 8570 4190 50  0001 L CNN
 F 1 "GND" H 8800 4100 50  0000 C CNN
 F 2 "" H 8700 4150 60  0001 C CNN
@@
 $EndComp
 $Comp
-L agg-kicad:GND #PWR021
+L agg-kicad:GND #PWR0109
 U 1 1 5A6E5C1D
 P 9650 1550
-F 0 "#PWR021" H 9520 1590 50  0001 L CNN
+F 0 "#PWR0109" H 9520 1590 50  0001 L CNN
 F 1 "GND" H 9650 1450 50  0000 C CNN
 F 2 "" H 9650 1550 50  0001 C CNN
@@
 $EndComp
 $Comp
-L agg-kicad:3v3 #PWR01
+L agg-kicad:3v3 #PWR0110
 U 1 1 5A8619B3
 P 2100 4500
-F 0 "#PWR01" H 2100 4610 50  0001 L CNN
+F 0 "#PWR0110" H 2100 4610 50  0001 L CNN
 F 1 "3v3" H 2100 4624 50  0000 C CNN
 F 2 "" H 2100 4500 60  0001 C CNN
@@
 $EndComp
 $Comp
-L agg-kicad:GND #PWR02
+L agg-kicad:GND #PWR0111
 U 1 1 5A861D30
 P 2100 4900
-F 0 "#PWR02" H 1970 4940 50  0001 L CNN
+F 0 "#PWR0111" H 1970 4940 50  0001 L CNN
 F 1 "GND" H 2100 4987 50  0000 C CNN
 F 2 "" H 2100 4900 60  0001 C CNN
@@
 	4050 5050 4000 5050
 $Comp
-L agg-kicad:GND #PWR010
+L agg-kicad:GND #PWR0112
 U 1 1 5A87D090
 P 4050 4500
-F 0 "#PWR010" H 3920 4540 50  0001 L CNN
+F 0 "#PWR0112" H 3920 4540 50  0001 L CNN
 F 1 "GND" H 4050 4587 50  0000 C CNN
 F 2 "" H 4050 4500 60  0001 C CNN
@@
 	4050 4450 4050 4500
 $Comp
-L agg-kicad:3v3 #PWR07
+L agg-kicad:3v3 #PWR0113
 U 1 1 5A87FD1C
 P 3850 4950
-F 0 "#PWR07" H 3850 5060 50  0001 L CNN
+F 0 "#PWR0113" H 3850 5060 50  0001 L CNN
 F 1 "3v3" H 3850 5074 50  0000 C CNN
 F 2 "" H 3850 4950 60  0001 C CNN
@@
 Connection ~ 5350 4450
 $Comp
-L agg-kicad:GND #PWR011
+L agg-kicad:GND #PWR0114
 U 1 1 5A8967D4
 P 5350 4650
-F 0 "#PWR011" H 5220 4690 50  0001 L CNN
+F 0 "#PWR0114" H 5220 4690 50  0001 L CNN
 F 1 "GND" H 5350 4550 50  0000 C CNN
 F 2 "" H 5350 4650 60  0001 C CNN
@@
 	3850 4950 4000 4950
 $Comp
-L agg-kicad:GND #PWR09
+L agg-kicad:GND #PWR0115
 U 1 1 5A8A8E50
 P 4000 5200
-F 0 "#PWR09" H 3870 5240 50  0001 L CNN
+F 0 "#PWR0115" H 3870 5240 50  0001 L CNN
 F 1 "GND" H 4000 5100 50  0000 C CNN
 F 2 "" H 4000 5200 60  0001 C CNN
@@
 $EndComp
 $Comp
-L agg-kicad:3v3 #PWR08
+L agg-kicad:3v3 #PWR0116
 U 1 1 5A8C5CC2
 P 3950 4050
-F 0 "#PWR08" H 3950 4160 50  0001 L CNN
+F 0 "#PWR0116" H 3950 4160 50  0001 L CNN
 F 1 "3v3" H 3950 4174 50  0000 C CNN
 F 2 "" H 3950 4050 60  0001 C CNN
@@
 $EndComp
 $Comp
-L agg-kicad:GND #PWR06
+L agg-kicad:GND #PWR0117
 U 1 1 5A89E908
 P 3550 1900
-F 0 "#PWR06" H 3420 1940 50  0001 L CNN
+F 0 "#PWR0117" H 3420 1940 50  0001 L CNN
 F 1 "GND" H 3550 1800 50  0000 C CNN
 F 2 "" H 3550 1900 60  0001 C CNN
@@
 $EndComp
 $Comp
-L agg-kicad:3v3 #PWR05
+L agg-kicad:3v3 #PWR0118
 U 1 1 5A89EBB4
 P 3550 1700
-F 0 "#PWR05" H 3550 1810 50  0001 L CNN
+F 0 "#PWR0118" H 3550 1810 50  0001 L CNN
 F 1 "3v3" H 3550 1824 50  0000 C CNN
 F 2 "" H 3550 1700 60  0001 C CNN
@@
 	3050 4650 3050 4700
 $Comp
-L agg-kicad:3v3 #PWR03
+L agg-kicad:3v3 #PWR0119
 U 1 1 5A956F5B
 P 3050 4450
-F 0 "#PWR03" H 3050 4560 50  0001 L CNN
+F 0 "#PWR0119" H 3050 4560 50  0001 L CNN
 F 1 "3v3" H 3050 4574 50  0000 C CNN
 F 2 "" H 3050 4450 60  0001 C CNN
@@
 $EndComp
 $Comp
-L agg-kicad:GND #PWR04
+L agg-kicad:GND #PWR0120
 U 1 1 5A956FCA
 P 3050 4850
-F 0 "#PWR04" H 2920 4890 50  0001 L CNN
+F 0 "#PWR0120" H 2920 4890 50  0001 L CNN
 F 1 "GND" H 3050 4750 50  0000 C CNN
 F 2 "" H 3050 4850 60  0001 C CNN
@@
 $EndComp
 $Comp
-L agg-kicad:3v3 #PWR020
+L agg-kicad:3v3 #PWR0121
 U 1 1 5B467DD6
 P 9350 3400
-F 0 "#PWR020" H 9350 3510 50  0001 L CNN
+F 0 "#PWR0121" H 9350 3510 50  0001 L CNN
 F 1 "3v3" H 9350 3524 50  0000 C CNN
 F 2 "" H 9350 3400 60  0001 C CNN
@@
 Connection ~ 3450 4250
 $Comp
-L agg-kicad:PART X3
+L agg-kicad:PART X1
 U 1 1 5B50EEE8
 P 7050 5550
-F 0 "X3" H 7578 5646 50  0000 L CNN
+F 0 "X1" H 7578 5646 50  0000 L CNN
 F 1 "MOUNT" H 7578 5555 50  0000 L CNN
 F 2 "agg:M2.5_MOUNT" H 7050 5550 50  0001 C CNN

Commit message: WIP: work on pcb, use guitar wire ground plane antenna and remove rx matching on si4460 as there is nothing to receive
Parts:
- R3: footprint agg:0603 -> agg:0603-L
Changed lines of the file:
@@
 EESchema Schematic File Version 4
+LIBS:jerboa-cache
 EELAYER 26 0
 EELAYER END
@@
 F 0 "R3" V 3954 4141 50  0000 L CNN
 F 1 "50" V 4045 4141 50  0000 L CNN
-F 2 "agg:0603" H 3950 4100 50  0001 C CNN
+F 2 "agg:0603-L" H 3950 4100 50  0001 C CNN
 F 3 "" H 3950 4100 50  0001 C CNN
 F 4 "2112878" H 3950 4100 60  0001 C CNN "Farnell"

Commit message: WIP: add clock circuitry to pcb
Connections:
- wire segments 148 -> 146
Other:
- moved on the sheet: R4, R5
Changed lines of the file:
@@
 NoConn ~ 8250 2350
 NoConn ~ 8250 2450
-NoConn ~ 8250 2750
 NoConn ~ 8250 3150
 NoConn ~ 8250 3350
@@
 Connection ~ 2100 4800
 NoConn ~ 4050 4750
-Wire Wire Line
-	4000 5150 4050 5150
-Wire Wire Line
-	4050 5050 4000 5050
 $Comp
 L agg-kicad:GND #PWR0112
@@
 Wire Wire Line
 	3950 4200 3950 4250
-Text Label 5150 4350 0    60   ~ 0
+Text Label 5100 4550 0    60   ~ 0
 MCU_CLK
-Wire Wire Line
-	5050 4350 5150 4350
-Text Label 5450 4450 0    60   ~ 0
+Text Label 5700 4350 0    60   ~ 0
 SI4460_CLK
-Wire Wire Line
-	5150 4450 5050 4450
 Text Label 6100 1950 2    60   ~ 0
 MCU_CLK
@@
 L agg-kicad:R R4
 U 1 1 5A88FCFB
-P 5150 4450
-F 0 "R4" H 5200 4628 50  0000 C CNN
-F 1 "10k" H 5200 4537 50  0000 C CNN
-F 2 "agg:0402" H 5150 4450 50  0001 C CNN
-F 3 "" H 5150 4450 50  0001 C CNN
-F 4 "2331444" H 5150 4450 60  0001 C CNN "Farnell"
-	1    5150 4450
+P 5400 4350
+F 0 "R4" H 5450 4528 50  0000 C CNN
+F 1 "10k" H 5450 4437 50  0000 C CNN
+F 2 "agg:0402" H 5400 4350 50  0001 C CNN
+F 3 "" H 5400 4350 50  0001 C CNN
+F 4 "2331444" H 5400 4350 60  0001 C CNN "Farnell"
+	1    5400 4350
 	1    0    0    -1
 $EndComp
@@
 L agg-kicad:R R5
 U 1 1 5A88FE03
-P 5350 4500
-F 0 "R5" V 5354 4541 50  0000 L CNN
-F 1 "10k" V 5445 4541 50  0000 L CNN
-F 2 "agg:0402" H 5350 4500 50  0001 C CNN
-F 3 "" H 5350 4500 50  0001 C CNN
-F 4 "2331444" H 5350 4500 60  0001 C CNN "Farnell"
-	1    5350 4500
+P 5600 4400
+F 0 "R5" V 5604 4441 50  0000 L CNN
+F 1 "10k" V 5695 4441 50  0000 L CNN
+F 2 "agg:0402" H 5600 4400 50  0001 C CNN
+F 3 "" H 5600 4400 50  0001 C CNN
+F 4 "2331444" H 5600 4400 60  0001 C CNN "Farnell"
+	1    5600 4400
 	0    1    1    0
 $EndComp
 Wire Wire Line
-	5350 4500 5350 4450
-Wire Wire Line
-	5250 4450 5350 4450
-Connection ~ 5350 4450
+	5600 4400 5600 4350
+Wire Wire Line
+	5500 4350 5600 4350
+Connection ~ 5600 4350
 $Comp
 L agg-kicad:GND #PWR0114
 U 1 1 5A8967D4
-P 5350 4650
-F 0 "#PWR0114" H 5220 4690 50  0001 L CNN
-F 1 "GND" H 5350 4550 50  0000 C CNN
-F 2 "" H 5350 4650 60  0001 C CNN
-F 3 "" H 5350 4650 60  0001 C CNN
-	1    5350 4650
-	1    0    0    -1
-$EndComp
-Wire Wire Line
-	5350 4650 5350 4600
+P 5600 4550
+F 0 "#PWR0114" H 5470 4590 50  0001 L CNN
+F 1 "GND" H 5600 4450 50  0000 C CNN
+F 2 "" H 5600 4550 60  0001 C CNN
+F 3 "" H 5600 4550 60  0001 C CNN
+	1    5600 4550
+	1    0    0    -1
+$EndComp
+Wire Wire Line
+	5600 4550 5600 4500
 Wire Wire Line
 	3950 4350 4050 4350
-Wire Wire Line
-	3850 4950 4000 4950
 $Comp
 L agg-kicad:GND #PWR0115
 U 1 1 5A8A8E50
-P 4000 5200
-F 0 "#PWR0115" H 3870 5240 50  0001 L CNN
-F 1 "GND" H 4000 5100 50  0000 C CNN
-F 2 "" H 4000 5200 60  0001 C CNN
-F 3 "" H 4000 5200 60  0001 C CNN
-	1    4000 5200
-	1    0    0    -1
-$EndComp
-Wire Wire Line
-	4000 5200 4000 5150
-NoConn ~ 5050 4550
-Wire Wire Line
-	4000 5050 4000 4950
-Connection ~ 4000 4950
+P 3950 5050
+F 0 "#PWR0115" H 3820 5090 50  0001 L CNN
+F 1 "GND" H 3950 4950 50  0000 C CNN
+F 2 "" H 3950 5050 60  0001 C CNN
+F 3 "" H 3950 5050 60  0001 C CNN
+	1    3950 5050
+	0    1    1    0
+$EndComp
 $Comp
 L agg-kicad:C C4
@@
 	2100 4800 2100 4900
 Wire Wire Line
-	5350 4450 5450 4450
-Wire Wire Line
-	4000 4950 4050 4950
+	5600 4350 5700 4350
 Wire Wire Line
 	3750 4450 3450 4450
@@
 Wire Wire Line
 	8600 1150 8250 1150
-Text Label 8600 1250 0    50   ~ 0
+Text Label 8350 2750 0    50   ~ 0
 LOW_BATT
 Wire Wire Line
@@
 Wire Wire Line
 	1400 7200 1600 7200
-Text Label 8350 3050 0    60   ~ 0
+Text Label 8600 1250 0    60   ~ 0
 MICRF_EN
-Wire Wire Line
-	8350 3050 8250 3050
 Text Label 3400 2300 0    60   ~ 0
 I2C_SCL
@@
 	1    0    0    -1
 $EndComp
+NoConn ~ 8250 3050
+Wire Wire Line
+	8250 2750 8350 2750
+Wire Wire Line
+	5050 4350 5400 4350
+NoConn ~ 5050 4450
+Wire Wire Line
+	5100 4550 5050 4550
+Wire Wire Line
+	3850 4950 4050 4950
+$Comp
+L agg-kicad:3v3 #PWR?
+U 1 1 5B28A204
+P 3950 5300
+F 0 "#PWR?" H 3950 5410 50  0001 L CNN
+F 1 "3v3" H 3950 5424 50  0000 C CNN
+F 2 "" H 3950 5300 60  0001 C CNN
+F 3 "" H 3950 5300 60  0001 C CNN
+	1    3950 5300
+	1    0    0    -1
+$EndComp
+Wire Wire Line
+	3950 5050 4050 5050
+Wire Wire Line
+	3950 5300 4050 5300
+Wire Wire Line
+	4050 5300 4050 5150
 $EndSCHEMATC

Commit message: WIP: more pcb layout
Parts:
- X1: footprint agg:M2.5_MOUNT -> agg:M2.5_HOLE
Changed lines of the file:
@@
 NoConn ~ 8250 2350
 NoConn ~ 8250 2450
-NoConn ~ 8250 3150
 NoConn ~ 8250 3350
 Wire Wire Line
@@
 Text Label 8400 2050 0    50   ~ 0
 GPS_~RESET
-Wire Wire Line
-	8400 2050 8250 2050
 $Comp
 L agg-kicad:SL18860DC IC1
@@
 Wire Wire Line
 	8400 2250 8250 2250
-$Comp
-L STM32L051K8U6:STM32L051K8U6 U1
-U 1 1 5A37D9A9
-P 7400 2500
-F 0 "U1" H 7400 4097 60  0000 C CNN
-F 1 "STM32L051K8U6" H 7400 3991 60  0000 C CNN
-F 2 "agg:QFN-32-EP-ST" H 7050 800 60  0001 L CNN
-F 3 "http://www.st.com/resource/en/datasheet/stm32l051t8.pdf" H 7050 700 60  0001 L CNN
-F 4 "2488323" H 7050 600 60  0001 L CNN "Farnell"
-	1    7400 2500
-	1    0    0    -1
-$EndComp
 Wire Wire Line
 	8250 3550 8400 3550
@@
 Wire Wire Line
 	1600 800  1400 800
-Text Label 8600 1150 0    50   ~ 0
+Text Label 8350 3050 0    50   ~ 0
 SOLAR_CELL_VOLTAGE
-Wire Wire Line
-	8600 1150 8250 1150
 Text Label 8350 2750 0    50   ~ 0
 LOW_BATT
@@
 F 0 "X1" H 7578 5646 50  0000 L CNN
 F 1 "MOUNT" H 7578 5555 50  0000 L CNN
-F 2 "agg:M2.5_MOUNT" H 7050 5550 50  0001 C CNN
+F 2 "agg:M2.5_HOLE" H 7050 5550 50  0001 C CNN
 F 3 "" H 7050 5550 50  0001 C CNN
 	1    7050 5550
 	1    0    0    -1
 $EndComp
-NoConn ~ 8250 3050
 Wire Wire Line
 	8250 2750 8350 2750
@@
 	3850 4950 4050 4950
 $Comp
-L agg-kicad:3v3 #PWR?
+L agg-kicad:3v3 #PWR0159
 U 1 1 5B28A204
 P 3950 5300
-F 0 "#PWR?" H 3950 5410 50  0001 L CNN
+F 0 "#PWR0159" H 3950 5410 50  0001 L CNN
 F 1 "3v3" H 3950 5424 50  0000 C CNN
 F 2 "" H 3950 5300 60  0001 C CNN
@@
 Wire Wire Line
 	4050 5300 4050 5150
+NoConn ~ 8250 1150
+Wire Wire Line
+	8250 3050 8350 3050
+$Comp
+L STM32L051K8U6:STM32L051K8U6 U1
+U 1 1 5A37D9A9
+P 7400 2500
+F 0 "U1" H 7400 4097 60  0000 C CNN
+F 1 "STM32L051K8U6" H 7400 3991 60  0000 C CNN
+F 2 "agg:QFN-32-EP-ST" H 7050 800 60  0001 L CNN
+F 3 "http://www.st.com/resource/en/datasheet/stm32l051t8.pdf" H 7050 700 60  0001 L CNN
+F 4 "2488323" H 7050 600 60  0001 L CNN "Farnell"
+	1    7400 2500
+	1    0    0    -1
+$EndComp
+NoConn ~ 8250 3150
+Wire Wire Line
+	8250 2050 8400 2050
 $EndSCHEMATC

Commit message: Stash dual radio version in separate branch
Parts:
- X1: footprint agg:M2.5_HOLE -> agg:M3_HOLE
Connections:
- net labels removed: LOW_BATT
- wire segments 146 -> 144
- no-connect marks 9 -> 10
Changed lines of the file:
@@
 F1 "power.sch" 60
 F2 "solar_cells" I R 1400 800 60
-F3 "LOW_BATT_WARNING" I R 1400 950 50
 $EndSheet
 $Sheet
@@
 	8250 3550 8400 3550
 Wire Wire Line
-	1400 950  1600 950
-Wire Wire Line
 	1600 800  1400 800
 Text Label 8350 3050 0    50   ~ 0
 SOLAR_CELL_VOLTAGE
-Text Label 8350 2750 0    50   ~ 0
-LOW_BATT
 Wire Wire Line
 	8250 1250 8600 1250
 Text Label 1600 800  0    50   ~ 0
 SOLAR_CELL_VOLTAGE
-Text Label 1600 950  0    50   ~ 0
-LOW_BATT
 Text Label 1600 6450 0    60   ~ 0
 SI4460_CLK
@@
 F 0 "X1" H 7578 5646 50  0000 L CNN
 F 1 "MOUNT" H 7578 5555 50  0000 L CNN
-F 2 "agg:M2.5_HOLE" H 7050 5550 50  0001 C CNN
+F 2 "agg:M3_HOLE" H 7050 5550 50  0001 C CNN
 F 3 "" H 7050 5550 50  0001 C CNN
 	1    7050 5550
 	1    0    0    -1
 $EndComp
-Wire Wire Line
-	8250 2750 8350 2750
 Wire Wire Line
 	5050 4350 5400 4350
@@
 Wire Wire Line
 	8250 2050 8400 2050
+NoConn ~ 8250 2750
 $EndSCHEMATC
