File: pcb/gps.sch (KiCad schematic (older format))
At the start: 0 parts

Commit message: Begin gps schematic, assuming dcdc converter used
Parts:
- added C? (x2): 4.7uF, agg:0805, symbol agg-kicad:C
- added C? (x2): 1uF, agg:0402, symbol agg-kicad:C
- added IC?: UBX-G7020, agg:QFN-40-EP-UBLOX, symbol agg-kicad:UBX-G7020
- added L?: 2.2uH, Jerboa:0806, symbol agg-kicad:L
Connections:
- net labels added: 3v3, GND
- wire segments 0 -> 18
Other:
- note added: "Notes:\n- See ubx-g7020 hardware integration manual for info including component values\n- Using DCDC converter; this option is set by the e fuses and appears to be set for chips in ublox max 7q modules\n"
Changed lines of the file:
@@
 $Descr A4 11693 8268
 encoding utf-8
-Sheet 1 4
+Sheet 3 4
 Title ""
 Date ""
@@
 Comment4 ""
 $EndDescr
+$Comp
+L agg-kicad:UBX-G7020 IC?
+U 1 1 5A3FD517
+P 5750 3250
+F 0 "IC?" H 5800 4575 50  0000 C CNN
+F 1 "UBX-G7020" H 5800 4484 50  0000 C CNN
+F 2 "agg:QFN-40-EP-UBLOX" H 5250 1950 50  0001 L CNN
+F 3 "" H 5150 4350 50  0001 C CNN
+	1    5750 3250
+	1    0    0    -1
+$EndComp
+$Comp
+L agg-kicad:3v3 #PWR?
+U 1 1 5A3FD845
+P 5100 1950
+F 0 "#PWR?" H 5100 2060 50  0001 L CNN
+F 1 "3v3" H 5100 2074 50  0000 C CNN
+F 2 "" H 5100 1950 60  0001 C CNN
+F 3 "" H 5100 1950 60  0001 C CNN
+	1    5100 1950
+	1    0    0    -1
+$EndComp
+$Comp
+L agg-kicad:C C?
+U 1 1 5A3FE2DB
+P 5000 2000
+F 0 "C?" H 5050 1805 50  0000 C CNN
+F 1 "4.7uF" H 5050 1896 50  0000 C CNN
+F 2 "agg:0805" H 5000 2000 50  0001 C CNN
+F 3 "" H 5000 2000 50  0001 C CNN
+F 4 "9227857" H 5000 2000 60  0001 C CNN "Farnell"
+	1    5000 2000
+	-1   0    0    1
+$EndComp
+$Comp
+L agg-kicad:L L?
+U 1 1 5A3FE3C6
+P 5000 2250
+F 0 "L?" H 5050 2428 50  0000 C CNN
+F 1 "2.2uH" H 5050 2337 50  0000 C CNN
+F 2 "Jerboa:0806" H 5000 2250 50  0001 C CNN
+F 3 "http://psearch.en.murata.com/inductor/product/LQM2MPN2R2NG0%23.pdf" H 5000 2250 50  0001 C CNN
+F 4 "2470314" H 5000 2250 60  0001 C CNN "Farnell"
+	1    5000 2250
+	1    0    0    -1
+$EndComp
+Wire Wire Line
+	5150 2250 5100 2250
+Wire Wire Line
+	5000 2250 5000 2350
+Connection ~ 5000 2350
+Wire Wire Line
+	5000 2350 5150 2350
+$Comp
+L agg-kicad:C C?
+U 1 1 5A3FE5F0
+P 4150 2550
+F 0 "C?" H 4200 2600 50  0000 C CNN
+F 1 "1uF" H 4200 2700 50  0000 C CNN
+F 2 "agg:0402" H 4150 2550 50  0001 C CNN
+F 3 "" H 4150 2550 50  0001 C CNN
+F 4 "1327658" H 4150 2550 60  0001 C CNN "Farnell"
+	1    4150 2550
+	-1   0    0    1
+$EndComp
+Wire Wire Line
+	4800 2350 5000 2350
+Wire Wire Line
+	5100 2150 5100 2000
+$Comp
+L agg-kicad:GND #PWR?
+U 1 1 5A3FF244
+P 4800 2000
+F 0 "#PWR?" H 4670 2040 50  0001 L CNN
+F 1 "GND" V 4800 1750 50  0000 L CNN
+F 2 "" H 4800 2000 60  0001 C CNN
+F 3 "" H 4800 2000 60  0001 C CNN
+	1    4800 2000
+	0    1    1    0
+$EndComp
+$Comp
+L agg-kicad:GND #PWR?
+U 1 1 5A3FF268
+P 4600 2350
+F 0 "#PWR?" H 4470 2390 50  0001 L CNN
+F 1 "GND" V 4550 2250 50  0000 L CNN
+F 2 "" H 4600 2350 60  0001 C CNN
+F 3 "" H 4600 2350 60  0001 C CNN
+	1    4600 2350
+	0    1    1    0
+$EndComp
+$Comp
+L agg-kicad:GND #PWR?
+U 1 1 5A3FF27F
+P 3950 2450
+F 0 "#PWR?" H 3820 2490 50  0001 L CNN
+F 1 "GND" V 3950 2200 50  0000 L CNN
+F 2 "" H 3950 2450 60  0001 C CNN
+F 3 "" H 3950 2450 60  0001 C CNN
+	1    3950 2450
+	0    1    1    0
+$EndComp
+$Comp
+L agg-kicad:GND #PWR?
+U 1 1 5A3FF296
+P 3950 2550
+F 0 "#PWR?" H 3820 2590 50  0001 L CNN
+F 1 "GND" V 3950 2300 50  0000 L CNN
+F 2 "" H 3950 2550 60  0001 C CNN
+F 3 "" H 3950 2550 60  0001 C CNN
+	1    3950 2550
+	0    1    1    0
+$EndComp
+Wire Wire Line
+	5000 2000 5100 2000
+Connection ~ 5100 2000
+Wire Wire Line
+	5100 2000 5100 1950
+Wire Wire Line
+	4900 2000 4800 2000
+Wire Wire Line
+	4700 2350 4600 2350
+$Comp
+L agg-kicad:3v3 #PWR?
+U 1 1 5A3FF673
+P 4400 2350
+F 0 "#PWR?" H 4400 2460 50  0001 L CNN
+F 1 "3v3" H 4400 2474 50  0000 C CNN
+F 2 "" H 4400 2350 60  0001 C CNN
+F 3 "" H 4400 2350 60  0001 C CNN
+	1    4400 2350
+	1    0    0    -1
+$EndComp
+Wire Wire Line
+	4300 2450 4400 2450
+Wire Wire Line
+	4150 2550 4400 2550
+Wire Wire Line
+	4400 2350 4400 2450
+Connection ~ 4400 2450
+Wire Wire Line
+	4400 2450 5150 2450
+Wire Wire Line
+	4400 2450 4400 2550
+Connection ~ 4400 2550
+Wire Wire Line
+	4400 2550 5150 2550
+Wire Wire Line
+	4200 2450 3950 2450
+Wire Wire Line
+	4050 2550 3950 2550
+Text Notes 900  1050 0    60   ~ 0
+Notes:\n- See ubx-g7020 hardware integration manual for info including component values\n- Using DCDC converter; this option is set by the e fuses and appears to be set for  chips in ublox max 7q modules\n
+$Comp
+L agg-kicad:C C?
+U 1 1 5A407461
+P 4800 2350
+F 0 "C?" H 4850 2155 50  0000 C CNN
+F 1 "4.7uF" H 4850 2246 50  0000 C CNN
+F 2 "agg:0805" H 4800 2350 50  0001 C CNN
+F 3 "" H 4800 2350 50  0001 C CNN
+F 4 "9227857" H 4800 2350 60  0001 C CNN "Farnell"
+	1    4800 2350
+	-1   0    0    1
+$EndComp
+Wire Wire Line
+	5150 2150 5100 2150
+$Comp
+L agg-kicad:C C?
+U 1 1 5A408D67
+P 4300 2450
+F 0 "C?" H 4350 2500 50  0000 C CNN
+F 1 "1uF" H 4350 2600 50  0000 C CNN
+F 2 "agg:0402" H 4300 2450 50  0001 C CNN
+F 3 "" H 4300 2450 50  0001 C CNN
+F 4 "1327658" H 4300 2450 60  0001 C CNN "Farnell"
+	1    4300 2450
+	-1   0    0    1
+$EndComp
 $EndSCHEMATC

Commit message: Add some component values
Parts:
- added C10: 2.2uF, agg:0402, symbol agg-kicad:C
- added C16, C4, C5: 1uF, agg:0402, symbol agg-kicad:C
- gave numbers to parts that had none: 5
Connections:
- wire segments 18 -> 36
Changed lines of the file:
@@
 $EndComp
 $Comp
-L agg-kicad:C C?
+L agg-kicad:C C7
 U 1 1 5A3FE2DB
 P 5000 2000
-F 0 "C?" H 5050 1805 50  0000 C CNN
+F 0 "C7" H 5050 1805 50  0000 C CNN
 F 1 "4.7uF" H 5050 1896 50  0000 C CNN
 F 2 "agg:0805" H 5000 2000 50  0001 C CNN
@@
 $EndComp
 $Comp
-L agg-kicad:L L?
+L agg-kicad:L L2
 U 1 1 5A3FE3C6
 P 5000 2250
-F 0 "L?" H 5050 2428 50  0000 C CNN
+F 0 "L2" H 5050 2428 50  0000 C CNN
 F 1 "2.2uH" H 5050 2337 50  0000 C CNN
 F 2 "Jerboa:0806" H 5000 2250 50  0001 C CNN
@@
 	5000 2350 5150 2350
 $Comp
-L agg-kicad:C C?
+L agg-kicad:C C8
 U 1 1 5A3FE5F0
 P 4150 2550
-F 0 "C?" H 4200 2600 50  0000 C CNN
+F 0 "C8" H 4200 2600 50  0000 C CNN
 F 1 "1uF" H 4200 2700 50  0000 C CNN
 F 2 "agg:0402" H 4150 2550 50  0001 C CNN
@@
 Notes:\n- See ubx-g7020 hardware integration manual for info including component values\n- Using DCDC converter; this option is set by the e fuses and appears to be set for  chips in ublox max 7q modules\n
 $Comp
-L agg-kicad:C C?
+L agg-kicad:C C6
 U 1 1 5A407461
 P 4800 2350
-F 0 "C?" H 4850 2155 50  0000 C CNN
+F 0 "C6" H 4850 2155 50  0000 C CNN
 F 1 "4.7uF" H 4850 2246 50  0000 C CNN
 F 2 "agg:0805" H 4800 2350 50  0001 C CNN
@@
 	5150 2150 5100 2150
 $Comp
-L agg-kicad:C C?
+L agg-kicad:C C9
 U 1 1 5A408D67
 P 4300 2450
-F 0 "C?" H 4350 2500 50  0000 C CNN
+F 0 "C9" H 4350 2500 50  0000 C CNN
 F 1 "1uF" H 4350 2600 50  0000 C CNN
 F 2 "agg:0402" H 4300 2450 50  0001 C CNN
@@
 	-1   0    0    1
 $EndComp
+Wire Wire Line
+	5150 2950 5100 2950
+Wire Wire Line
+	5100 2950 5100 2850
+Wire Wire Line
+	5100 2750 5150 2750
+Wire Wire Line
+	5150 2850 5100 2850
+Connection ~ 5100 2850
+Wire Wire Line
+	5100 2850 5100 2750
+$Comp
+L agg-kicad:C C4
+U 1 1 5A40F9D1
+P 4250 3050
+F 0 "C4" H 4300 3100 50  0000 C CNN
+F 1 "1uF" H 4300 3200 50  0000 C CNN
+F 2 "agg:0402" H 4250 3050 50  0001 C CNN
+F 3 "" H 4250 3050 50  0001 C CNN
+F 4 "1327658" H 4250 3050 60  0001 C CNN "Farnell"
+	1    4250 3050
+	0    -1   -1   0
+$EndComp
+$Comp
+L agg-kicad:C C16
+U 1 1 5A4104B9
+P 4500 3150
+F 0 "C16" H 4550 3200 50  0000 C CNN
+F 1 "1uF" H 4550 3300 50  0000 C CNN
+F 2 "agg:0402" H 4500 3150 50  0001 C CNN
+F 3 "" H 4500 3150 50  0001 C CNN
+F 4 "1327658" H 4500 3150 60  0001 C CNN "Farnell"
+	1    4500 3150
+	0    -1   -1   0
+$EndComp
+$Comp
+L agg-kicad:C C5
+U 1 1 5A41105B
+P 5000 3350
+F 0 "C5" H 5050 3400 50  0000 C CNN
+F 1 "1uF" H 5050 3500 50  0000 C CNN
+F 2 "agg:0402" H 5000 3350 50  0001 C CNN
+F 3 "" H 5000 3350 50  0001 C CNN
+F 4 "1327658" H 5000 3350 60  0001 C CNN "Farnell"
+	1    5000 3350
+	0    -1   -1   0
+$EndComp
+$Comp
+L agg-kicad:C C10
+U 1 1 5A411184
+P 4750 3250
+F 0 "C10" H 4800 3300 50  0000 C CNN
+F 1 "2.2uF" H 4800 3400 50  0000 C CNN
+F 2 "agg:0402" H 4750 3250 50  0001 C CNN
+F 3 "" H 4750 3250 50  0001 C CNN
+F 4 "2672109" H 4750 3250 50  0001 C CNN "Farnell"
+	1    4750 3250
+	0    -1   -1   0
+$EndComp
+$Comp
+L agg-kicad:GND #PWR?
+U 1 1 5A413B66
+P 4250 3450
+F 0 "#PWR?" H 4120 3490 50  0001 L CNN
+F 1 "GND" H 4250 3350 50  0000 C CNN
+F 2 "" H 4250 3450 50  0001 C CNN
+F 3 "" H 4250 3450 50  0001 C CNN
+	1    4250 3450
+	1    0    0    -1
+$EndComp
+$Comp
+L agg-kicad:GND #PWR?
+U 1 1 5A414298
+P 5000 2650
+F 0 "#PWR?" H 4870 2690 50  0001 L CNN
+F 1 "GND" V 5000 2400 50  0000 L CNN
+F 2 "" H 5000 2650 60  0001 C CNN
+F 3 "" H 5000 2650 60  0001 C CNN
+	1    5000 2650
+	0    1    1    0
+$EndComp
+Wire Wire Line
+	5150 2650 5000 2650
+Wire Wire Line
+	5000 3250 5150 3250
+Wire Wire Line
+	5150 3150 4750 3150
+Wire Wire Line
+	4500 3050 5150 3050
+Connection ~ 5100 2950
+Wire Wire Line
+	4250 2950 5100 2950
+Wire Wire Line
+	4500 3150 4500 3400
+Wire Wire Line
+	5000 3350 5000 3400
+Wire Wire Line
+	4750 3250 4750 3400
+Wire Wire Line
+	5000 3400 4750 3400
+Connection ~ 4750 3400
+Wire Wire Line
+	4750 3400 4500 3400
+Wire Wire Line
+	4250 3450 4250 3400
+Connection ~ 4500 3400
+Wire Wire Line
+	4500 3400 4250 3400
+Connection ~ 4250 3400
+Wire Wire Line
+	4250 3400 4250 3050
 $EndSCHEMATC

Commit message: Schematic almost done.
Parts:
- removed C10: 2.2uF, agg:0402, symbol agg-kicad:C
- removed C16, C4, C5, C8, C9: 1uF, agg:0402, symbol agg-kicad:C
- removed C6, C7: 4.7uF, agg:0805, symbol agg-kicad:C
- removed IC?: UBX-G7020, agg:QFN-40-EP-UBLOX, symbol agg-kicad:UBX-G7020
- removed L2: 2.2uH, Jerboa:0806, symbol agg-kicad:L
- added C301: C, symbol C
- added IC301: MAX-7Q, agg-unchecked:MAX-7Q, symbol MAX-7Q
- added P301: COAX, agg:SMA-EDGE, symbol COAX
Connections:
- net labels added: GPS_RX, GPS_TX
- wire segments 36 -> 14
- no-connect marks 0 -> 7
Other:
- note added: "GPS"
- note removed: "Notes:\n- See ubx-g7020 hardware integration manual for info including component values\n- Using DCDC converter; this option is set by the e fuses and appears to be set for chips in ublox max 7q modules\n"

Commit message: Attempt to fix symbol library problems from old kicad version
Parts:
- C301: symbol C -> agg-kicad:C
- IC301: footprint agg-unchecked:MAX-7Q -> agg:MAX-7Q; symbol MAX-7Q -> agg-kicad:MAX-7Q
- P301: symbol COAX -> agg-kicad:COAX
Connections:
- wire segments 14 -> 19
Changed lines of the file:
@@
-EESchema Schematic File Version 2
-LIBS:agg-kicad
+EESchema Schematic File Version 4
 LIBS:jerboa-cache
-EELAYER 25 0
+EELAYER 26 0
 EELAYER END
 $Descr A4 11693 8268
@@
 $EndDescr
 $Comp
-L MAX-7Q IC301
+L agg-kicad:MAX-7Q IC301
 U 1 1 5A6DE5A1
 P 5850 3300
 F 0 "IC301" H 5450 3800 50  0000 L CNN
 F 1 "MAX-7Q" H 5450 2600 50  0000 L CNN
-F 2 "agg-unchecked:MAX-7Q" H 5450 2500 50  0001 L CNN
+F 2 "agg:MAX-7Q" H 5450 2500 50  0001 L CNN
 F 3 "" H 5800 3300 50  0001 C CNN
 F 4 "MAX-7Q" H 5450 2400 50  0001 L CNN "HabSupplies"
@@
 $EndComp
 Wire Wire Line
-	5100 3100 5350 3100
+	5100 3100 5250 3100
 Wire Wire Line
-	5250 2800 5250 3100
+	5250 2800 5250 2900
 Wire Wire Line
 	5350 3000 5250 3000
@@
 Connection ~ 5250 2900
 Wire Wire Line
-	5100 3200 5350 3200
+	5100 3200 5250 3200
 Connection ~ 5250 3200
 Connection ~ 5250 3100
 $Comp
-L GND #PWR013
+L agg-kicad:GND #PWR013
 U 1 1 5A6DE6B0
 P 5250 3250
@@
 	5250 3250 5250 3200
 $Comp
-L C C301
+L agg-kicad:C C301
 U 1 1 5A6DE6E0
 P 5100 3100
@@
 $EndComp
 $Comp
-L 3v3 #PWR014
+L agg-kicad:3v3 #PWR014
 U 1 1 5A6DE74F
 P 5250 2800
@@
 	6400 2900 6400 2850
 $Comp
-L COAX P301
+L agg-kicad:COAX P301
 U 1 1 5A6DE78F
 P 6700 2750
@@
 	6700 3000 6700 2850
 Wire Wire Line
-	6800 2850 6800 3150
+	6800 2850 6800 3100
 Wire Wire Line
 	6250 3100 6800 3100
 Connection ~ 6800 3100
 $Comp
-L GND #PWR015
+L agg-kicad:GND #PWR015
 U 1 1 5A6DE826
 P 6800 3150
@@
 $EndComp
 $Comp
-L GND #PWR016
+L agg-kicad:GND #PWR016
 U 1 1 5A6DE840
 P 6400 2850
@@
 Text HLabel 5250 3600 0    60   Input ~ 0
 GPS_RX
+Wire Wire Line
+	5250 3000 5250 3100
+Wire Wire Line
+	5250 2900 5250 3000
+Wire Wire Line
+	5250 3200 5350 3200
+Wire Wire Line
+	5250 3100 5350 3100
+Wire Wire Line
+	6800 3100 6800 3150
 $EndSCHEMATC

Commit message: Some schematic work, create a todo with ideas for power supply components
Parts:
- removed IC301: MAX-7Q, agg:MAX-7Q, symbol agg-kicad:MAX-7Q
- added D?: ESD_DIODE, agg:0402, symbol agg-kicad:ESD_DIODE
- added IC?: MAX-M8Q, agg:MAX-M8Q, symbol agg-kicad:MAX-M8Q
- C301: value C -> 100nF; footprint (none) -> agg:0402; Farnell (none) -> 2496810
Connections:
- net labels added: GPS_~RESET
- wire segments 19 -> 23
- no-connect marks 7 -> 8
Other:
- moved on the sheet: C301, P301
Changed lines of the file:
@@
 $EndDescr
 $Comp
-L agg-kicad:MAX-7Q IC301
-U 1 1 5A6DE5A1
-P 5850 3300
-F 0 "IC301" H 5450 3800 50  0000 L CNN
-F 1 "MAX-7Q" H 5450 2600 50  0000 L CNN
-F 2 "agg:MAX-7Q" H 5450 2500 50  0001 L CNN
-F 3 "" H 5800 3300 50  0001 C CNN
-F 4 "MAX-7Q" H 5450 2400 50  0001 L CNN "HabSupplies"
-	1    5850 3300
+L agg-kicad:C C301
+U 1 1 5A6DE6E0
+P 4950 2700
+F 0 "C301" H 5000 2770 50  0000 C CNN
+F 1 "100nF" H 5000 2600 50  0000 C CNN
+F 2 "agg:0402" H 4950 2700 50  0001 C CNN
+F 3 "" H 4950 2700 50  0001 C CNN
+F 4 "2496810" H 4950 2700 50  0001 C CNN "Farnell"
+	1    4950 2700
+	0    1    1    0
+$EndComp
+$Comp
+L agg-kicad:COAX P301
+U 1 1 5A6DE78F
+P 6800 3500
+F 0 "P301" H 6800 3600 50  0000 C CNN
+F 1 "COAX" H 6800 3350 50  0000 C CNN
+F 2 "agg:SMA-EDGE" H 6800 3290 50  0001 C CNN
+F 3 "" H 6900 3400 50  0001 C CNN
+F 4 "1608592" H 6800 3220 50  0001 C CNN "Farnell"
+	1    6800 3500
+	1    0    0    -1
+$EndComp
+Text Notes 5600 2150 0    118  ~ 0
+GPS
+Text HLabel 6500 2900 2    60   Input ~ 0
+GPS_TX
+Text HLabel 6500 2800 2    60   Input ~ 0
+GPS_RX
+$Comp
+L agg-kicad:MAX-M8Q IC?
+U 1 1 5A6E4106
+P 5800 3000
+F 0 "IC?" H 5800 3725 50  0000 C CNN
+F 1 "MAX-M8Q" H 5800 3634 50  0000 C CNN
+F 2 "agg:MAX-M8Q" H 5300 2300 50  0001 L CNN
+F 3 "https://www.u-blox.com/sites/default/files/MAX-M8-FW3_DataSheet_%28UBX-15031506%29.pdf" H 5300 2200 50  0001 L CNN
+	1    5800 3000
+	1    0    0    -1
+$EndComp
+$Comp
+L agg-kicad:3v3 #PWR?
+U 1 1 5A6F25D1
+P 5100 2450
+F 0 "#PWR?" H 5100 2560 50  0001 L CNN
+F 1 "3v3" H 5100 2540 50  0000 C CNN
+F 2 "" H 5100 2450 60  0000 C CNN
+F 3 "" H 5100 2450 60  0000 C CNN
+	1    5100 2450
 	1    0    0    -1
 $EndComp
 Wire Wire Line
-	5100 3100 5250 3100
+	5200 2500 5100 2500
 Wire Wire Line
-	5250 2800 5250 2900
+	5100 2500 5100 2450
 Wire Wire Line
-	5350 3000 5250 3000
-Connection ~ 5250 3000
+	5200 2700 5100 2700
 Wire Wire Line
-	5350 2900 5250 2900
-Connection ~ 5250 2900
+	5100 2700 5100 2600
+Connection ~ 5100 2500
 Wire Wire Line
-	5100 3200 5250 3200
-Connection ~ 5250 3200
-Connection ~ 5250 3100
+	5200 2600 5100 2600
+Connection ~ 5100 2600
+Wire Wire Line
+	5100 2600 5100 2500
 $Comp
-L agg-kicad:GND #PWR013
-U 1 1 5A6DE6B0
-P 5250 3250
-F 0 "#PWR013" H 5120 3290 50  0001 L CNN
-F 1 "GND" H 5250 3150 50  0000 C CNN
-F 2 "" H 5250 3250 60  0000 C CNN
-F 3 "" H 5250 3250 60  0000 C CNN
-	1    5250 3250
+L agg-kicad:GND #PWR?
+U 1 1 5A6F2D41
+P 5100 3050
+F 0 "#PWR?" H 4970 3090 50  0001 L CNN
+F 1 "GND" H 5000 3000 50  0000 C CNN
+F 2 "" H 5100 3050 60  0000 C CNN
+F 3 "" H 5100 3050 60  0000 C CNN
+	1    5100 3050
 	1    0    0    -1
 $EndComp
 Wire Wire Line
-	5250 3250 5250 3200
+	5100 3000 5100 3050
+Wire Wire Line
+	5100 3000 5200 3000
+Wire Wire Line
+	5200 2900 5100 2900
+Wire Wire Line
+	5100 2900 5100 3000
+Connection ~ 5100 3000
+Wire Wire Line
+	5200 2800 5100 2800
+Wire Wire Line
+	5100 2800 5100 2900
+Connection ~ 5100 2900
+NoConn ~ 6400 2500
+NoConn ~ 6400 2600
+Wire Wire Line
+	6500 2800 6400 2800
+Wire Wire Line
+	6400 2900 6500 2900
+NoConn ~ 6400 3100
+NoConn ~ 6400 3200
+NoConn ~ 6400 3300
 $Comp
-L agg-kicad:C C301
-U 1 1 5A6DE6E0
-P 5100 3100
-F 0 "C301" H 5150 3170 50  0000 C CNN
-F 1 "C" H 5150 3000 50  0000 C CNN
-F 2 "" H 5100 3100 50  0001 C CNN
-F 3 "" H 5100 3100 50  0001 C CNN
-	1    5100 3100
+L agg-kicad:ESD_DIODE D?
+U 1 1 5A6F5EFB
+P 6500 3600
+F 0 "D?" V 6500 3658 50  0000 L CNN
+F 1 "ESD_DIODE" H 6450 3500 50  0001 L CNN
+F 2 "agg:0402" H 6450 3400 50  0001 L CNN
+F 3 "http://www.farnell.com/datasheets/1772768.pdf" H 6400 3600 50  0001 C CNN
+F 4 "2368169" H 6450 3300 50  0001 L CNN "Farnell"
+	1    6500 3600
 	0    1    1    0
 $EndComp
 $Comp
-L agg-kicad:3v3 #PWR014
-U 1 1 5A6DE74F
-P 5250 2800
-F 0 "#PWR014" H 5250 2910 50  0001 L CNN
-F 1 "3v3" H 5250 2890 50  0000 C CNN
-F 2 "" H 5250 2800 60  0000 C CNN
-F 3 "" H 5250 2800 60  0000 C CNN
-	1    5250 2800
+L agg-kicad:GND #PWR?
+U 1 1 5A6F5FFD
+P 6500 3800
+F 0 "#PWR?" H 6370 3840 50  0001 L CNN
+F 1 "GND" H 6500 3887 50  0000 C CNN
+F 2 "" H 6500 3800 50  0001 C CNN
+F 3 "" H 6500 3800 50  0001 C CNN
+	1    6500 3800
 	1    0    0    -1
 $EndComp
 Wire Wire Line
-	6250 2900 6400 2900
+	6500 3800 6500 3750
 Wire Wire Line
-	6400 2900 6400 2850
-$Comp
-L agg-kicad:COAX P301
-U 1 1 5A6DE78F
-P 6700 2750
-F 0 "P301" H 6700 2850 50  0000 C CNN
-F 1 "COAX" H 6700 2600 50  0000 C CNN
-F 2 "agg:SMA-EDGE" H 6700 2540 50  0001 C CNN
-F 3 "" H 6800 2650 50  0001 C CNN
-F 4 "1608592" H 6700 2470 50  0001 C CNN "Farnell"
-	1    6700 2750
-	0    -1   -1   0
-$EndComp
+	6500 3500 6400 3500
 Wire Wire Line
-	6250 3000 6700 3000
+	6500 3500 6700 3500
+Connection ~ 6500 3500
 Wire Wire Line
-	6700 3000 6700 2850
+	6700 3600 6700 3750
 Wire Wire Line
-	6800 2850 6800 3100
+	6700 3750 6500 3750
+Connection ~ 6500 3750
 Wire Wire Line
-	6250 3100 6800 3100
-Connection ~ 6800 3100
-$Comp
-L agg-kicad:GND #PWR015
-U 1 1 5A6DE826
-P 6800 3150
-F 0 "#PWR015" H 6670 3190 50  0001 L CNN
-F 1 "GND" H 6800 3050 50  0000 C CNN
-F 2 "" H 6800 3150 60  0000 C CNN
-F 3 "" H 6800 3150 60  0000 C CNN
-	1    6800 3150
-	1    0    0    -1
-$EndComp
-$Comp
-L agg-kicad:GND #PWR016
-U 1 1 5A6DE840
-P 6400 2850
-F 0 "#PWR016" H 6270 2890 50  0001 L CNN
-F 1 "GND" H 6400 2750 50  0000 C CNN
-F 2 "" H 6400 2850 60  0000 C CNN
-F 3 "" H 6400 2850 60  0000 C CNN
-	1    6400 2850
-	-1   0    0    1
-$EndComp
-NoConn ~ 6250 3200
-NoConn ~ 6250 3600
-NoConn ~ 6250 3700
-NoConn ~ 6250 3800
-NoConn ~ 6250 3900
-NoConn ~ 5350 3800
-NoConn ~ 5350 3900
+	6500 3750 6500 3700
+NoConn ~ 5200 3400
+NoConn ~ 5200 3300
+Text HLabel 5150 3200 0    60   Input ~ 0
+GPS_~RESET
 Wire Wire Line
-	5350 3500 5250 3500
+	5200 3200 5150 3200
+NoConn ~ 5200 3500
 Wire Wire Line
-	5350 3600 5250 3600
-Text Notes 5600 2150 0    118  ~ 0
-GPS
-Text HLabel 5250 3500 0    60   Input ~ 0
-GPS_TX
-Text HLabel 5250 3600 0    60   Input ~ 0
-GPS_RX
+	4950 2700 5100 2700
+Connection ~ 5100 2700
 Wire Wire Line
-	5250 3000 5250 3100
-Wire Wire Line
-	5250 2900 5250 3000
-Wire Wire Line
-	5250 3200 5350 3200
-Wire Wire Line
-	5250 3100 5350 3100
-Wire Wire Line
-	6800 3100 6800 3150
+	4950 2800 5100 2800
+Connection ~ 5100 2800
 $EndSCHEMATC

Commit message: Add TPS61025 switching regulator to schematic
Parts:
- C301: Farnell 2496810 -> 1288282
Changed lines of the file:
@@
 F 2 "agg:0402" H 4950 2700 50  0001 C CNN
 F 3 "" H 4950 2700 50  0001 C CNN
-F 4 "2496810" H 4950 2700 50  0001 C CNN "Farnell"
+F 4 "1288282" H 4950 2700 50  0001 C CNN "Farnell"
 	1    4950 2700
 	0    1    1    0

Commit message: Create some more schematic symbols and footprints
Changed lines of the file:
@@
 	5200 2500 5100 2500
 Wire Wire Line
-	5100 2500 5100 2450
+	5100 2450 5100 2700
 Wire Wire Line
-	5200 2700 5100 2700
-Wire Wire Line
-	5100 2700 5100 2600
+	4950 2700 5200 2700
 Connection ~ 5100 2500
 Wire Wire Line
 	5200 2600 5100 2600
 Connection ~ 5100 2600
-Wire Wire Line
-	5100 2600 5100 2500
 $Comp
 L agg-kicad:GND #PWR?
@@
 $EndComp
 Wire Wire Line
-	5100 3000 5100 3050
+	5100 2800 5100 3050
 Wire Wire Line
 	5100 3000 5200 3000
 Wire Wire Line
 	5200 2900 5100 2900
-Wire Wire Line
-	5100 2900 5100 3000
 Connection ~ 5100 3000
 Wire Wire Line
-	5200 2800 5100 2800
-Wire Wire Line
-	5100 2800 5100 2900
+	4950 2800 5200 2800
 Connection ~ 5100 2900
 NoConn ~ 6400 2500
@@
 $EndComp
 Wire Wire Line
-	6500 3800 6500 3750
+	6500 3700 6500 3800
 Wire Wire Line
-	6500 3500 6400 3500
-Wire Wire Line
-	6500 3500 6700 3500
+	6400 3500 6700 3500
 Connection ~ 6500 3500
 Wire Wire Line
@@
 	6700 3750 6500 3750
 Connection ~ 6500 3750
-Wire Wire Line
-	6500 3750 6500 3700
 NoConn ~ 5200 3400
 NoConn ~ 5200 3300
@@
 	5200 3200 5150 3200
 NoConn ~ 5200 3500
-Wire Wire Line
-	4950 2700 5100 2700
 Connection ~ 5100 2700
-Wire Wire Line
-	4950 2800 5100 2800
 Connection ~ 5100 2800
 $EndSCHEMATC
