File: pcb/power.sch (KiCad schematic (older format))
At the start: 0 parts

Commit message: Schematic almost done.
Parts:
- added C201, C203: 2u2, symbol C
- added C202: 1n, symbol C
- added IC201: ADP3335, agg:MSOP-8, symbol ADP3335
- added J201: CONN_01x02, symbol CONN_01x02
Connections:
- net labels added: 3v3, GND, VBATT
- wire segments 0 -> 18
Changed lines of the file:
@@
 Comment4 ""
 $EndDescr
+$Comp
+L ADP3335 IC201
+U 1 1 5A6DE9D3
+P 5250 3700
+F 0 "IC201" H 5050 3900 50  0000 L CNN
+F 1 "ADP3335" H 5050 3400 50  0000 L CNN
+F 2 "agg:MSOP-8" H 5050 3300 50  0001 L CNN
+F 3 "" H 5650 3300 50  0001 C CNN
+F 4 "2067775" H 5050 3200 50  0001 L CNN "Farnell"
+	1    5250 3700
+	1    0    0    -1
+$EndComp
+Wire Wire Line
+	5800 3600 5800 3750
+Connection ~ 5800 3700
+Wire Wire Line
+	5800 3850 5800 3900
+Wire Wire Line
+	4850 3800 4950 3800
+Wire Wire Line
+	4850 3600 4850 3800
+Connection ~ 4850 3700
+$Comp
+L CONN_01x02 J201
+U 1 1 5A6DEB31
+P 4450 3750
+F 0 "J201" V 4350 3600 50  0000 L CNN
+F 1 "CONN_01x02" V 4250 3500 50  0000 L CNN
+F 2 "" H 4450 3750 50  0001 C CNN
+F 3 "" H 4450 3750 50  0001 C CNN
+	1    4450 3750
+	1    0    0    -1
+$EndComp
+Wire Wire Line
+	4550 3600 4550 3750
+Wire Wire Line
+	4550 3850 4550 3950
+Connection ~ 4550 3700
+$Comp
+L VBATT #PWR09
+U 1 1 5A6DEBBC
+P 4550 3600
+F 0 "#PWR09" H 4550 3710 50  0001 L CNN
+F 1 "VBATT" H 4550 3690 50  0000 C CNN
+F 2 "" H 4550 3600 60  0000 C CNN
+F 3 "" H 4550 3600 60  0000 C CNN
+	1    4550 3600
+	1    0    0    -1
+$EndComp
+$Comp
+L GND #PWR010
+U 1 1 5A6DEBD4
+P 4550 3950
+F 0 "#PWR010" H 4420 3990 50  0001 L CNN
+F 1 "GND" H 4550 3850 50  0000 C CNN
+F 2 "" H 4550 3950 60  0000 C CNN
+F 3 "" H 4550 3950 60  0000 C CNN
+	1    4550 3950
+	1    0    0    -1
+$EndComp
+Connection ~ 4550 3900
+$Comp
+L C C202
+U 1 1 5A6DEC39
+P 5800 3750
+F 0 "C202" H 5850 3820 50  0000 C CNN
+F 1 "1n" H 5850 3680 50  0000 C CNN
+F 2 "" H 5800 3750 50  0001 C CNN
+F 3 "" H 5800 3750 50  0001 C CNN
+F 4 "Value" H 5800 3750 60  0001 C CNN "Fieldname"
+	1    5800 3750
+	0    1    1    0
+$EndComp
+$Comp
+L C C203
+U 1 1 5A6DEC8C
+P 6050 3750
+F 0 "C203" H 6100 3820 50  0000 C CNN
+F 1 "2u2" H 6100 3680 50  0000 C CNN
+F 2 "" H 6050 3750 50  0001 C CNN
+F 3 "" H 6050 3750 50  0001 C CNN
+F 4 "Value" H 6050 3750 60  0001 C CNN "Fieldname"
+	1    6050 3750
+	0    1    1    0
+$EndComp
+Wire Wire Line
+	6050 3700 6050 3750
+$Comp
+L 3v3 #PWR011
+U 1 1 5A6DECCE
+P 5800 3600
+F 0 "#PWR011" H 5800 3710 50  0001 L CNN
+F 1 "3v3" H 5800 3690 50  0000 C CNN
+F 2 "" H 5800 3600 60  0000 C CNN
+F 3 "" H 5800 3600 60  0000 C CNN
+	1    5800 3600
+	1    0    0    -1
+$EndComp
+$Comp
+L GND #PWR012
+U 1 1 5A6DECEA
+P 6050 3900
+F 0 "#PWR012" H 5920 3940 50  0001 L CNN
+F 1 "GND" H 6050 3800 50  0000 C CNN
+F 2 "" H 6050 3900 60  0000 C CNN
+F 3 "" H 6050 3900 60  0000 C CNN
+	1    6050 3900
+	1    0    0    -1
+$EndComp
+Wire Wire Line
+	6050 3900 6050 3850
+$Comp
+L C C201
+U 1 1 5A6DED5C
+P 4700 3750
+F 0 "C201" H 4750 3820 50  0000 C CNN
+F 1 "2u2" H 4750 3680 50  0000 C CNN
+F 2 "" H 4700 3750 50  0001 C CNN
+F 3 "" H 4700 3750 50  0001 C CNN
+F 4 "Value" H 4700 3750 60  0001 C CNN "Fieldname"
+	1    4700 3750
+	0    1    1    0
+$EndComp
+Wire Wire Line
+	4700 3850 4700 3900
+Connection ~ 4700 3900
+Wire Wire Line
+	4700 3750 4700 3700
+Connection ~ 4700 3700
+Wire Wire Line
+	4550 3900 4950 3900
+Wire Wire Line
+	4550 3700 4950 3700
+Wire Wire Line
+	5650 3600 5650 3800
+Connection ~ 5650 3700
+Connection ~ 5650 3600
+Connection ~ 5650 3800
+Wire Wire Line
+	5650 3800 5550 3800
+Wire Wire Line
+	5550 3600 5650 3600
+Wire Wire Line
+	5550 3700 6050 3700
+Wire Wire Line
+	5800 3900 5550 3900
+Wire Wire Line
+	4950 3600 4850 3600
 $EndSCHEMATC

Commit message: Attempt to fix symbol library problems from old kicad version
Parts:
- C201, C202, C203: symbol C -> agg-kicad:C
- IC201: symbol ADP3335 -> agg-kicad:ADP3335
- J201: symbol CONN_01x02 -> agg-kicad:CONN_01x02
Connections:
- wire segments 18 -> 28
Changed lines of the file:
@@
-EESchema Schematic File Version 2
-LIBS:agg-kicad
+EESchema Schematic File Version 4
 LIBS:jerboa-cache
-EELAYER 25 0
+EELAYER 26 0
 EELAYER END
 $Descr A4 11693 8268
@@
 $EndDescr
 $Comp
-L ADP3335 IC201
+L agg-kicad:ADP3335 IC201
 U 1 1 5A6DE9D3
 P 5250 3700
@@
 $EndComp
 Wire Wire Line
-	5800 3600 5800 3750
+	5800 3600 5800 3700
 Connection ~ 5800 3700
 Wire Wire Line
@@
 	4850 3800 4950 3800
 Wire Wire Line
-	4850 3600 4850 3800
+	4850 3600 4850 3700
 Connection ~ 4850 3700
 $Comp
-L CONN_01x02 J201
+L agg-kicad:CONN_01x02 J201
 U 1 1 5A6DEB31
 P 4450 3750
@@
 $EndComp
 Wire Wire Line
-	4550 3600 4550 3750
+	4550 3600 4550 3700
 Wire Wire Line
-	4550 3850 4550 3950
+	4550 3850 4550 3900
 Connection ~ 4550 3700
 $Comp
-L VBATT #PWR09
+L agg-kicad:VBATT #PWR09
 U 1 1 5A6DEBBC
 P 4550 3600
@@
 $EndComp
 $Comp
-L GND #PWR010
+L agg-kicad:GND #PWR010
 U 1 1 5A6DEBD4
 P 4550 3950
@@
 Connection ~ 4550 3900
 $Comp
-L C C202
+L agg-kicad:C C202
 U 1 1 5A6DEC39
 P 5800 3750
@@
 $EndComp
 $Comp
-L C C203
+L agg-kicad:C C203
 U 1 1 5A6DEC8C
 P 6050 3750
@@
 	6050 3700 6050 3750
 $Comp
-L 3v3 #PWR011
+L agg-kicad:3v3 #PWR011
 U 1 1 5A6DECCE
 P 5800 3600
@@
 $EndComp
 $Comp
-L GND #PWR012
+L agg-kicad:GND #PWR012
 U 1 1 5A6DECEA
 P 6050 3900
@@
 	6050 3900 6050 3850
 $Comp
-L C C201
+L agg-kicad:C C201
 U 1 1 5A6DED5C
 P 4700 3750
@@
 Connection ~ 4700 3700
 Wire Wire Line
-	4550 3900 4950 3900
+	4550 3900 4700 3900
 Wire Wire Line
-	4550 3700 4950 3700
+	4550 3700 4700 3700
 Wire Wire Line
-	5650 3600 5650 3800
+	5650 3600 5650 3700
 Connection ~ 5650 3700
-Connection ~ 5650 3600
-Connection ~ 5650 3800
 Wire Wire Line
 	5650 3800 5550 3800
@@
 	5550 3600 5650 3600
 Wire Wire Line
-	5550 3700 6050 3700
+	5550 3700 5650 3700
 Wire Wire Line
 	5800 3900 5550 3900
 Wire Wire Line
 	4950 3600 4850 3600
+Wire Wire Line
+	5800 3700 5800 3750
+Wire Wire Line
+	5800 3700 6050 3700
+Wire Wire Line
+	4850 3700 4850 3800
+Wire Wire Line
+	4850 3700 4950 3700
+Wire Wire Line
+	4550 3700 4550 3750
+Wire Wire Line
+	4550 3900 4550 3950
+Wire Wire Line
+	4700 3900 4950 3900
+Wire Wire Line
+	4700 3700 4850 3700
+Wire Wire Line
+	5650 3700 5650 3800
+Wire Wire Line
+	5650 3700 5800 3700
 $EndSCHEMATC

Commit message: Some schematic work, create a todo with ideas for power supply components
Parts:
- removed C201, C203: 2u2, symbol agg-kicad:C
- removed C202: 1n, symbol agg-kicad:C
- removed IC201: ADP3335, agg:MSOP-8, symbol agg-kicad:ADP3335
- removed J201: CONN_01x02, symbol agg-kicad:CONN_01x02
Connections:
- net labels removed: 3v3, GND, VBATT
- wire segments 28 -> 0
Changed lines of the file:
@@
 Comment4 ""
 $EndDescr
-$Comp
-L agg-kicad:ADP3335 IC201
-U 1 1 5A6DE9D3
-P 5250 3700
-F 0 "IC201" H 5050 3900 50  0000 L CNN
-F 1 "ADP3335" H 5050 3400 50  0000 L CNN
-F 2 "agg:MSOP-8" H 5050 3300 50  0001 L CNN
-F 3 "" H 5650 3300 50  0001 C CNN
-F 4 "2067775" H 5050 3200 50  0001 L CNN "Farnell"
-	1    5250 3700
-	1    0    0    -1
-$EndComp
-Wire Wire Line
-	5800 3600 5800 3700
-Connection ~ 5800 3700
-Wire Wire Line
-	5800 3850 5800 3900
-Wire Wire Line
-	4850 3800 4950 3800
-Wire Wire Line
-	4850 3600 4850 3700
-Connection ~ 4850 3700
-$Comp
-L agg-kicad:CONN_01x02 J201
-U 1 1 5A6DEB31
-P 4450 3750
-F 0 "J201" V 4350 3600 50  0000 L CNN
-F 1 "CONN_01x02" V 4250 3500 50  0000 L CNN
-F 2 "" H 4450 3750 50  0001 C CNN
-F 3 "" H 4450 3750 50  0001 C CNN
-	1    4450 3750
-	1    0    0    -1
-$EndComp
-Wire Wire Line
-	4550 3600 4550 3700
-Wire Wire Line
-	4550 3850 4550 3900
-Connection ~ 4550 3700
-$Comp
-L agg-kicad:VBATT #PWR09
-U 1 1 5A6DEBBC
-P 4550 3600
-F 0 "#PWR09" H 4550 3710 50  0001 L CNN
-F 1 "VBATT" H 4550 3690 50  0000 C CNN
-F 2 "" H 4550 3600 60  0000 C CNN
-F 3 "" H 4550 3600 60  0000 C CNN
-	1    4550 3600
-	1    0    0    -1
-$EndComp
-$Comp
-L agg-kicad:GND #PWR010
-U 1 1 5A6DEBD4
-P 4550 3950
-F 0 "#PWR010" H 4420 3990 50  0001 L CNN
-F 1 "GND" H 4550 3850 50  0000 C CNN
-F 2 "" H 4550 3950 60  0000 C CNN
-F 3 "" H 4550 3950 60  0000 C CNN
-	1    4550 3950
-	1    0    0    -1
-$EndComp
-Connection ~ 4550 3900
-$Comp
-L agg-kicad:C C202
-U 1 1 5A6DEC39
-P 5800 3750
-F 0 "C202" H 5850 3820 50  0000 C CNN
-F 1 "1n" H 5850 3680 50  0000 C CNN
-F 2 "" H 5800 3750 50  0001 C CNN
-F 3 "" H 5800 3750 50  0001 C CNN
-F 4 "Value" H 5800 3750 60  0001 C CNN "Fieldname"
-	1    5800 3750
-	0    1    1    0
-$EndComp
-$Comp
-L agg-kicad:C C203
-U 1 1 5A6DEC8C
-P 6050 3750
-F 0 "C203" H 6100 3820 50  0000 C CNN
-F 1 "2u2" H 6100 3680 50  0000 C CNN
-F 2 "" H 6050 3750 50  0001 C CNN
-F 3 "" H 6050 3750 50  0001 C CNN
-F 4 "Value" H 6050 3750 60  0001 C CNN "Fieldname"
-	1    6050 3750
-	0    1    1    0
-$EndComp
-Wire Wire Line
-	6050 3700 6050 3750
-$Comp
-L agg-kicad:3v3 #PWR011
-U 1 1 5A6DECCE
-P 5800 3600
-F 0 "#PWR011" H 5800 3710 50  0001 L CNN
-F 1 "3v3" H 5800 3690 50  0000 C CNN
-F 2 "" H 5800 3600 60  0000 C CNN
-F 3 "" H 5800 3600 60  0000 C CNN
-	1    5800 3600
-	1    0    0    -1
-$EndComp
-$Comp
-L agg-kicad:GND #PWR012
-U 1 1 5A6DECEA
-P 6050 3900
-F 0 "#PWR012" H 5920 3940 50  0001 L CNN
-F 1 "GND" H 6050 3800 50  0000 C CNN
-F 2 "" H 6050 3900 60  0000 C CNN
-F 3 "" H 6050 3900 60  0000 C CNN
-	1    6050 3900
-	1    0    0    -1
-$EndComp
-Wire Wire Line
-	6050 3900 6050 3850
-$Comp
-L agg-kicad:C C201
-U 1 1 5A6DED5C
-P 4700 3750
-F 0 "C201" H 4750 3820 50  0000 C CNN
-F 1 "2u2" H 4750 3680 50  0000 C CNN
-F 2 "" H 4700 3750 50  0001 C CNN
-F 3 "" H 4700 3750 50  0001 C CNN
-F 4 "Value" H 4700 3750 60  0001 C CNN "Fieldname"
-	1    4700 3750
-	0    1    1    0
-$EndComp
-Wire Wire Line
-	4700 3850 4700 3900
-Connection ~ 4700 3900
-Wire Wire Line
-	4700 3750 4700 3700
-Connection ~ 4700 3700
-Wire Wire Line
-	4550 3900 4700 3900
-Wire Wire Line
-	4550 3700 4700 3700
-Wire Wire Line
-	5650 3600 5650 3700
-Connection ~ 5650 3700
-Wire Wire Line
-	5650 3800 5550 3800
-Wire Wire Line
-	5550 3600 5650 3600
-Wire Wire Line
-	5550 3700 5650 3700
-Wire Wire Line
-	5800 3900 5550 3900
-Wire Wire Line
-	4950 3600 4850 3600
-Wire Wire Line
-	5800 3700 5800 3750
-Wire Wire Line
-	5800 3700 6050 3700
-Wire Wire Line
-	4850 3700 4850 3800
-Wire Wire Line
-	4850 3700 4950 3700
-Wire Wire Line
-	4550 3700 4550 3750
-Wire Wire Line
-	4550 3900 4550 3950
-Wire Wire Line
-	4700 3900 4950 3900
-Wire Wire Line
-	4700 3700 4850 3700
-Wire Wire Line
-	5650 3700 5650 3800
-Wire Wire Line
-	5650 3700 5800 3700
 $EndSCHEMATC

Commit message: Add TPS61025 switching regulator to schematic
Parts:
- added C?: 10uF, agg:0402, symbol agg-kicad:C
- added C?: 100nF, agg:0402, symbol agg-kicad:C
- added C?: 2.2uF, agg:0402, symbol agg-kicad:C
- added C?: 100uF, Jerboa:avx_2312, symbol agg-kicad:CP
- added J? (x2): CONN_01x02, agg:SIL-254P-02, symbol agg-kicad:CONN_01x02
- added L?: 6.8uH, Jerboa:wurth_7447789006, symbol agg-kicad:L
- added R?: 604k, agg:0402, symbol agg-kicad:R
- added R?: 499k, agg:0402, symbol agg-kicad:R
- added R?: 1M, agg:0402, symbol agg-kicad:R
- added U?: TPS61025DRCR, Jerboa:VSON-10, symbol TPS6102x:TPS6102x
Connections:
- new net: C?.1, C?.1, J?.1, L?.1, R?.1, U?.1 (EN), U?.6 (VBAT)
- new net: L?.2, U?.9 (SW)
- new net: R?.1, R?.2, U?.7 (LBI)
- new net: R?.2, U?.4 (LBO)
- new net 3v3: C?.1, C?.2, R?.1, U?.2 (VOUT)
- new net GND: C?.1, C?.2, C?.2, C?.2, J?.2, J?.2, R?.2, U?.10 (PGND), U?.5 (GND), U?.8 (PS), U?.PAD (PowerPAD)
- new net solar_cells: J?.1
- no-connect marks 0 -> 1
Other:
- note added: "Analog in from solar cells"
- note added: "Battery/capacitor input"

Commit message: Draft a PCB for the battery breakout board
Connections:
- net LOW_BATT_WARNING: now reaches R?.2, U?.4 (LBO)
Changed lines of the file:
@@
 	1    0    0    -1
 $EndComp
+Text HLabel 7250 4000 2    50   Input ~ 0
+LOW_BATT_WARNING
+Wire Wire Line
+	7250 4000 7100 4000
+Connection ~ 7100 4000
 $EndSCHEMATC

Commit message: Create some more schematic symbols and footprints
Changed lines of the file:
@@
 $EndComp
 Wire Wire Line
-	5250 3400 5150 3400
+	4000 3400 5250 3400
 Text Notes 2900 3450 0    50   ~ 0
 Battery/capacitor input
@@
 Connection ~ 4150 3400
 Wire Wire Line
-	4150 3400 4000 3400
-Wire Wire Line
 	4600 3450 4600 3400
 Connection ~ 4600 3400
-Wire Wire Line
-	4600 3400 4500 3400
 $Comp
 L agg-kicad:L L?
@@
 	5250 3800 4900 3800
 Wire Wire Line
-	4900 3800 4900 3700
+	4900 3700 4900 3900
 Connection ~ 4900 3800
 Wire Wire Line
 	4900 3600 4900 3400
-Wire Wire Line
-	4600 3400 4900 3400
 Connection ~ 4900 3400
-Wire Wire Line
-	4900 3400 5150 3400
-Wire Wire Line
-	4900 3800 4900 3900
 $Comp
 L agg-kicad:GND #PWR?
@@
 $EndComp
 Wire Wire Line
-	5250 4200 5150 4200
+	5050 4200 5250 4200
 Wire Wire Line
 	5250 4100 5150 4100
@@
 	5150 4100 5150 4200
 Wire Wire Line
-	4000 3500 4000 3600
-Wire Wire Line
-	4000 3600 4150 3600
+	4000 3500 4000 3650
+Wire Wire Line
+	4000 3600 4600 3600
 Wire Wire Line
 	4600 3600 4600 3550
@@
 	4150 3550 4150 3600
 Connection ~ 4150 3600
-Wire Wire Line
-	4000 3650 4000 3600
 Connection ~ 4000 3600
 Wire Wire Line
@@
 $EndComp
 Wire Wire Line
-	6350 4200 6450 4200
+	6350 4200 6550 4200
 Wire Wire Line
 	6450 4200 6450 4100
@@
 $EndComp
 Wire Wire Line
-	6800 3550 6800 3500
+	6800 3500 6800 3600
 Connection ~ 6800 3550
-Wire Wire Line
-	6800 3550 6800 3600
 Wire Wire Line
 	6800 3400 6800 3300
@@
 	7100 3600 7100 3300
 Wire Wire Line
-	6800 3300 7100 3300
+	6350 3300 7200 3300
 Connection ~ 7100 3300
 Wire Wire Line
-	7100 3300 7200 3300
-Wire Wire Line
 	7100 3700 7100 4000
 Wire Wire Line
-	7100 4000 6350 4000
+	6350 4000 7250 4000
 Wire Wire Line
 	6550 4250 6550 4200
-Wire Wire Line
-	6550 4200 6450 4200
 Connection ~ 6450 4200
 Wire Wire Line
 	5050 4250 5050 4200
-Wire Wire Line
-	5050 4200 5150 4200
 Connection ~ 5150 4200
-Wire Wire Line
-	4150 3400 4500 3400
 Connection ~ 4500 3400
-Wire Wire Line
-	4150 3600 4600 3600
 $Comp
 L TPS6102x:TPS6102x U?
@@
 Wire Wire Line
 	6450 3400 6450 3300
-Wire Wire Line
-	6350 3300 6450 3300
 Connection ~ 6450 3300
-Wire Wire Line
-	6450 3300 6800 3300
 Wire Wire Line
 	6450 3500 6450 3550
@@
 Text HLabel 7250 4000 2    50   Input ~ 0
 LOW_BATT_WARNING
-Wire Wire Line
-	7250 4000 7100 4000
 Connection ~ 7100 4000
 $EndSCHEMATC
