File: pcb/power.sch (KiCad schematic (older format))
At the start: 11 parts

Commit message: WIP: create and add componenents for the micrf rtty radio, also do some work on schematic
Changed lines of the file:
@@
 $Descr A4 11693 8268
 encoding utf-8
-Sheet 1 4
+Sheet 2 4
 Title ""
 Date ""
@@
 $EndComp
 Wire Wire Line
-	4000 3400 5250 3400
+	4000 3400 4150 3400
 Text Notes 2900 3450 0    50   ~ 0
 Battery/capacitor input
@@
 	5250 3800 4900 3800
 Wire Wire Line
-	4900 3700 4900 3900
+	4900 3700 4900 3800
 Connection ~ 4900 3800
 Wire Wire Line
@@
 $EndComp
 Wire Wire Line
-	5050 4200 5250 4200
+	5050 4200 5150 4200
 Wire Wire Line
 	5250 4100 5150 4100
@@
 	5150 4100 5150 4200
 Wire Wire Line
-	4000 3500 4000 3650
-Wire Wire Line
-	4000 3600 4600 3600
+	4000 3500 4000 3600
+Wire Wire Line
+	4000 3600 4150 3600
 Wire Wire Line
 	4600 3600 4600 3550
@@
 $EndComp
 Wire Wire Line
-	6350 4200 6550 4200
+	6350 4200 6450 4200
 Wire Wire Line
 	6450 4200 6450 4100
@@
 $EndComp
 Wire Wire Line
-	6800 3500 6800 3600
+	6800 3500 6800 3550
 Connection ~ 6800 3550
 Wire Wire Line
@@
 	7100 3600 7100 3300
 Wire Wire Line
-	6350 3300 7200 3300
+	6350 3300 6450 3300
 Connection ~ 7100 3300
 Wire Wire Line
 	7100 3700 7100 4000
 Wire Wire Line
-	6350 4000 7250 4000
+	6350 4000 7100 4000
 Wire Wire Line
 	6550 4250 6550 4200
@@
 LOW_BATT_WARNING
 Connection ~ 7100 4000
+Wire Wire Line
+	4150 3400 4500 3400
+Wire Wire Line
+	4600 3400 4900 3400
+Wire Wire Line
+	5150 3400 5250 3400
+Wire Wire Line
+	4900 3800 4900 3900
+Wire Wire Line
+	4900 3400 5150 3400
+Wire Wire Line
+	4150 3600 4600 3600
+Wire Wire Line
+	4000 3600 4000 3650
+Wire Wire Line
+	6800 3550 6800 3600
+Wire Wire Line
+	6800 3300 7100 3300
+Wire Wire Line
+	7100 3300 7200 3300
+Wire Wire Line
+	6450 4200 6550 4200
+Wire Wire Line
+	5150 4200 5250 4200
+Wire Wire Line
+	4500 3400 4600 3400
+Wire Wire Line
+	6450 3300 6800 3300
+Wire Wire Line
+	7100 4000 7250 4000
 $EndSCHEMATC

Commit message: Finish schematic, generate first BOM
Parts:
- C13: renamed from C?; Farnell 1288282 -> 2533923
- R11: renamed from R?; Farnell 1469723 -> 2059189
- gave numbers to parts that had none: 9
Connections:
- wire segments 52 -> 54
Changed lines of the file:
@@
 $EndDescr
 $Comp
-L agg-kicad:CONN_01x02 J?
+L agg-kicad:CONN_01x02 J3
 U 1 1 5A722F1A
 P 3900 3400
-F 0 "J?" H 3931 3615 50  0000 C CNN
-F 1 "CONN_01x02" H 3931 3524 50  0000 C CNN
+F 0 "J3" H 3800 3600 50  0000 C CNN
+F 1 "CONN_01x02" H 3700 3500 50  0000 C CNN
 F 2 "agg:SIL-254P-02" H 3900 3400 50  0001 C CNN
 F 3 "http://www.farnell.com/datasheets/2290158.pdf" H 3900 3400 50  0001 C CNN
@@
 Analog in from solar cells
 $Comp
-L agg-kicad:GND #PWR?
+L agg-kicad:GND #PWR023
 U 1 1 5A72304B
 P 4100 4300
-F 0 "#PWR?" H 3970 4340 50  0001 L CNN
+F 0 "#PWR023" H 3970 4340 50  0001 L CNN
 F 1 "GND" H 4100 4200 50  0000 C CNN
 F 2 "" H 4100 4300 50  0001 C CNN
@@
 	4100 4100 4000 4100
 $Comp
-L agg-kicad:GND #PWR?
+L agg-kicad:GND #PWR022
 U 1 1 5A7230D2
 P 4000 3650
-F 0 "#PWR?" H 3870 3690 50  0001 L CNN
-F 1 "GND" H 4000 3550 50  0000 C CNN
+F 0 "#PWR022" H 3870 3690 50  0001 L CNN
+F 1 "GND" H 3900 3650 50  0000 C CNN
 F 2 "" H 4000 3650 50  0001 C CNN
 F 3 "" H 4000 3650 50  0001 C CNN
@@
 $EndComp
 Wire Wire Line
-	4000 3400 4150 3400
+	4000 3400 4050 3400
 Text Notes 2900 3450 0    50   ~ 0
 Battery/capacitor input
 $Comp
-L agg-kicad:C C?
+L agg-kicad:C C12
 U 1 1 5A72323C
 P 4150 3450
-F 0 "C?" V 4154 3508 50  0000 L CNN
+F 0 "C12" V 4154 3508 50  0000 L CNN
 F 1 "10uF" V 4245 3508 50  0000 L CNN
 F 2 "agg:0402" H 4150 3450 50  0001 C CNN
@@
 $EndComp
 $Comp
-L agg-kicad:C C?
+L agg-kicad:C C13
 U 1 1 5A7232C1
 P 4600 3450
-F 0 "C?" V 4604 3508 50  0000 L CNN
+F 0 "C13" V 4604 3508 50  0000 L CNN
 F 1 "100nF" V 4695 3508 50  0000 L CNN
 F 2 "agg:0402" H 4600 3450 50  0001 C CNN
 F 3 "" H 4600 3450 50  0001 C CNN
-F 4 "1288282" H 4600 3450 50  0001 C CNN "Farnell"
+F 4 "2533923" H 4600 3450 50  0001 C CNN "Farnell"
 	1    4600 3450
 	0    1    1    0
@@
 Connection ~ 4600 3400
 $Comp
-L agg-kicad:L L?
+L agg-kicad:L L1
 U 1 1 5A72334A
 P 4700 3300
-F 0 "L?" H 4750 3478 50  0000 C CNN
+F 0 "L1" H 4750 3478 50  0000 C CNN
 F 1 "6.8uH" H 4750 3387 50  0000 C CNN
 F 2 "Jerboa:wurth_7447789006" H 4700 3300 50  0001 C CNN
@@
 Connection ~ 5150 3400
 $Comp
-L agg-kicad:R R?
+L agg-kicad:R R10
 U 1 1 5A72341A
 P 4900 3600
-F 0 "R?" V 4904 3641 50  0000 L CNN
+F 0 "R10" V 4904 3641 50  0000 L CNN
 F 1 "604k" V 4995 3641 50  0000 L CNN
 F 2 "agg:0402" H 4900 3600 50  0001 C CNN
@@
 $EndComp
 $Comp
-L agg-kicad:R R?
+L agg-kicad:R R11
 U 1 1 5A7234B5
 P 4900 3900
-F 0 "R?" V 4904 3941 50  0000 L CNN
+F 0 "R11" V 4904 3941 50  0000 L CNN
 F 1 "499k" V 4995 3941 50  0000 L CNN
 F 2 "agg:0402" H 4900 3900 50  0001 C CNN
 F 3 "" H 4900 3900 50  0001 C CNN
-F 4 "1469723" H 4900 3900 50  0001 C CNN "Farnell"
+F 4 "2059189" H 4900 3900 50  0001 C CNN "Farnell"
 	1    4900 3900
 	0    1    1    0
@@
 Connection ~ 4900 3400
 $Comp
-L agg-kicad:GND #PWR?
+L agg-kicad:GND #PWR024
 U 1 1 5A7237FD
 P 4900 4050
-F 0 "#PWR?" H 4770 4090 50  0001 L CNN
+F 0 "#PWR024" H 4770 4090 50  0001 L CNN
 F 1 "GND" H 4900 3950 50  0000 C CNN
 F 2 "" H 4900 4050 50  0001 C CNN
@@
 	4900 4000 4900 4050
 $Comp
-L agg-kicad:GND #PWR?
+L agg-kicad:GND #PWR025
 U 1 1 5A723902
 P 5050 4250
-F 0 "#PWR?" H 4920 4290 50  0001 L CNN
+F 0 "#PWR025" H 4920 4290 50  0001 L CNN
 F 1 "GND" H 5050 4150 50  0000 C CNN
 F 2 "" H 5050 4250 50  0001 C CNN
@@
 	4000 3500 4000 3600
 Wire Wire Line
-	4000 3600 4150 3600
+	4000 3600 4050 3600
 Wire Wire Line
 	4600 3600 4600 3550
@@
 	4800 3300 5250 3300
 $Comp
-L agg-kicad:GND #PWR?
+L agg-kicad:GND #PWR026
 U 1 1 5A724A2A
 P 6550 4250
-F 0 "#PWR?" H 6420 4290 50  0001 L CNN
+F 0 "#PWR026" H 6420 4290 50  0001 L CNN
 F 1 "GND" H 6550 4150 50  0000 C CNN
 F 2 "" H 6550 4250 50  0001 C CNN
@@
 	6450 4100 6350 4100
 $Comp
-L agg-kicad:R R?
+L agg-kicad:R R12
 U 1 1 5A725405
 P 7100 3600
-F 0 "R?" V 7104 3641 50  0000 L CNN
+F 0 "R12" V 7104 3641 50  0000 L CNN
 F 1 "1M" V 7195 3641 50  0000 L CNN
 F 2 "agg:0402" H 7100 3600 50  0001 C CNN
@@
 NoConn ~ 6350 3650
 $Comp
-L agg-kicad:C C?
+L agg-kicad:C C14
 U 1 1 5A725A05
 P 6450 3400
-F 0 "C?" V 6454 3458 50  0000 L CNN
+F 0 "C14" V 6454 3458 50  0000 L CNN
 F 1 "2.2uF" V 6545 3458 50  0000 L CNN
 F 2 "agg:0402" H 6450 3400 50  0001 C CNN
@@
 $EndComp
 $Comp
-L agg-kicad:3v3 #PWR?
+L agg-kicad:3v3 #PWR028
 U 1 1 5A725B18
 P 7200 3250
-F 0 "#PWR?" H 7200 3360 50  0001 L CNN
+F 0 "#PWR028" H 7200 3360 50  0001 L CNN
 F 1 "3v3" H 7200 3374 50  0000 C CNN
 F 2 "" H 7200 3250 50  0001 C CNN
@@
 	7200 3300 7200 3250
 $Comp
-L agg-kicad:GND #PWR?
+L agg-kicad:GND #PWR027
 U 1 1 5A72606D
 P 6800 3600
-F 0 "#PWR?" H 6670 3640 50  0001 L CNN
+F 0 "#PWR027" H 6670 3640 50  0001 L CNN
 F 1 "GND" H 6800 3500 50  0000 C CNN
 F 2 "" H 6800 3600 50  0001 C CNN
@@
 Connection ~ 4500 3400
 $Comp
-L TPS6102x:TPS6102x U?
+L TPS6102x:TPS6102x U2
 U 1 1 5A724BBB
 P 5800 3750
-F 0 "U?" H 5800 4425 50  0000 C CNN
+F 0 "U2" H 5800 4425 50  0000 C CNN
 F 1 "TPS61025DRCR" H 5800 4334 50  0000 C CNN
 F 2 "Jerboa:VSON-10" H 5800 3000 50  0001 C CNN
@@
 $EndComp
 $Comp
-L agg-kicad:CP C?
+L agg-kicad:CP C15
 U 1 1 5A72677F
 P 6800 3500
-F 0 "C?" V 6896 3442 50  0000 R CNN
+F 0 "C15" V 6896 3442 50  0000 R CNN
 F 1 "100uF" V 6805 3442 50  0000 R CNN
 F 2 "Jerboa:avx_2312" H 6800 3500 50  0001 C CNN
@@
 	6450 3550 6800 3550
 $Comp
-L agg-kicad:CONN_01x02 J?
+L agg-kicad:CONN_01x02 J4
 U 1 1 5A7274B5
 P 3900 4100
-F 0 "J?" H 3931 4315 50  0000 C CNN
+F 0 "J4" H 3931 4315 50  0000 C CNN
 F 1 "CONN_01x02" H 3931 4224 50  0000 C CNN
 F 2 "agg:SIL-254P-02" H 3900 4100 50  0001 C CNN
@@
 Wire Wire Line
 	7100 4000 7250 4000
+$Comp
+L agg-kicad:PWR #FLG0102
+U 1 1 5B50ADD5
+P 4050 3400
+F 0 "#FLG0102" H 4050 3560 50  0001 C CNN
+F 1 "PWR" H 4050 3534 50  0000 C CNN
+F 2 "" H 4050 3400 50  0001 C CNN
+F 3 "" H 4050 3400 50  0001 C CNN
+	1    4050 3400
+	1    0    0    -1
+$EndComp
+Connection ~ 4050 3400
+Wire Wire Line
+	4050 3400 4150 3400
+$Comp
+L agg-kicad:PWR #FLG0103
+U 1 1 5B50ADFF
+P 4050 3600
+F 0 "#FLG0103" H 4050 3760 50  0001 C CNN
+F 1 "PWR" H 4100 3550 50  0000 C CNN
+F 2 "" H 4050 3600 50  0001 C CNN
+F 3 "" H 4050 3600 50  0001 C CNN
+	1    4050 3600
+	1    0    0    -1
+$EndComp
+Connection ~ 4050 3600
+Wire Wire Line
+	4050 3600 4150 3600
 $EndSCHEMATC
