File: pcb/power.sch (KiCad schematic (older format))
At the start: 11 parts, among them J3 CONN_01x02, J4 CONN_01x02, U2 TPS61025DRCR

Commit message: Schematic (and some pcb) using si4460 for both 144MHz and 434MHz
Parts:
- removed R10: 604k, agg:0402, symbol agg-kicad:R
- removed R11: 499k, agg:0402, symbol agg-kicad:R
- removed R12: 1M, agg:0402, symbol agg-kicad:R
Connections:
- net labels added: BATT_V
- net labels removed: LOW_BATT_WARNING
- wire segments 54 -> 44
- no-connect marks 1 -> 2
Changed lines of the file:
@@
 EESchema Schematic File Version 4
-LIBS:jerboa-cache
 EELAYER 26 0
 EELAYER END
@@
 Text Notes 2800 4150 0    50   ~ 0
 Analog in from solar cells
-$Comp
-L agg-kicad:GND #PWR0122
-U 1 1 5A72304B
-P 4100 4300
-F 0 "#PWR0122" H 3970 4340 50  0001 L CNN
-F 1 "GND" H 4100 4200 50  0000 C CNN
-F 2 "" H 4100 4300 50  0001 C CNN
-F 3 "" H 4100 4300 50  0001 C CNN
-	1    4100 4300
-	1    0    0    -1
-$EndComp
 Wire Wire Line
 	4000 4200 4100 4200
-Wire Wire Line
-	4100 4200 4100 4300
 Text HLabel 4100 4100 2    50   Input ~ 0
 solar_cells
@@
 	4100 4100 4000 4100
 $Comp
-L agg-kicad:GND #PWR0123
+L agg-kicad:GND #PWR023
 U 1 1 5A7230D2
 P 4000 3650
-F 0 "#PWR0123" H 3870 3690 50  0001 L CNN
+F 0 "#PWR023" H 3870 3690 50  0001 L CNN
 F 1 "GND" H 3900 3650 50  0000 C CNN
 F 2 "" H 4000 3650 50  0001 C CNN
@@
 Connection ~ 5150 3400
 $Comp
-L agg-kicad:R R10
-U 1 1 5A72341A
-P 4900 3600
-F 0 "R10" V 4904 3641 50  0000 L CNN
-F 1 "604k" V 4995 3641 50  0000 L CNN
-F 2 "agg:0402" H 4900 3600 50  0001 C CNN
-F 3 "" H 4900 3600 50  0001 C CNN
-F 4 "2073163" H 4900 3600 50  0001 C CNN "Farnell"
-	1    4900 3600
-	0    1    1    0
-$EndComp
-$Comp
-L agg-kicad:R R11
-U 1 1 5A7234B5
-P 4900 3900
-F 0 "R11" V 4904 3941 50  0000 L CNN
-F 1 "499k" V 4995 3941 50  0000 L CNN
-F 2 "agg:0402" H 4900 3900 50  0001 C CNN
-F 3 "" H 4900 3900 50  0001 C CNN
-F 4 "2059189" H 4900 3900 50  0001 C CNN "Farnell"
-	1    4900 3900
-	0    1    1    0
-$EndComp
-Wire Wire Line
-	5250 3800 4900 3800
-Wire Wire Line
-	4900 3700 4900 3800
-Connection ~ 4900 3800
-Wire Wire Line
-	4900 3600 4900 3400
-Connection ~ 4900 3400
-$Comp
-L agg-kicad:GND #PWR0124
+L agg-kicad:GND #PWR025
 U 1 1 5A7237FD
-P 4900 4050
-F 0 "#PWR0124" H 4770 4090 50  0001 L CNN
-F 1 "GND" H 4900 3950 50  0000 C CNN
-F 2 "" H 4900 4050 50  0001 C CNN
-F 3 "" H 4900 4050 50  0001 C CNN
-	1    4900 4050
-	1    0    0    -1
-$EndComp
-Wire Wire Line
-	4900 4000 4900 4050
-$Comp
-L agg-kicad:GND #PWR0125
+P 5200 3850
+F 0 "#PWR025" H 5070 3890 50  0001 L CNN
+F 1 "GND" H 5200 3750 50  0000 C CNN
+F 2 "" H 5200 3850 50  0001 C CNN
+F 3 "" H 5200 3850 50  0001 C CNN
+	1    5200 3850
+	1    0    0    -1
+$EndComp
+$Comp
+L agg-kicad:GND #PWR024
 U 1 1 5A723902
 P 5050 4250
-F 0 "#PWR0125" H 4920 4290 50  0001 L CNN
+F 0 "#PWR024" H 4920 4290 50  0001 L CNN
 F 1 "GND" H 5050 4150 50  0000 C CNN
 F 2 "" H 5050 4250 50  0001 C CNN
@@
 	4800 3300 5250 3300
 $Comp
-L agg-kicad:GND #PWR0126
+L agg-kicad:GND #PWR026
 U 1 1 5A724A2A
 P 6550 4250
-F 0 "#PWR0126" H 6420 4290 50  0001 L CNN
+F 0 "#PWR026" H 6420 4290 50  0001 L CNN
 F 1 "GND" H 6550 4150 50  0000 C CNN
 F 2 "" H 6550 4250 50  0001 C CNN
@@
 Wire Wire Line
 	6450 4100 6350 4100
-$Comp
-L agg-kicad:R R12
-U 1 1 5A725405
-P 7100 3600
-F 0 "R12" V 7104 3641 50  0000 L CNN
-F 1 "1M" V 7195 3641 50  0000 L CNN
-F 2 "agg:0402" H 7100 3600 50  0001 C CNN
-F 3 "" H 7100 3600 50  0001 C CNN
-F 4 "2447127" H 7100 3600 50  0001 C CNN "Farnell"
-	1    7100 3600
-	0    1    1    0
-$EndComp
 NoConn ~ 6350 3650
 $Comp
@@
 $EndComp
 $Comp
-L agg-kicad:3v3 #PWR0127
+L agg-kicad:3v3 #PWR028
 U 1 1 5A725B18
 P 7200 3250
-F 0 "#PWR0127" H 7200 3360 50  0001 L CNN
+F 0 "#PWR028" H 7200 3360 50  0001 L CNN
 F 1 "3v3" H 7200 3374 50  0000 C CNN
 F 2 "" H 7200 3250 50  0001 C CNN
@@
 	7200 3300 7200 3250
 $Comp
-L agg-kicad:GND #PWR0128
+L agg-kicad:GND #PWR027
 U 1 1 5A72606D
 P 6800 3600
-F 0 "#PWR0128" H 6670 3640 50  0001 L CNN
+F 0 "#PWR027" H 6670 3640 50  0001 L CNN
 F 1 "GND" H 6800 3500 50  0000 C CNN
 F 2 "" H 6800 3600 50  0001 C CNN
@@
 Connection ~ 6800 3300
 Wire Wire Line
-	7100 3600 7100 3300
-Wire Wire Line
 	6350 3300 6450 3300
-Connection ~ 7100 3300
-Wire Wire Line
-	7100 3700 7100 4000
-Wire Wire Line
-	6350 4000 7100 4000
 Wire Wire Line
 	6550 4250 6550 4200
@@
 	1    0    0    -1
 $EndComp
-Text HLabel 7250 4000 2    50   Input ~ 0
-LOW_BATT_WARNING
-Connection ~ 7100 4000
 Wire Wire Line
 	4150 3400 4500 3400
 Wire Wire Line
-	4600 3400 4900 3400
-Wire Wire Line
 	5150 3400 5250 3400
 Wire Wire Line
-	4900 3800 4900 3900
-Wire Wire Line
-	4900 3400 5150 3400
-Wire Wire Line
 	4150 3600 4600 3600
 Wire Wire Line
@@
 	6800 3550 6800 3600
 Wire Wire Line
-	6800 3300 7100 3300
-Wire Wire Line
-	7100 3300 7200 3300
-Wire Wire Line
 	6450 4200 6550 4200
 Wire Wire Line
@@
 Wire Wire Line
 	6450 3300 6800 3300
-Wire Wire Line
-	7100 4000 7250 4000
-$Comp
-L agg-kicad:PWR #FLG0102
+$Comp
+L agg-kicad:PWR #FLG02
 U 1 1 5B50ADD5
 P 4050 3400
-F 0 "#FLG0102" H 4050 3560 50  0001 C CNN
+F 0 "#FLG02" H 4050 3560 50  0001 C CNN
 F 1 "PWR" H 4050 3534 50  0000 C CNN
 F 2 "" H 4050 3400 50  0001 C CNN
@@
 	4050 3400 4150 3400
 $Comp
-L agg-kicad:PWR #FLG0103
+L agg-kicad:PWR #FLG03
 U 1 1 5B50ADFF
 P 4050 3600
-F 0 "#FLG0103" H 4050 3760 50  0001 C CNN
+F 0 "#FLG03" H 4050 3760 50  0001 C CNN
 F 1 "PWR" H 4100 3550 50  0000 C CNN
 F 2 "" H 4050 3600 50  0001 C CNN
@@
 Wire Wire Line
 	4050 3600 4150 3600
+Wire Wire Line
+	4600 3400 5150 3400
+Wire Wire Line
+	5250 3800 5200 3800
+Wire Wire Line
+	5200 3800 5200 3850
+Text HLabel 4100 4200 2    50   Input ~ 0
+BATT_V
+Wire Wire Line
+	6800 3300 7200 3300
+NoConn ~ 6350 4000
 $EndSCHEMATC

Commit message: WIP: Begin making schematic changes - replace boost regulator with ADP1607 and add load switch for radio power
Parts:
- removed C13: 100nF, agg:0402, symbol agg-kicad:C
- removed C14: 2.2uF, agg:0402, symbol agg-kicad:C
- removed C15: 100uF, Jerboa:avx_2312, symbol agg-kicad:CP
- removed L1: 6.8uH, Jerboa:wurth_7447789006, symbol agg-kicad:L
- removed U2: TPS61025DRCR, Jerboa:VSON-10, symbol TPS6102x:TPS6102x
- added C?: 10uF, agg:0402, symbol agg-kicad:C
- added C?: 470pF, agg:0402, symbol agg-kicad:C
- added IC?: ADP1607, Jerboa:LFCSP-2x2, symbol adp1607:ADP1607
- added L?: 2.2uH, Jerboa:0806, symbol agg-kicad:L
- added R?: 953k, agg:0402, symbol agg-kicad:R
- added R?: 620k, agg:0402, symbol agg-kicad:R
- added R?: 470k, agg:0402, symbol agg-kicad:R
- added R?: 4k7, agg:0402, symbol agg-kicad:R
- added U?: FDC6329L, Jerboa:SuperSOT-6, symbol FDC6329L:FDC6329L
Connections:
- net labels added: 3v3_switched, RADIO_PWR_EN
- wire segments 44 -> 53
- no-connect marks 2 -> 0
Other:
- note added: "Boost Regulator"
- note added: "Radio Power Load Switch"
- moved on the sheet: C12, J3, J4

Commit message: Finish redoing clock circuitry
Parts:
- added C? (x2): 1uF, agg:0402, symbol agg-kicad:C
- added U?: NCP4620, agg:SC-70-5, symbol ncp4620:NCP4620
Connections:
- net labels added: 1v8
- wire segments 53 -> 63
Other:
- note added: "1V8 Regulator"
- moved on the sheet: C?, R?, U?

Commit message: Begin routing pcb (again)
Parts:
- gave numbers to parts that had none: 12
Connections:
- wire segments 63 -> 64
Changed lines of the file:
@@
 Connection ~ 2150 1300
 Wire Wire Line
-	2000 1400 2000 1500
-Wire Wire Line
-	2000 1500 2050 1500
-Wire Wire Line
 	2150 1450 2150 1500
-Connection ~ 2000 1500
 $Comp
 L agg-kicad:3v3 #PWR028
@@
 Wire Wire Line
 	2150 1300 2450 1300
-Wire Wire Line
-	2000 1500 2000 1550
 $Comp
 L agg-kicad:PWR #FLG02
@@
 Wire Wire Line
 	2050 1300 2150 1300
-$Comp
-L agg-kicad:PWR #FLG03
-U 1 1 5B50ADFF
-P 2050 1500
-F 0 "#FLG03" H 2050 1660 50  0001 C CNN
-F 1 "PWR" H 2100 1450 50  0000 C CNN
-F 2 "" H 2050 1500 50  0001 C CNN
-F 3 "" H 2050 1500 50  0001 C CNN
-	1    2050 1500
-	1    0    0    -1
-$EndComp
-Connection ~ 2050 1500
-Wire Wire Line
-	2050 1500 2150 1500
 Text HLabel 1900 2750 2    50   Input ~ 0
 BATT_V
 $Comp
-L adp1607:ADP1607 IC?
+L adp1607:ADP1607 IC1
 U 1 1 5B42BBE5
 P 2900 1500
-F 0 "IC?" H 2900 1925 50  0000 C CNN
+F 0 "IC1" H 2900 1925 50  0000 C CNN
 F 1 "ADP1607" H 2900 1834 50  0000 C CNN
 F 2 "Jerboa:LFCSP-2x2" H 2600 1100 50  0001 L CNN
@@
 $EndComp
 $Comp
-L agg-kicad:L L?
+L agg-kicad:L L1
 U 1 1 5B42BF34
 P 2850 950
-F 0 "L?" H 2900 1128 50  0000 C CNN
+F 0 "L1" H 2900 1128 50  0000 C CNN
 F 1 "2.2uH" H 2900 1037 50  0000 C CNN
 F 2 "Jerboa:0806" H 2850 950 50  0001 C CNN
@@
 $EndComp
 $Comp
-L agg-kicad:R R?
+L agg-kicad:R R1
 U 1 1 5B42C0C7
 P 3500 1450
-F 0 "R?" V 3504 1491 50  0000 L CNN
+F 0 "R1" V 3504 1491 50  0000 L CNN
 F 1 "953k" V 3595 1491 50  0000 L CNN
 F 2 "agg:0402" H 3500 1450 50  0001 C CNN
@@
 $EndComp
 $Comp
-L agg-kicad:R R?
+L agg-kicad:R R2
 U 1 1 5B42C17D
 P 3500 1650
-F 0 "R?" V 3504 1691 50  0000 L CNN
+F 0 "R2" V 3504 1691 50  0000 L CNN
 F 1 "620k" V 3595 1691 50  0000 L CNN
 F 2 "agg:0402" H 3500 1650 50  0001 C CNN
@@
 $EndComp
 $Comp
-L agg-kicad:GND #PWR?
+L agg-kicad:GND #PWR0103
 U 1 1 5B42C1C1
 P 3500 1800
-F 0 "#PWR?" H 3370 1840 50  0001 L CNN
+F 0 "#PWR0103" H 3370 1840 50  0001 L CNN
 F 1 "GND" H 3500 1700 50  0000 C CNN
 F 2 "" H 3500 1800 50  0001 C CNN
@@
 $EndComp
 $Comp
-L agg-kicad:GND #PWR?
+L agg-kicad:GND #PWR0105
 U 1 1 5B42C212
 P 2450 1750
-F 0 "#PWR?" H 2320 1790 50  0001 L CNN
+F 0 "#PWR0105" H 2320 1790 50  0001 L CNN
 F 1 "GND" H 2450 1650 50  0000 C CNN
 F 2 "" H 2450 1750 50  0001 C CNN
@@
 	2450 950  2450 1300
 $Comp
-L agg-kicad:C C?
+L agg-kicad:C C1
 U 1 1 5B4322AF
 P 3900 1500
-F 0 "C?" V 3904 1558 50  0000 L CNN
+F 0 "C1" V 3904 1558 50  0000 L CNN
 F 1 "10uF" V 3995 1558 50  0000 L CNN
 F 2 "agg:0402" H 3900 1500 50  0001 C CNN
@@
 $EndComp
 $Comp
-L agg-kicad:GND #PWR?
+L agg-kicad:GND #PWR0106
 U 1 1 5B432308
 P 3900 1650
-F 0 "#PWR?" H 3770 1690 50  0001 L CNN
+F 0 "#PWR0106" H 3770 1690 50  0001 L CNN
 F 1 "GND" H 3900 1550 50  0000 C CNN
 F 2 "" H 3900 1650 50  0001 C CNN
@@
 	3900 1400 4200 1400
 $Comp
-L 3v3_switched:3v3_switched #PWR?
+L 3v3_switched:3v3_switched #PWR0107
 U 1 1 5B443E8C
 P 7200 1150
-F 0 "#PWR?" H 7200 1260 50  0001 L CNN
+F 0 "#PWR0107" H 7200 1260 50  0001 L CNN
 F 1 "3v3_switched" H 7200 1274 50  0000 C CNN
 F 2 "" H 7200 1150 50  0001 C CNN
@@
 $EndComp
 $Comp
-L FDC6329L:FDC6329L U?
+L FDC6329L:FDC6329L U2
 U 1 1 5B444992
 P 6300 1300
-F 0 "U?" H 6300 1647 60  0000 C CNN
+F 0 "U2" H 6300 1647 60  0000 C CNN
 F 1 "FDC6329L" H 6300 1541 60  0000 C CNN
 F 2 "Jerboa:SuperSOT-6" H 6300 650 60  0001 C CNN
@@
 	7200 1200 7200 1150
 $Comp
-L agg-kicad:R R?
+L agg-kicad:R R3
 U 1 1 5B44548F
 P 5500 1300
-F 0 "R?" V 5504 1341 50  0000 L CNN
+F 0 "R3" V 5504 1341 50  0000 L CNN
 F 1 "470k" V 5595 1341 50  0000 L CNN
 F 2 "agg:0402" H 5500 1300 50  0001 C CNN
@@
 	5500 1650 5650 1650
 $Comp
-L agg-kicad:R R?
+L agg-kicad:R R4
 U 1 1 5B45A92C
 P 7050 1750
-F 0 "R?" V 7054 1791 50  0000 L CNN
+F 0 "R4" V 7054 1791 50  0000 L CNN
 F 1 "4k7" V 7145 1791 50  0000 L CNN
 F 2 "agg:0402" H 7050 1750 50  0001 C CNN
@@
 $EndComp
 $Comp
-L agg-kicad:GND #PWR?
+L agg-kicad:GND #PWR0108
 U 1 1 5B45ABFF
 P 7050 1900
-F 0 "#PWR?" H 6920 1940 50  0001 L CNN
+F 0 "#PWR0108" H 6920 1940 50  0001 L CNN
 F 1 "GND" H 7050 1800 50  0000 C CNN
 F 2 "" H 7050 1900 50  0001 C CNN
@@
 	7050 1850 7050 1900
 $Comp
-L agg-kicad:3v3 #PWR?
+L agg-kicad:3v3 #PWR0109
 U 1 1 5B45B85D
 P 5350 1450
-F 0 "#PWR?" H 5350 1560 50  0001 L CNN
+F 0 "#PWR0109" H 5350 1560 50  0001 L CNN
 F 1 "3v3" H 5350 1574 50  0000 C CNN
 F 2 "" H 5350 1450 50  0001 C CNN
@@
 P 6250 800
 AR Path="/5A37ABC3/5B4621D7" Ref="C?"  Part="1"
-AR Path="/5A37ABBB/5B4621D7" Ref="C?"  Part="1"
-F 0 "C?" H 6300 995 50  0000 C CNN
+AR Path="/5A37ABBB/5B4621D7" Ref="C2"  Part="1"
+F 0 "C2" H 6300 995 50  0000 C CNN
 F 1 "470pF" H 6300 904 50  0000 C CNN
 F 2 "agg:0402" H 6250 800 50  0001 C CNN
@@
 Connection ~ 3500 1400
 $Comp
-L ncp4620:NCP4620 U?
+L ncp4620:NCP4620 U3
 U 1 1 5B47A899
 P 9700 1500
-F 0 "U?" H 9700 1847 60  0000 C CNN
+F 0 "U3" H 9700 1847 60  0000 C CNN
 F 1 "NCP4620" H 9700 1741 60  0000 C CNN
 F 2 "agg:SC-70-5" H 9700 1100 60  0001 C CNN
@@
 1V8 Regulator
 $Comp
-L 3v3_switched:3v3_switched #PWR?
+L 3v3_switched:3v3_switched #PWR0110
 U 1 1 5B47B468
 P 9150 1300
-F 0 "#PWR?" H 9150 1410 50  0001 L CNN
+F 0 "#PWR0110" H 9150 1410 50  0001 L CNN
 F 1 "3v3_switched" H 9150 1424 50  0000 C CNN
 F 2 "" H 9150 1300 50  0001 C CNN
@@
 P 9150 1600
 AR Path="/5B47B986" Ref="C?"  Part="1"
-AR Path="/5A37ABBB/5B47B986" Ref="C?"  Part="1"
-F 0 "C?" H 9200 1795 50  0000 C CNN
+AR Path="/5A37ABBB/5B47B986" Ref="C3"  Part="1"
+F 0 "C3" H 9200 1795 50  0000 C CNN
 F 1 "1uF" H 9200 1704 50  0000 C CNN
 F 2 "agg:0402" H 9150 1600 50  0001 C CNN
@@
 $EndComp
 $Comp
-L agg-kicad:GND #PWR?
+L agg-kicad:GND #PWR0111
 U 1 1 5B47C44A
 P 9150 1650
-F 0 "#PWR?" H 9020 1690 50  0001 L CNN
+F 0 "#PWR0111" H 9020 1690 50  0001 L CNN
 F 1 "GND" H 9150 1550 50  0000 C CNN
 F 2 "" H 9150 1650 50  0001 C CNN
@@
 P 10250 1450
 AR Path="/5B47F85A" Ref="C?"  Part="1"
-AR Path="/5A37ABBB/5B47F85A" Ref="C?"  Part="1"
-F 0 "C?" H 10300 1645 50  0000 C CNN
+AR Path="/5A37ABBB/5B47F85A" Ref="C4"  Part="1"
+F 0 "C4" H 10300 1645 50  0000 C CNN
 F 1 "1uF" H 10300 1554 50  0000 C CNN
 F 2 "agg:0402" H 10250 1450 50  0001 C CNN
@@
 $EndComp
 $Comp
-L agg-kicad:GND #PWR?
+L agg-kicad:GND #PWR0112
 U 1 1 5B47F8E6
 P 10250 1600
-F 0 "#PWR?" H 10120 1640 50  0001 L CNN
+F 0 "#PWR0112" H 10120 1640 50  0001 L CNN
 F 1 "GND" H 10250 1500 50  0000 C CNN
 F 2 "" H 10250 1600 50  0001 C CNN
@@
 $EndComp
 $Comp
-L agg-kicad:1v8 #PWR?
+L agg-kicad:1v8 #PWR0113
 U 1 1 5B47F93E
 P 10250 1350
-F 0 "#PWR?" H 10250 1460 50  0001 L CNN
+F 0 "#PWR0113" H 10250 1460 50  0001 L CNN
 F 1 "1v8" H 10250 1474 50  0000 C CNN
 F 2 "" H 10250 1350 50  0001 C CNN
@@
 Wire Wire Line
 	10250 1600 10250 1550
+$Comp
+L agg-kicad:PWR #FLG03
+U 1 1 5B50ADFF
+P 2050 1500
+F 0 "#FLG03" H 2050 1660 50  0001 C CNN
+F 1 "PWR" H 2100 1450 50  0000 C CNN
+F 2 "" H 2050 1500 50  0001 C CNN
+F 3 "" H 2050 1500 50  0001 C CNN
+	1    2050 1500
+	1    0    0    -1
+$EndComp
+$Comp
+L agg-kicad:PWR #FLG0101
+U 1 1 5B509E1B
+P 7350 1300
+F 0 "#FLG0101" H 7350 1460 50  0001 C CNN
+F 1 "PWR" H 7350 1434 50  0000 C CNN
+F 2 "" H 7350 1300 50  0001 C CNN
+F 3 "" H 7350 1300 50  0001 C CNN
+	1    7350 1300
+	1    0    0    -1
+$EndComp
+Wire Wire Line
+	7350 1300 7200 1300
+Connection ~ 7200 1300
+Wire Wire Line
+	2000 1400 2000 1500
+Wire Wire Line
+	2050 1500 2150 1500
+Wire Wire Line
+	2050 1500 2000 1500
+Connection ~ 2050 1500
+Connection ~ 2000 1500
+Wire Wire Line
+	2000 1500 2000 1550
 $EndSCHEMATC
