File: pcb/radio.sch (KiCad schematic (older format))
At the start: 47 parts, among them IC3 Si4460, P3 COAX, P4 COAX, U3 MCP4812, U4 TMP102, U5 MICRF112YMM, X1 Antenna (434MHz), X2 Antenna (434MHz), Y2 13.56MHz

Commit message: Fix footprint name error (agg:0805-L does not exist)
Parts:
- L2, L8: footprint agg:0805-L -> agg:0805
Changed lines of the file:
@@
 Title "Jerboa Radio Schematics"
 Date "2018-06-12"
-Rev "1.0"
+Rev "1.1"
 Comp "Cambridge University Spaceflight"
 Comment1 "Greg Brooks"
@@
 F 0 "L2" V 6404 2041 50  0000 L CNN
 F 1 "56nH" V 6495 2041 50  0000 L CNN
-F 2 "agg:0805-L" H 6400 2000 50  0001 C CNN
+F 2 "agg:0805" H 6400 2000 50  0001 C CNN
 F 3 "" H 6400 2000 50  0001 C CNN
 F 4 "1711831" H 0   0   50  0001 C CNN "Farnell"
@@
 F 0 "L8" V 8300 3950 50  0000 L CNN
 F 1 "680nH" V 8400 3800 50  0000 L CNN
-F 2 "agg:0805-L" H 8300 4100 50  0001 C CNN
+F 2 "agg:0805" H 8300 4100 50  0001 C CNN
 F 3 "" H 8300 4100 50  0001 C CNN
 F 4 "2286391" H 0   0   50  0001 C CNN "Farnell"

Commit message: Redo si4460 matching for 169MHz
Parts:
- removed C26: 3.9pF, agg:0402, symbol agg-kicad:C
- removed C28, C31: 15pF, agg:0402, symbol agg-kicad:C
- removed C29: 2.2pF, agg:0402, symbol agg-kicad:C
- removed C30: 8.2pF, agg:0402, symbol agg-kicad:C
- removed C33: 6.8pF, agg:0402, symbol agg-kicad:C
- removed L2: 56nH, agg:0805, symbol agg-kicad:L
- removed L3: 220nH, agg:0603-L, symbol agg-kicad:L
- removed L4: 51nH, agg:0402-L, symbol agg-kicad:L
- removed L5: 39nH, agg:0603-L, symbol agg-kicad:L
- removed L6, L7: 18nH, agg:0402-L, symbol agg-kicad:L
- added C0: 39pF, agg:0402, symbol agg-kicad:C
- added CC2: 470pF, agg:0402, symbol agg-kicad:C
- added CM1: 6.8pF, agg:0402, symbol agg-kicad:C
- added CM2, CM3: 18pF, agg:0402, symbol agg-kicad:C
- added CP1: 3pF, agg:0402, symbol agg-kicad:C
- added CP2: 2pF, agg:0402, symbol agg-kicad:C
- added CR1: 12pF, agg:0402, symbol agg-kicad:C
- added CR2: 6.2pF, agg:0402, symbol agg-kicad:C
- added L0: 22nH, agg:0402, symbol agg-kicad:L
- added LM1: 56nH, agg:0402-L, symbol agg-kicad:L
- added LM2, LM4: 47nH, agg:0402-L, symbol agg-kicad:L
- added LM3: 68nH, agg:0402-L, symbol agg-kicad:L
- added LR1: 220nH, agg:0402, symbol agg-kicad:L
- added LR2: 150nH, agg:0402-L, symbol agg-kicad:L
- added Lchoke1: 470nH, agg:0603-L, symbol agg-kicad:L
- renumbered C27 to C26, C32 to C27, C34 to C28, C35 to C29, C36 to C30, C37 to C31, C38 to C32, D3 to D2, D4 to D3, L8 to L2, L9 to L3, P3 to P2, P4 to P3, X1 to X2, X2 to X3
Connections:
- wire segments 171 -> 182
Other:
- note added: "https://www.silabs.com/documents/public/application-notes/AN627.pdf\n169MHz matching (Direct Tie CLE)"
- note removed: "https://www.silabs.com/documents/public/application-notes/AN627.pdf"

Commit message: WIP: work on pcb, use guitar wire ground plane antenna and remove rx matching on si4460 as there is nothing to receive
Parts:
- removed CR1: 12pF, agg:0402, symbol agg-kicad:C
- removed CR2: 6.2pF, agg:0402, symbol agg-kicad:C
- removed LR1: 220nH, agg:0402, symbol agg-kicad:L
- removed LR2: 150nH, agg:0402-L, symbol agg-kicad:L
- removed X2, X3: Antenna (434MHz), symbol agg-kicad:PART
- added TP1: TESTPAD, Jerboa:ANT_GND_PASSTHROUGH, symbol agg-kicad:TESTPAD
- L3, LM1, LM2, LM3, LM4: footprint agg:0402-L -> agg:0402
- P2: value COAX -> 144MHz; footprint agg:SMA-EDGE -> Jerboa:GND_PLANE_ANT; Farnell 1608592 -> (none)
- P3: value COAX -> 434MHz; footprint agg:SMA-EDGE -> Jerboa:GND_PLANE_ANT; Farnell 1608592 -> (none)
Connections:
- wire segments 182 -> 174
Other:
- note added: "Antenna GND plane pass through"
- note added: "Don't need rx"
Changed lines of the file:
@@
 EESchema Schematic File Version 4
+LIBS:jerboa-cache
 EELAYER 26 0
 EELAYER END
@@
 P 9000 1600
 F 0 "P2" H 9000 1700 50  0000 C CNN
-F 1 "COAX" H 9000 1450 50  0000 C CNN
-F 2 "agg:SMA-EDGE" H 9000 1390 50  0001 C CNN
+F 1 "144MHz" H 9000 1450 50  0000 C CNN
+F 2 "Jerboa:GND_PLANE_ANT" H 9000 1390 50  0001 C CNN
 F 3 "" H 9100 1500 50  0001 C CNN
-F 4 "1608592" H 9000 1320 50  0001 C CNN "Farnell"
 	1    9000 1600
 	1    0    0    -1
@@
 	1    0    0    -1
 $EndComp
-$Comp
-L agg-kicad:GND #PWR0134
-U 1 1 5B258845
-P 6400 2500
-F 0 "#PWR0134" H 6270 2540 50  0001 L CNN
-F 1 "GND" H 6400 2400 50  0000 C CNN
-F 2 "" H 6400 2500 60  0000 C CNN
-F 3 "" H 6400 2500 60  0000 C CNN
-	1    6400 2500
-	1    0    0    -1
-$EndComp
 Wire Wire Line
 	6200 1500 6500 1500
@@
 	6200 1850 6400 1850
 Wire Wire Line
-	7350 1850 7350 1500
-Wire Wire Line
-	6400 2000 6400 1850
-Wire Wire Line
-	6400 2100 6400 2250
-Wire Wire Line
 	6200 2250 6400 2250
-Connection ~ 6400 2250
-Wire Wire Line
-	6400 2250 6400 2350
-Wire Wire Line
-	6400 2450 6400 2500
-Wire Wire Line
-	7350 2250 7350 1850
-Connection ~ 7350 1850
 $Comp
 L agg-kicad:GND #PWR0135
@@
 F 0 "L3" H 8850 4350 50  0000 C CNN
 F 1 "43nH" H 8850 4450 50  0000 C CNN
-F 2 "agg:0402-L" H 8800 4300 50  0001 C CNN
+F 2 "agg:0402" H 8800 4300 50  0001 C CNN
 F 3 "" H 8800 4300 50  0001 C CNN
 F 4 "2470331" H 0   0   50  0001 C CNN "Farnell"
@@
 P 9400 4300
 F 0 "P3" H 9400 4400 50  0000 C CNN
-F 1 "COAX" H 9400 4150 50  0000 C CNN
-F 2 "agg:SMA-EDGE" H 9400 4090 50  0001 C CNN
+F 1 "434MHz" H 9400 4150 50  0000 C CNN
+F 2 "Jerboa:GND_PLANE_ANT" H 9400 4090 50  0001 C CNN
 F 3 "" H 9500 4200 50  0001 C CNN
-F 4 "1608592" H 9400 4020 50  0001 C CNN "Farnell"
 	1    9400 4300
 	1    0    0    -1
@@
 	8900 4300 9300 4300
 Connection ~ 8900 4300
-$Comp
-L agg-kicad:PART X2
-U 1 1 5B504041
-P 9300 1650
-F 0 "X2" H 9828 1746 50  0000 L CNN
-F 1 "Antenna (434MHz)" H 9828 1655 50  0000 L CNN
-F 2 "" H 9300 1650 50  0001 C CNN
-F 3 "https://www.mouser.co.uk/datasheet/2/743/ANT-SS433%20V1.1-768740.pdf" H 9300 1650 50  0001 C CNN
-F 4 "471-ANT-SS433" H 9300 1650 50  0001 C CNN "Mouser"
-	1    9300 1650
-	1    0    0    -1
-$EndComp
-$Comp
-L agg-kicad:PART X3
-U 1 1 5B5043B9
-P 9550 4400
-F 0 "X3" H 10078 4496 50  0000 L CNN
-F 1 "Antenna (434MHz)" H 10078 4405 50  0000 L CNN
-F 2 "" H 9550 4400 50  0001 C CNN
-F 3 "https://www.mouser.co.uk/datasheet/2/743/ANT-SS433%20V1.1-768740.pdf" H 9550 4400 50  0001 C CNN
-F 4 "471-ANT-SS433" H 9550 4400 50  0001 C CNN "Mouser"
-	1    9550 4400
-	1    0    0    -1
-$EndComp
 Text Notes 7300 2800 0    50   ~ 0
 https://www.silabs.com/documents/public/application-notes/AN627.pdf\n169MHz matching (Direct Tie CLE)
@@
 F 0 "LM1" H 7150 1700 50  0000 C CNN
 F 1 "56nH" H 7150 1600 50  0000 C CNN
-F 2 "agg:0402-L" H 7050 1500 50  0001 C CNN
+F 2 "agg:0402" H 7050 1500 50  0001 C CNN
 F 3 "" H 7050 1500 50  0001 C CNN
 F 4 "1669639" H 7050 1500 50  0001 C CNN "Farnell"
@@
 	7000 1500 7050 1500
 Wire Wire Line
-	7150 1500 7350 1500
-Wire Wire Line
 	7000 1700 7000 1650
-$Comp
-L agg-kicad:C CR2
-U 1 1 5B2576E8
-P 6750 1850
-F 0 "CR2" H 6800 2045 50  0000 C CNN
-F 1 "6.2pF" H 6800 1954 50  0000 C CNN
-F 2 "agg:0402" H 6750 1850 50  0001 C CNN
-F 3 "" H 6750 1850 50  0001 C CNN
-F 4 "1885324" H 6750 1850 50  0001 C CNN "Farnell"
-	1    6750 1850
-	1    0    0    -1
-$EndComp
-$Comp
-L agg-kicad:L LR1
-U 1 1 5B25788E
-P 6400 2000
-F 0 "LR1" V 6404 2041 50  0000 L CNN
-F 1 "220nH" V 6495 2041 50  0000 L CNN
-F 2 "agg:0402" H 6400 2000 50  0001 C CNN
-F 3 "" H 6400 2000 50  0001 C CNN
-F 4 "2424700" H 6400 2000 50  0001 C CNN "Farnell"
-	1    6400 2000
-	0    1    1    0
-$EndComp
-$Comp
-L agg-kicad:L LR2
-U 1 1 5B257969
-P 6750 2250
-F 0 "LR2" H 6800 2428 50  0000 C CNN
-F 1 "150nH" H 6800 2337 50  0000 C CNN
-F 2 "agg:0402-L" H 6750 2250 50  0001 C CNN
-F 3 "" H 6750 2250 50  0001 C CNN
-F 4 "2491614" H 6750 2250 50  0001 C CNN "Farnell"
-	1    6750 2250
-	1    0    0    -1
-$EndComp
-$Comp
-L agg-kicad:C CR1
-U 1 1 5B257ADB
-P 6400 2350
-F 0 "CR1" V 6404 2408 50  0000 L CNN
-F 1 "12pF" V 6495 2408 50  0000 L CNN
-F 2 "agg:0402" H 6400 2350 50  0001 C CNN
-F 3 "" H 6400 2350 50  0001 C CNN
-F 4 "1885336" H 6400 2350 50  0001 C CNN "Farnell"
-	1    6400 2350
-	0    1    1    0
-$EndComp
-Wire Wire Line
-	6850 1850 7350 1850
-Wire Wire Line
-	6850 2250 7350 2250
-Wire Wire Line
-	6750 2250 6400 2250
-Wire Wire Line
-	6750 1850 6400 1850
-Connection ~ 6400 1850
 $Comp
 L agg-kicad:L LM2
@@
 F 0 "LM2" H 7500 1678 50  0000 C CNN
 F 1 "47nH" H 7500 1587 50  0000 C CNN
-F 2 "agg:0402-L" H 7450 1500 50  0001 C CNN
+F 2 "agg:0402" H 7450 1500 50  0001 C CNN
 F 3 "" H 7450 1500 50  0001 C CNN
 F 4 "1343090" H 7450 1500 50  0001 C CNN "Farnell"
@@
 F 0 "LM3" H 7800 1678 50  0000 C CNN
 F 1 "68nH" H 7800 1587 50  0000 C CNN
-F 2 "agg:0402-L" H 7750 1500 50  0001 C CNN
+F 2 "agg:0402" H 7750 1500 50  0001 C CNN
 F 3 "" H 7750 1500 50  0001 C CNN
 F 4 "1669641" H 7750 1500 50  0001 C CNN "Farnell"
@@
 F 0 "LM4" H 8100 1678 50  0000 C CNN
 F 1 "47nH" H 8100 1587 50  0000 C CNN
-F 2 "agg:0402-L" H 8050 1500 50  0001 C CNN
+F 2 "agg:0402" H 8050 1500 50  0001 C CNN
 F 3 "" H 8050 1500 50  0001 C CNN
 F 4 "1343090" H 0   0   50  0001 C CNN "Farnell"
@@
 	7750 1500 7650 1500
 Wire Wire Line
-	7450 1500 7350 1500
-Connection ~ 7350 1500
-Wire Wire Line
 	7650 1650 7650 1500
 Connection ~ 7650 1500
@@
 Wire Wire Line
 	8150 1200 8250 1200
+Text Notes 8900 5700 0    50   ~ 0
+Antenna GND plane pass through
+$Comp
+L agg-kicad:TESTPAD TP1
+U 1 1 5B23257E
+P 9350 5750
+F 0 "TP1" H 9447 5750 50  0000 L CNN
+F 1 "TESTPAD" H 9350 5675 50  0001 L CNN
+F 2 "Jerboa:ANT_GND_PASSTHROUGH" H 9350 5600 50  0001 L CNN
+F 3 "" H 9350 5750 50  0001 C CNN
+F 4 "https://www.ebay.co.uk/itm/Ernie-Ball-Custom-Gauge-Guitar-Single-Strings-Electric-or-Acoustic-Pack-6-13-/360959212478" H 9350 5750 50  0001 C CNN "Ebay"
+	1    9350 5750
+	1    0    0    -1
+$EndComp
+$Comp
+L agg-kicad:GND #PWR0158
+U 1 1 5B232690
+P 9300 5800
+F 0 "#PWR0158" H 9170 5840 50  0001 L CNN
+F 1 "GND" H 9300 5700 50  0000 C CNN
+F 2 "" H 9300 5800 60  0000 C CNN
+F 3 "" H 9300 5800 60  0000 C CNN
+	1    9300 5800
+	1    0    0    -1
+$EndComp
+Wire Wire Line
+	9300 5800 9300 5750
+Wire Wire Line
+	9300 5750 9350 5750
+Wire Wire Line
+	7150 1500 7450 1500
+Wire Wire Line
+	6400 1850 6400 2250
+Text Notes 6450 2100 0    50   ~ 0
+Don't need rx
 $EndSCHEMATC

Commit message: WIP: more pcb layout, add rx stuff again
Parts:
- added CR1: 12pF, agg:0402, symbol agg-kicad:C
- added CR2: 6.2pF, agg:0402, symbol agg-kicad:C
- added LR1: 220nH, agg:0402, symbol agg-kicad:L
- added LR2: 150nH, agg:0402, symbol agg-kicad:L
Connections:
- wire segments 174 -> 184
Other:
- note removed: "Don't need rx"
Changed lines of the file:
@@
 	9300 5750 9350 5750
 Wire Wire Line
-	7150 1500 7450 1500
+	6400 2100 6400 2250
 Wire Wire Line
-	6400 1850 6400 2250
-Text Notes 6450 2100 0    50   ~ 0
-Don't need rx
+	6400 2000 6400 1850
+Wire Wire Line
+	6850 2250 7350 2250
+$Comp
+L agg-kicad:L LR2
+U 1 1 5B257969
+P 6750 2250
+F 0 "LR2" H 6800 2428 50  0000 C CNN
+F 1 "150nH" H 6800 2337 50  0000 C CNN
+F 2 "agg:0402" H 6750 2250 50  0001 C CNN
+F 3 "" H 6750 2250 50  0001 C CNN
+F 4 "2491614" H 6750 2250 50  0001 C CNN "Farnell"
+	1    6750 2250
+	1    0    0    -1
+$EndComp
+Wire Wire Line
+	6400 2450 6400 2500
+Connection ~ 6400 2250
+Wire Wire Line
+	6400 2250 6400 2350
+$Comp
+L agg-kicad:GND #PWR0134
+U 1 1 5B258845
+P 6400 2500
+F 0 "#PWR0134" H 6270 2540 50  0001 L CNN
+F 1 "GND" H 6400 2400 50  0000 C CNN
+F 2 "" H 6400 2500 60  0000 C CNN
+F 3 "" H 6400 2500 60  0000 C CNN
+	1    6400 2500
+	1    0    0    -1
+$EndComp
+$Comp
+L agg-kicad:C CR1
+U 1 1 5B257ADB
+P 6400 2350
+F 0 "CR1" V 6404 2408 50  0000 L CNN
+F 1 "12pF" V 6495 2408 50  0000 L CNN
+F 2 "agg:0402" H 6400 2350 50  0001 C CNN
+F 3 "" H 6400 2350 50  0001 C CNN
+F 4 "1885336" H 6400 2350 50  0001 C CNN "Farnell"
+	1    6400 2350
+	0    1    1    0
+$EndComp
+Wire Wire Line
+	6750 2250 6400 2250
+$Comp
+L agg-kicad:L LR1
+U 1 1 5B25788E
+P 6400 2000
+F 0 "LR1" V 6404 2041 50  0000 L CNN
+F 1 "220nH" V 6495 2041 50  0000 L CNN
+F 2 "agg:0402" H 6400 2000 50  0001 C CNN
+F 3 "" H 6400 2000 50  0001 C CNN
+F 4 "2424700" H 6400 2000 50  0001 C CNN "Farnell"
+	1    6400 2000
+	0    1    1    0
+$EndComp
+Connection ~ 6400 1850
+Wire Wire Line
+	6750 1850 6400 1850
+$Comp
+L agg-kicad:C CR2
+U 1 1 5B2576E8
+P 6750 1850
+F 0 "CR2" H 6800 2045 50  0000 C CNN
+F 1 "6.2pF" H 6800 1954 50  0000 C CNN
+F 2 "agg:0402" H 6750 1850 50  0001 C CNN
+F 3 "" H 6750 1850 50  0001 C CNN
+F 4 "1885324" H 6750 1850 50  0001 C CNN "Farnell"
+	1    6750 1850
+	1    0    0    -1
+$EndComp
+Wire Wire Line
+	6850 1850 7350 1850
+Wire Wire Line
+	7350 2250 7350 1850
+Wire Wire Line
+	7450 1500 7350 1500
+Wire Wire Line
+	7150 1500 7350 1500
+Connection ~ 7350 1500
+Connection ~ 7350 1850
+Wire Wire Line
+	7350 1850 7350 1500
 $EndSCHEMATC

Commit message: Schematic (and some pcb) using si4460 for both 144MHz and 434MHz
Parts:
- removed C22: 36pF, agg:0402, symbol agg-kicad:C
- removed C23: 12pF, agg:0402, symbol agg-kicad:C
- removed C24: 18pF, agg:0402, symbol agg-kicad:C
- removed C26, C29, C31, C32: 100nF, agg:0402, symbol agg-kicad:C
- removed C28: 2.2pF, agg:0402, symbol agg-kicad:C
- removed D2: D_Capacitance, agg:SOD-323, symbol Device:D_Capacitance
- removed D3: D_Capacitance, Jerboa:SC-79, symbol Device:D_Capacitance
- removed L2: 680nH, agg:0805, symbol agg-kicad:L
- removed L3: 43nH, agg:0402, symbol agg-kicad:L
- removed P3: 434MHz, Jerboa:GND_PLANE_ANT, symbol agg-kicad:COAX
- removed R13: 10k, agg:0402, symbol agg-kicad:R
- removed R14, R15: 1M, agg:0402, symbol agg-kicad:R
- removed R16: 4k7, agg:0402, symbol agg-kicad:R
- removed R17, R18: 100k, agg:0402, symbol agg-kicad:R
- removed U3: MCP4812, agg:SOIC-8, symbol mcp4812:MCP4812
- removed U4: TMP102, agg:SOT-666, symbol TMP102:TMP102
- removed U5: MICRF112YMM, agg:MSOP-10, symbol micrf112YMM:MICRF112YMM
- removed Y2: 13.56MHz, agg:XTAL-50x32, symbol agg-kicad:XTAL
- added D2, D3: ESD_DIODE, agg:0402, symbol agg-kicad:ESD_DIODE
- added L10, L7: 18nH, agg:0402, symbol agg-kicad:L
- added L4: 56nH, agg:0402, symbol agg-kicad:L
- added P2: 434MHz, Jerboa:GND_PLANE_ANT, symbol agg-kicad:COAX
- added U3: BGS12PL6E6327XTSA1, Jerboa:DFN-6-infineon, symbol BGS12PL6E6327XTSA1:BGS12PL6E6327XTSA1
- C20: value 100nF -> 10nF; Farnell 2533923 -> 2332514
- C21: value 10uF -> 18pF; footprint Jerboa:1411 -> agg:0402; Farnell 1754183 -> 2522556
- C25: value 10nF -> 8.2pF; Farnell 2627339 -> 1865418
- C27: value 1.2pF -> 15pF; Farnell 2310300 -> 2520723
- C30: value 6.8pF -> 8.2pF; Farnell 2310317 -> 1865418
- L2: renamed from Lchoke1; value 470nH -> 390nH; footprint agg:0603-L -> agg:0603; Farnell 2215632 -> 1711818
- renumbered CR1 to C22, C0 to C23, CR2 to C24, CM1 to C26, CM2 to C28, CP1 to C29, CM3 to C31, CP2 to C32, CC2 to C33, LM3 to L11, LM4 to L12, LR1 to L3, LR2 to L5, L0 to L6, LM1 to L8, LM2 to L9, P2 to P3
Connections:
- net labels added: FREQ_CTRL, RADIO_TX_144, RADIO_TX_434
- net labels removed: COARSE, DAC_NCS, DAC_SCK, DAC_SDI, FINE, MICRF_EN, RADIO_TX, TMP_ALERT, TMP_SCL, TMP_SDA
- wire segments 184 -> 114
- no-connect marks 7 -> 6
Other:
- note added: "Large"
- note added: "Si4460 Antenna Matching - 169MHz"
- note added: "Si4460 Antenna Matching - 434MHz"
- note added: "https://www.silabs.com/documents/public/application-notes/AN627.pdf\n434MHz matching (Split Tx CLE)"
- note removed: "Based on joey (https://github.com/cuspaceflight/joey-m)"
- note removed: "MICRF 434MHz FSK Circuit"
- note removed: "Si4460 Antenna Matching"
- note removed: "Use to monitor crystal temperature"
- note removed: "ceramic"
- note removed: "tantalum"
- moved on the sheet: C17, C18, C19, C22, C23, C24, C26, C28, C29, C31, C32, C33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

Commit message: Add footprints for 50ohm matching of antennas, work on schematic & pcb
Parts:
- added C34, C35: C, agg:0603, symbol agg-kicad:C
- added L13, L14: L, agg:0603, symbol agg-kicad:L
- L2: value 390nH -> 250nH; Farnell 1711818 -> (none); Mouser (none) -> 81-LQW18ANR22J8ZD
- L4: footprint agg:0402 -> agg:0603; Farnell 1669639 -> 1711807
Connections:
- wire segments 114 -> 122
Other:
- note added: "Impedance matching (match to 50ohms as filter matches to Zload)\nValues unknown"
- note added: "Inductor sets DC bias,\nswitch can only pass RF (not DC)"
- note added: "LC resonant tank"
- note added: "Low pass filter"
- note added: "See also http://tt7hab.blogspot.com/2017/05/the-tt7f-v15-revision.html"
- note added: "Vdd = sqrt(0.01/ (2*pi^2 * 144MHz * 1.25pF) ) = 1.68V\nIdd = 2 * pi^2 * 144MHz * 1.25pF * Vdd = 0.00596A\nRdc = (3.3V - Vdd) / Idd = 272.2ohm (set PA_PWR_LVL register appropriately)\n"
- note added: "Vdd = sqrt(0.02/ (2*pi^2 * 434MHz * 1.25pF) ) = 1.37V\nIdd = 2 * pi^2 * 434MHz * 1.25pF * Vdd = 0.0146A\nRdc = (3.3V - Vdd) / Idd = 132.1ohm (set PA_PWR_LVL register appropriately)\n"
- note added: "Zload = (0.2815)/(2 * pi * 144MHz * 1.25pF) * e^j * 49.0524degrees\nZload = 163.1 + 188.0j ohm at 144MHz"
- note added: "Zload = (0.2815)/(2 * pi * 434MHz * 1.25pF) * e^j * 49.0524degrees\nZload = 54.12 + 62.38j ohm at 434MHz"
- moved on the sheet: C22, C23, C24, C26, C28, C29, C31, C32, C33, D2, D3, L11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
