File: pcb/radio.sch (KiCad schematic (older format))
At the start: 34 parts, among them IC3 Si4460, IC4 BGS12AL7, P2 434MHz, P3 144MHz

Commit message: Finish redoing clock circuitry
Parts:
- added C?: 10nF, agg:0402, symbol agg-kicad:C
- added C?: 100pF, agg:0402, symbol agg-kicad:C
- added Y?: TCXO, agg:TG-5006CG, symbol agg-kicad:TCXO
Connections:
- net labels added: 1v8
- net labels removed: SI4460_XIN
- wire segments 113 -> 118
Other:
- note added: "Impedance matching\n(match to 50ohms as filter matches to Zload)\nValues unknown"
- note removed: "Impedance matching (match to 50ohms as filter matches to Zload)\nValues unknown"
- moved on the sheet: C17, C18, C19, C20, C21, C23, C25, C26, C27, C28, C29, C30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

Commit message: Begin routing pcb (again)
Parts:
- gave numbers to parts that had none: 3
Changed lines of the file:
@@
 	7650 1850 9050 1850
 $Comp
-L 3v3_switched:3v3_switched #PWR?
+L 3v3_switched:3v3_switched #PWR0114
 U 1 1 5B455DF5
 P 1400 1200
-F 0 "#PWR?" H 1400 1310 50  0001 L CNN
+F 0 "#PWR0114" H 1400 1310 50  0001 L CNN
 F 1 "3v3_switched" H 1400 1324 50  0000 C CNN
 F 2 "" H 1400 1200 50  0001 C CNN
@@
 $EndComp
 $Comp
-L 3v3_switched:3v3_switched #PWR?
+L 3v3_switched:3v3_switched #PWR0115
 U 1 1 5B456116
 P 3600 1500
-F 0 "#PWR?" H 3600 1610 50  0001 L CNN
+F 0 "#PWR0115" H 3600 1610 50  0001 L CNN
 F 1 "3v3_switched" H 3600 1624 50  0000 C CNN
 F 2 "" H 3600 1500 50  0001 C CNN
@@
 $EndComp
 $Comp
-L 3v3_switched:3v3_switched #PWR?
+L 3v3_switched:3v3_switched #PWR0116
 U 1 1 5B456364
 P 5100 1800
-F 0 "#PWR?" H 5100 1910 50  0001 L CNN
+F 0 "#PWR0116" H 5100 1910 50  0001 L CNN
 F 1 "3v3_switched" H 5100 1924 50  0000 C CNN
 F 2 "" H 5100 1800 50  0001 C CNN
@@
 	5700 500  5700 5400
 $Comp
-L agg-kicad:TCXO Y?
+L agg-kicad:TCXO Y1
 U 1 1 5B4A0C26
 P 1450 1900
-F 0 "Y?" H 1450 2125 50  0000 C CNN
+F 0 "Y1" H 1450 2125 50  0000 C CNN
 F 1 "TCXO" H 1450 2034 50  0000 C CNN
 F 2 "agg:TG-5006CG" H 1250 1900 50  0001 C CNN
@@
 $EndComp
 $Comp
-L agg-kicad:C C?
+L agg-kicad:C C13
 U 1 1 5B4A15A9
 P 1000 2000
-F 0 "C?" H 1050 2195 50  0000 C CNN
+F 0 "C13" H 1050 2195 50  0000 C CNN
 F 1 "10nF" H 1050 2104 50  0000 C CNN
 F 2 "agg:0402" H 1000 2000 50  0001 C CNN
@@
 $EndComp
 $Comp
-L agg-kicad:GND #PWR?
+L agg-kicad:GND #PWR0117
 U 1 1 5B4A1958
 P 1000 2050
-F 0 "#PWR?" H 870 2090 50  0001 L CNN
+F 0 "#PWR0117" H 870 2090 50  0001 L CNN
 F 1 "GND" H 1000 1950 50  0000 C CNN
 F 2 "" H 1000 2050 60  0000 C CNN
@@
 $EndComp
 $Comp
-L agg-kicad:1v8 #PWR?
+L agg-kicad:1v8 #PWR0118
 U 1 1 5B4A19DA
 P 1000 1850
-F 0 "#PWR?" H 1000 1960 50  0001 L CNN
+F 0 "#PWR0118" H 1000 1960 50  0001 L CNN
 F 1 "1v8" H 1000 1974 50  0000 C CNN
 F 2 "" H 1000 1850 50  0001 C CNN
@@
 Connection ~ 1000 2000
 $Comp
-L agg-kicad:C C?
+L agg-kicad:C C14
 U 1 1 5B4AF076
 P 1850 1900
-F 0 "C?" H 1900 1970 50  0000 C CNN
+F 0 "C14" H 1900 1970 50  0000 C CNN
 F 1 "100pF" H 1900 1830 50  0000 C CNN
 F 2 "agg:0402" H 1850 1900 50  0001 C CNN
