File: pcb/jerboa.kicad_pcb (KiCad board)
At the start: 2 copper layers, 72 parts, among them IC1 ADP1607, IC2 MAX-M8Q, IC3 Si4460, IC4 BGS12AL7, J1 CONN_01x02, J2 CONN_01x03, J3 CONN_01x02, J4 CONN_01x02, P1 SWD_TC, P2 434MHz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

Commit message: More PCB routing
Parts:
- moved D1 25.6 mm to (149.6, 107.5), turned to 180 degrees
- moved R6 25.1 mm to (147.4, 106.9), turned to 270 degrees
- moved J3 20.2 mm to (130.2, 116.9)
- moved R2 17.7 mm to (161.4, 130.3)
- moved C12 17.7 mm to (161.1, 127.2)
- moved IC1 17.7 mm to (161.8, 125.3)
- moved L1 17.7 mm to (163.9, 126.2)
- moved C1 16.2 mm to (158.6, 124.5)
- moved R1 16.2 mm to (159.2, 129.1)
- moved J1 6.15 mm to (150.3, 119.3)
- moved D2 5.10 mm to (145.4, 90.1), turned to 180 degrees
- moved C16 4.98 mm to (135.8, 111.1)
- moved C35 4.53 mm to (150.3, 90.8), turned to 90 degrees
- moved AE1 3.56 mm to (137.3, 129.0)
- moved IC2 3.56 mm to (140.6, 118.3)
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Connections:
- U1 pad 25: Net-(U1-Pad25) -> Net-(R6-Pad1)
- U1 pad 32: Net-(R6-Pad1) -> Net-(U1-Pad32)
Routing:
- net 3v3: track 21.3 -> 65.1 mm, vias 0 -> 2
- net /NRST: track 2.09 -> 21.7 mm
- net 3v3_switched: track 24.7 -> 41.4 mm
- net GND: track 36.1 -> 51.6 mm, vias 16 -> 19
- net /RADIO_PWR_EN: track 0.00 -> 14.7 mm
- net /BATT_V: track 0.00 -> 7.73 mm
- net /RX_GPS_from_MCU: track 0.00 -> 7.44 mm
- net /TX_GPS_from_MCU: track 0.00 -> 7.40 mm
- net /SOLAR_CELL_VOLTAGE: track 0.00 -> 5.59 mm
- net Net-(D2-Pad1): track 0.00 -> 4.73 mm
- net Net-(C30-Pad1): track 0.00 -> 4.72 mm
- net /SWCLK: track 0.00 -> 4.19 mm
- net /SWDIO: track 0.00 -> 3.87 mm
- net Net-(C25-Pad1): track 0.00 -> 3.28 mm
- net Net-(C27-Pad1): track 0.00 -> 2.67 mm
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
Commit message: Even more PCB routing
Parts:
- moved J3 27.0 mm to (131.1, 143.9)
- moved J1 19.4 mm to (153.6, 138.4)
- moved IC1 10.1 mm to (164.1, 115.5)
- moved R2 10.1 mm to (163.7, 120.5)
- moved C1 10.1 mm to (160.9, 114.7)
- moved C12 10.1 mm to (163.4, 117.4)
- moved R1 10.1 mm to (161.6, 119.3)
- moved L1 10.1 mm to (166.2, 116.4)
- moved R4 7.05 mm to (140.1, 108.7), turned to 0 degrees
- moved C2 6.64 mm to (135.8, 108.1)
- moved R3 6.64 mm to (135.8, 110.2)
- moved U2 6.64 mm to (137.7, 109.2)
- moved C16 4.90 mm to (140.7, 111.2), turned to 90 degrees
- moved C9 3.30 mm to (143.7, 99.9), turned to 270 degrees
- moved J4 2.75 mm to (136.8, 104.1), turned to 90 degrees
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Routing:
- net 3v3_switched: track 41.4 -> 50.7 mm
- net /NRST: track 21.7 -> 26.6 mm
- net GND: track 51.6 -> 55.6 mm, vias 19 -> 21
- net /SWCLK: track 4.19 -> 1.56 mm
- net /BATT_V: track 7.73 -> 5.44 mm
- net /RADIO_PWR_EN: track 14.7 -> 17.0 mm, vias 0 -> 3
- net /SWDIO: track 3.87 -> 1.78 mm
- net /GPS_~RESET: track 0.00 -> 1.48 mm, vias 0 -> 1
- net Net-(R4-Pad1): track 0.99 -> 1.63 mm
- net /RX_GPS_from_MCU: track 7.44 -> 8.03 mm
- net 3v3: track 65.1 -> 64.6 mm
- net /SOLAR_CELL_VOLTAGE: track 5.59 -> 5.04 mm

Commit message: Finish first iteration of Jerboa PCB
Parts:
- added X2: CUSF_LOGO, Jerboa:cusf_logo, B.Cu at (149.2, 114.2)
- moved P3 50.9 mm to (155.4, 134.7), turned to 270 degrees
- moved TP1 48.5 mm to (149.9, 135.0), turned to 180 degrees
- moved L13 48.0 mm to (157.1, 132.3), turned to 180 degrees
- moved P2 47.3 mm to (144.4, 134.7), turned to 90 degrees
- moved D3 46.2 mm to (154.5, 132.5), turned to 180 degrees
- moved J3 45.4 mm to (143.6, 100.2), turned to 90 degrees
- moved C28 45.2 mm to (150.6, 133.2), turned to 180 degrees
- moved C34 44.4 mm to (157.8, 129.8), turned to 90 degrees
- moved C26 44.4 mm to (148.7, 133.1), turned to 270 degrees
- moved C33 44.2 mm to (156.4, 130.5), turned to 270 degrees
- moved C29 43.1 mm to (152.8, 131.5), turned to 90 degrees
- moved L12 42.7 mm to (154.6, 130.6), turned to 0 degrees
- moved L11 42.4 mm to (151.6, 131.5), turned to 90 degrees
- moved D2 42.0 mm to (146.3, 132.1), turned to 0 degrees
- moved L3 41.8 mm to (150.4, 131.5), turned to 270 degrees
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Connections:
- IC2 pad 5: Net-(IC2-Pad5) -> /GPS_EXTINT
- U1 pad 18: Net-(U1-Pad18) -> /GPS_EXTINT
Routing:
- net GND: track 55.6 -> 147.2 mm, vias 21 -> 49
- net 3v3: track 64.6 -> 107.0 mm, vias 2 -> 4
- net /GPS_~RESET: track 1.48 -> 14.6 mm, vias 1 -> 2
- net /RADIO_PWR_EN: track 17.0 -> 4.72 mm, vias 3 -> 0
- net 3v3_switched: track 50.7 -> 62.2 mm, vias 0 -> 2
- net Net-(C12-Pad1): track 0.00 -> 9.37 mm
- net /GPS_EXTINT: track 0.00 -> 8.61 mm
- net Net-(IC1-Pad3): track 0.00 -> 6.76 mm
- net 1v8: track 1.10 -> 5.65 mm
- net Net-(IC1-Pad5): track 0.00 -> 3.66 mm
- net /SWCLK: track 1.56 -> 4.19 mm
- net /SWDIO: track 1.78 -> 3.87 mm
- net /BATT_V: track 5.44 -> 6.40 mm
- added copper zone on B.Cu, net GND
- added copper zone on F.Cu, net GND
Other:
- board outline added: 20.8 x 47.7 mm
- board text added: "+"
- board text added: "-"
- board text added: "144MHz"
- board text added: "3V3 out"
- board text added: "434MHz"
- board text added: "En"
- board text added: "Jerboa"
- board text added: "SCL"
- board text added: "SDA"
- board text added: "Solar_V"
- board text added: "V_batt"
- board text added: "Vin"
- board text added: "http://www.cusf.co.uk/"
