File: pcb/wspr_breakout/wspr_breakout.sch (KiCad schematic (older format))
At the start: 10 parts

Commit message: Update wspr breakout footprints
Parts:
- U?: footprint (none) -> agg:MSOP-10; Farnell (none) -> Value
- U?: footprint Jerboa:SuperSOT-6 -> jerboa:SuperSOT-6
- Y?: footprint Jerboa:ASTX_H11 -> jerboa:ASTX_H11
Changed lines of the file:
@@
 F 0 "U?" H 7850 3197 60  0000 C CNN
 F 1 "SI5351A_10_pin" H 7850 3091 60  0000 C CNN
-F 2 "" H 7350 2950 60  0001 C CNN
+F 2 "agg:MSOP-10" H 7350 2950 60  0001 C CNN
 F 3 "" H 7350 2950 60  0001 C CNN
+F 4 "Value" H 7350 2950 60  0001 C CNN "Farnell"
 	1    7350 2950
 	1    0    0    -1
@@
 F 0 "U?" H 2650 3097 60  0000 C CNN
 F 1 "FDC6329L" H 2650 2991 60  0000 C CNN
-F 2 "Jerboa:SuperSOT-6" H 2650 2100 60  0001 C CNN
+F 2 "jerboa:SuperSOT-6" H 2650 2100 60  0001 C CNN
 F 3 "http://www.farnell.com/datasheets/2285836.pdf" H 2650 2200 60  0001 C CNN
 F 4 "1652469" H 2650 2000 60  0001 C CNN "Farnell"
@@
 F 0 "Y?" H 6000 3575 50  0000 C CNN
 F 1 "TCXO" H 6000 3484 50  0000 C CNN
-F 2 "Jerboa:ASTX_H11" H 6000 2950 50  0001 C CNN
+F 2 "jerboa:ASTX_H11" H 6000 2950 50  0001 C CNN
 F 3 "http://www.abracon.com/Oscillators/ASTX-H11.pdf" H 6000 3000 50  0001 C CNN
 F 4 "Value" H 6000 3350 60  0001 C CNN "Farnell"
