File: pcb/solar_breakout/solar_breakout.sch (KiCad schematic (older format))
At the start: 29 parts

Commit message: Make super capacitor footprint
Parts:
- C?: footprint (none) -> jerboa:super_capacitor
Changed lines of the file:
@@
 F 0 "C?" V 7246 3492 50  0000 R CNN
 F 1 "50" V 7155 3492 50  0000 R CNN
-F 2 "" H 7150 3550 50  0001 C CNN
+F 2 "jerboa:super_capacitor" H 7150 3550 50  0001 C CNN
 F 3 "http://www.farnell.com/datasheets/2675068.pdf" H 7150 3550 50  0001 C CNN
 F 4 "2696619" H 0   0   50  0001 C CNN "Farnell"

Commit message: Check component footprints, Farnell numbers etc. Make some changes
Parts:
- C?: footprint agg:0402 -> agg:0603; Farnell 1327624 -> 2760492
- C?: footprint agg:1206 -> agg:0402; Farnell 1135175 -> 2611904
- C? (x2): footprint agg:0603 -> agg:0805; Farnell 2470448 -> 1463389
- D?: footprint agg:DO-214AC-SMA -> (none)
- IC?: Farnell 1898600 -> (none); Mouser (none) -> 584-LTC3105EDD#PBF
- J?: Farnell Value -> (none)
- L?: footprint agg:0805 -> agg:1812; Farnell 2286356 -> 1515459
Other:
- note added: ">=3W"
- note added: "Or use the 40F one as \nit has a significantly \ngreater energy density \n(so similar energy storage \nwith significant mass saving)"
- note added: "agg:DO-214AC-SMA\nbut don't need footprint\nas this will not be mounted\nto board"
- note removed: "Flying wires, \nthermally coupled\nto solar cells\n(no smd footprint)"
Changed lines of the file:
@@
 EESchema Schematic File Version 4
-LIBS:solar_breakout-cache
-EELAYER 29 0
+EELAYER 26 0
 EELAYER END
 $Descr A4 11693 8268
@@
 F 3 "" H 6000 1900 50  0001 C CNN
 F 4 "1593411" H 6000 1900 60  0001 C CNN "Farnell"
+F 5 "" H 0   0   50  0001 C CNN "Mouser"
 	1    6000 1900
 	1    0    0    -1
@@
 F 3 "" H 7250 1900 50  0001 C CNN
 F 4 "1593411" H 7250 1900 60  0001 C CNN "Farnell"
+F 5 "" H 0   0   50  0001 C CNN "Mouser"
 	1    7250 1900
 	1    0    0    -1
@@
 F 3 "https://uk.farnell.com/yageo/rc0402fr-07510kl/res-510k-1-0-063w-0402-thick-film/dp/1458807" H 6700 3550 50  0001 C CNN
 F 4 "1458807" H 0   0   50  0001 C CNN "Farnell"
+F 5 "" H 0   0   50  0001 C CNN "Mouser"
 	1    6700 3550
 	0    1    1    0
@@
 F 3 "http://www.farnell.com/datasheets/2563624.pdf" H 6700 3350 50  0001 C CNN
 F 4 "2447431" H 0   0   50  0001 C CNN "Farnell"
+F 5 "" H 0   0   50  0001 C CNN "Mouser"
 	1    6700 3350
 	0    1    1    0
@@
 F 3 "http://www.farnell.com/datasheets/2675068.pdf" H 7150 3550 50  0001 C CNN
 F 4 "2696619" H 0   0   50  0001 C CNN "Farnell"
+F 5 "" H 0   0   50  0001 C CNN "Mouser"
 	1    7150 3550
 	0    -1   -1   0
@@
 F 0 "L?" H 5800 3078 50  0000 C CNN
 F 1 "10u" H 5800 2987 50  0000 C CNN
-F 2 "agg:0805" H 5750 2900 50  0001 C CNN
-F 3 "http://www.farnell.com/datasheets/1681885.pdf" H 5750 2900 50  0001 C CNN
-F 4 "2286356" H 0   0   50  0001 C CNN "Farnell"
+F 2 "agg:1812" H 5750 2900 50  0001 C CNN
+F 3 "http://www.farnell.com/datasheets/5132.pdf" H 5750 2900 50  0001 C CNN
+F 4 "1515459" H 0   0   50  0001 C CNN "Farnell"
+F 5 "" H 0   0   50  0001 C CNN "Mouser"
 	1    5750 2900
 	1    0    0    -1
@@
 F 3 "http://www.farnell.com/datasheets/2189109.pdf" H 6350 3850 50  0001 C CNN
 F 4 "2688503" H 0   0   50  0001 C CNN "Farnell"
+F 5 "" H 0   0   50  0001 C CNN "Mouser"
 	1    6350 3850
 	0    1    1    0
@@
 F 0 "C?" V 5054 3658 50  0000 L CNN
 F 1 "10n" V 5145 3658 50  0000 L CNN
-F 2 "agg:0402" H 5050 3600 50  0001 C CNN
-F 3 "http://www.farnell.com/datasheets/2237835.pdf" H 5050 3600 50  0001 C CNN
-F 4 "1327624" H 0   0   50  0001 C CNN "Farnell"
+F 2 "agg:0603" H 5050 3600 50  0001 C CNN
+F 3 "http://www.farnell.com/datasheets/2290180.pdf" H 5050 3600 50  0001 C CNN
+F 4 "2760492" H 0   0   50  0001 C CNN "Farnell"
+F 5 "" H 0   0   50  0001 C CNN "Mouser"
 	1    5050 3600
 	0    1    1    0
@@
 F 0 "C?" H 5300 3005 50  0000 C CNN
 F 1 "10u" H 5300 3096 50  0000 C CNN
-F 2 "agg:1206" H 5250 3200 50  0001 C CNN
-F 3 "http://www.farnell.com/datasheets/2096548.pdf" H 5250 3200 50  0001 C CNN
-F 4 "1135175" H 0   0   50  0001 C CNN "Farnell"
+F 2 "agg:0402" H 5250 3200 50  0001 C CNN
+F 3 "http://www.farnell.com/datasheets/2079148.pdf" H 5250 3200 50  0001 C CNN
+F 4 "2611904" H 0   0   50  0001 C CNN "Farnell"
+F 5 "" H 0   0   50  0001 C CNN "Mouser"
 	1    5250 3200
 	-1   0    0    1
@@
 F 0 "C?" V 5304 3758 50  0000 L CNN
 F 1 "1u" V 5395 3758 50  0000 L CNN
-F 2 "agg:0603" H 5300 3700 50  0001 C CNN
-F 3 "http://www.farnell.com/datasheets/2048284.pdf" H 5300 3700 50  0001 C CNN
-F 4 "2470448" H 0   0   50  0001 C CNN "Farnell"
+F 2 "agg:0805" H 5300 3700 50  0001 C CNN
+F 3 "http://www.farnell.com/datasheets/2315442.pdf" H 5300 3700 50  0001 C CNN
+F 4 "1463389" H 0   0   50  0001 C CNN "Farnell"
+F 5 "" H 0   0   50  0001 C CNN "Mouser"
 	1    5300 3700
 	0    1    1    0
@@
 F 3 "http://www.farnell.com/datasheets/2031615.pdf" H 6250 3450 50  0001 C CNN
 F 4 "2533782" H 6250 3450 60  0001 C CNN "Farnell"
+F 5 "" H 0   0   50  0001 C CNN "Mouser"
 	1    6250 3450
 	0    -1   -1   0
@@
 F 0 "C?" V 6904 3508 50  0000 L CNN
 F 1 "1u" V 6995 3508 50  0000 L CNN
-F 2 "agg:0603" H 6900 3450 50  0001 C CNN
-F 3 "http://www.farnell.com/datasheets/2048284.pdf" H 6900 3450 50  0001 C CNN
-F 4 "2470448" H 0   0   50  0001 C CNN "Farnell"
+F 2 "agg:0805" H 6900 3450 50  0001 C CNN
+F 3 "http://www.farnell.com/datasheets/2315442.pdf" H 6900 3450 50  0001 C CNN
+F 4 "1463389" H 0   0   50  0001 C CNN "Farnell"
+F 5 "" H 0   0   50  0001 C CNN "Mouser"
 	1    6900 3450
 	0    1    1    0
@@
 	7150 3550 7150 4050
 Connection ~ 6900 4050
-Text Notes 3550 3750 0    60   ~ 0
-Flying wires, \nthermally coupled\nto solar cells\n(no smd footprint)
 $Comp
 L agg-kicad:LTC3105 IC?
@@
 F 1 "LTC3105" H 5800 3934 50  0000 C CNN
 F 2 "agg:DFN-10-EP-LT" H 5500 2900 50  0001 L CNN
-F 3 "http://www.farnell.com/datasheets/1999327.pdf" H 5400 3800 50  0001 C CNN
-F 4 "1898600" H 5500 2800 50  0001 L CNN "Farnell"
+F 3 "https://www.mouser.co.uk/datasheet/2/609/3105fb-1270124.pdf" H 5400 3800 50  0001 C CNN
+F 4 "584-LTC3105EDD#PBF" H 0   0   50  0001 C CNN "Mouser"
 	1    5800 3500
 	1    0    0    -1
@@
 F 0 "D?" V 2796 7192 50  0000 R CNN
 F 1 "MRA4003T3" V 2705 7192 50  0000 R CNN
-F 2 "agg:DO-214AC-SMA" H 2700 7250 50  0001 C CNN
+F 2 "" H 2700 7250 50  0001 C CNN
 F 3 "http://www.farnell.com/datasheets/2028669.pdf" H 2700 7250 50  0001 C CNN
-F 4 "1459134" H 2700 7250 60  0001 C CNN "Farnell"
+F 4 "" H 0   0   50  0001 C CNN "Mouser"
+F 5 "1459134" H 2700 7250 60  0001 C CNN "Farnell"
 	1    2700 7250
 	0    -1   -1   0
@@
 F 2 "agg:SIL-254P-02" H 2850 1700 50  0001 C CNN
 F 3 "" H 2850 1700 50  0001 C CNN
+F 4 "" H 0   0   50  0001 C CNN "Mouser"
 	1    2850 1700
 	1    0    0    -1
@@
 F 2 "agg:SIL-254P-02" H 2850 3200 50  0001 C CNN
 F 3 "" H 2850 3200 50  0001 C CNN
+F 4 "" H 0   0   50  0001 C CNN "Mouser"
 	1    2850 3200
 	1    0    0    -1
@@
 F 3 "" H 7550 3500 50  0001 C CNN
 F 4 "1593411" H 7550 3500 60  0001 C CNN "Farnell"
+F 5 "" H 0   0   50  0001 C CNN "Mouser"
 	1    7550 3500
 	-1   0    0    1
@@
 F 3 "http://www.farnell.com/datasheets/2007092.pdf" H 7400 3700 50  0001 C CNN
 F 4 "2476361" H 7400 3700 60  0001 C CNN "Farnell"
+F 5 "" H 0   0   50  0001 C CNN "Mouser"
 	1    7400 3700
 	0    1    1    0
@@
 Wire Wire Line
 	1650 6400 1650 6250
-$Comp
-L agg-kicad:CONN_01x02 J?
-U 1 1 5A81FA4C
-P 4550 3650
-F 0 "J?" H 4581 3865 50  0000 C CNN
-F 1 "CONN_01x02" H 4581 3774 50  0000 C CNN
-F 2 "agg:SIL-254P-02" H 4550 3650 50  0001 C CNN
-F 3 "" H 4550 3650 50  0001 C CNN
-F 4 "Value" H 4550 3650 60  0001 C CNN "Farnell"
-	1    4550 3650
-	1    0    0    -1
-$EndComp
-Wire Wire Line
-	4650 3650 4700 3650
-Wire Wire Line
-	4650 3750 4700 3750
 Text Label 750  7500 0    60   ~ 0
 Array_1_-
@@
 Wire Wire Line
 	4700 3300 4700 3650
-Connection ~ 4700 3650
 Text Label 4700 4000 2    60   ~ 0
 D_cathode
 Wire Wire Line
 	4700 4000 4700 3750
-Connection ~ 4700 3750
 Wire Notes Line
 	500  5900 3300 5900
@@
 F 3 "http://www.farnell.com/datasheets/2238474.pdf" H 3450 1770 50  0001 C CNN
 F 4 "1843668" H 3400 1700 60  0001 C CNN "Farnell"
+F 5 "" H 0   0   50  0001 C CNN "Mouser"
 	1    3400 1700
 	-1   0    0    1
@@
 F 3 "http://www.farnell.com/datasheets/2238474.pdf" H 3450 3270 50  0001 C CNN
 F 4 "1843668" H 3400 3200 60  0001 C CNN "Farnell"
+F 5 "" H 0   0   50  0001 C CNN "Mouser"
 	1    3400 3200
 	-1   0    0    1
@@
 	3600 2900 3600 3200
 Connection ~ 3600 2900
+Text Notes 6950 3200 0    50   ~ 0
+Or use the 40F one as \nit has a significantly \ngreater energy density \n(so similar energy storage \nwith significant mass saving)
+Wire Notes Line
+	7100 3600 7100 3250
+Wire Notes Line
+	7100 3250 6900 3250
+Wire Notes Line
+	6900 3250 6900 2750
+Wire Notes Line
+	6900 2750 8100 2750
+Wire Notes Line
+	8100 2750 8100 3250
+Wire Notes Line
+	8100 3250 7200 3250
+Wire Notes Line
+	7200 3250 7200 3600
+Wire Notes Line
+	7100 3600 7200 3600
+Connection ~ 4700 3750
+Wire Wire Line
+	4650 3750 4700 3750
+Connection ~ 4700 3650
+Wire Wire Line
+	4650 3650 4700 3650
+$Comp
+L agg-kicad:CONN_01x02 J?
+U 1 1 5A81FA4C
+P 4550 3650
+F 0 "J?" H 4581 3865 50  0000 C CNN
+F 1 "CONN_01x02" H 4581 3774 50  0000 C CNN
+F 2 "agg:SIL-254P-02" H 4550 3650 50  0001 C CNN
+F 3 "" H 4550 3650 50  0001 C CNN
+F 4 "" H 0   0   50  0001 C CNN "Mouser"
+	1    4550 3650
+	1    0    0    -1
+$EndComp
+Text Notes 2800 7100 0    50   ~ 0
+agg:DO-214AC-SMA\nbut don't need footprint\nas this will not be mounted\nto board
+Text Notes 7450 3800 0    50   ~ 0
+>=3W
 $EndSCHEMATC

Commit message: Begin solar pcb
Parts:
- gave numbers to parts that had none: 29
Connections:
- wire segments 99 -> 104

Commit message: Work on pcb
Connections:
- wire segments 104 -> 103
Changed lines of the file:
@@
-$EndComp
-$Comp
-L agg-kicad:CONN_01x02 J5
-U 1 1 5A7C8C5D
-P 7250 1900
-F 0 "J5" H 7281 2115 50  0000 C CNN
-F 1 "CONN_01x02" H 7281 2024 50  0000 C CNN
-F 2 "agg:SIL-254P-02" H 7250 1900 50  0001 C CNN
-F 3 "" H 7250 1900 50  0001 C CNN
-F 4 "1593411" H 7250 1900 60  0001 C CNN "Farnell"
-F 5 "" H 0   0   50  0001 C CNN "Mouser"
-	1    7250 1900
-	1    0    0    -1
 $EndComp
 $Comp
@@
 	1    0    0    -1
 $EndComp
-$Comp
-L agg-kicad:GND #PWR06
-U 1 1 5A7C8EBA
-P 7550 2050
-F 0 "#PWR06" H 7420 2090 50  0001 L CNN
-F 1 "GND" H 7550 2137 50  0000 C CNN
-F 2 "" H 7550 2050 50  0001 C CNN
-F 3 "" H 7550 2050 50  0001 C CNN
-	1    7550 2050
-	1    0    0    -1
-$EndComp
-Text Label 7500 1900 0    50   ~ 0
-Panel_V
-Wire Wire Line
-	7350 1900 7500 1900
-Wire Wire Line
-	7350 2000 7550 2000
-Wire Wire Line
-	7550 2000 7550 2050
 Text Label 6250 1900 0    50   ~ 0
 Cap_V
@@
 	3200 3300 3100 3300
 Connection ~ 3100 3300
+$Comp
+L agg-kicad:CONN_01x02 J5
+U 1 1 5A7C8C5D
+P 7250 1900
+F 0 "J5" H 7281 2115 50  0000 C CNN
+F 1 "CONN_01x02" H 7281 2024 50  0000 C CNN
+F 2 "agg:SIL-254P-02" H 7250 1900 50  0001 C CNN
+F 3 "" H 7250 1900 50  0001 C CNN
+F 4 "1593411" H 7250 1900 60  0001 C CNN "Farnell"
+F 5 "" H 0   0   50  0001 C CNN "Mouser"
+	1    7250 1900
+	1    0    0    -1
+$EndComp
+Text Label 7500 1900 0    50   ~ 0
+Panel_V
+Wire Wire Line
+	7350 1900 7500 1900
+Text Label 7500 2000 0    50   ~ 0
+Cap_V
+Wire Wire Line
+	7500 2000 7350 2000
 $EndSCHEMATC

Commit message: Add more stuff to pcb
Parts:
- R1: value R -> 30k; Farnell Value -> 2447333
Changed lines of the file:
@@
 F 3 "" H 6000 1900 50  0001 C CNN
 F 4 "1593411" H 6000 1900 60  0001 C CNN "Farnell"
-F 5 "" H 0   0   50  0001 C CNN "Mouser"
 	1    6000 1900
 	1    0    0    -1
@@
 F 3 "https://uk.farnell.com/yageo/rc0402fr-07510kl/res-510k-1-0-063w-0402-thick-film/dp/1458807" H 6700 3550 50  0001 C CNN
 F 4 "1458807" H 0   0   50  0001 C CNN "Farnell"
-F 5 "" H 0   0   50  0001 C CNN "Mouser"
 	1    6700 3550
 	0    1    1    0
@@
 F 3 "http://www.farnell.com/datasheets/2563624.pdf" H 6700 3350 50  0001 C CNN
 F 4 "2447431" H 0   0   50  0001 C CNN "Farnell"
-F 5 "" H 0   0   50  0001 C CNN "Mouser"
 	1    6700 3350
 	0    1    1    0
@@
 F 3 "http://www.farnell.com/datasheets/2675068.pdf" H 7150 3550 50  0001 C CNN
 F 4 "2696619" H 0   0   50  0001 C CNN "Farnell"
-F 5 "" H 0   0   50  0001 C CNN "Mouser"
 	1    7150 3550
 	0    -1   -1   0
@@
 F 3 "http://www.farnell.com/datasheets/5132.pdf" H 5750 2900 50  0001 C CNN
 F 4 "1515459" H 0   0   50  0001 C CNN "Farnell"
-F 5 "" H 0   0   50  0001 C CNN "Mouser"
 	1    5750 2900
 	1    0    0    -1
@@
 F 3 "http://www.farnell.com/datasheets/2189109.pdf" H 6350 3850 50  0001 C CNN
 F 4 "2688503" H 0   0   50  0001 C CNN "Farnell"
-F 5 "" H 0   0   50  0001 C CNN "Mouser"
 	1    6350 3850
 	0    1    1    0
@@
 F 3 "http://www.farnell.com/datasheets/2290180.pdf" H 5050 3600 50  0001 C CNN
 F 4 "2760492" H 0   0   50  0001 C CNN "Farnell"
-F 5 "" H 0   0   50  0001 C CNN "Mouser"
 	1    5050 3600
 	0    1    1    0
@@
 F 3 "http://www.farnell.com/datasheets/2079148.pdf" H 5250 3200 50  0001 C CNN
 F 4 "2611904" H 0   0   50  0001 C CNN "Farnell"
-F 5 "" H 0   0   50  0001 C CNN "Mouser"
 	1    5250 3200
 	-1   0    0    1
@@
 F 3 "http://www.farnell.com/datasheets/2315442.pdf" H 5300 3700 50  0001 C CNN
 F 4 "1463389" H 0   0   50  0001 C CNN "Farnell"
-F 5 "" H 0   0   50  0001 C CNN "Mouser"
 	1    5300 3700
 	0    1    1    0
@@
 F 3 "http://www.farnell.com/datasheets/2031615.pdf" H 6250 3450 50  0001 C CNN
 F 4 "2533782" H 6250 3450 60  0001 C CNN "Farnell"
-F 5 "" H 0   0   50  0001 C CNN "Mouser"
 	1    6250 3450
 	0    -1   -1   0
@@
 F 3 "http://www.farnell.com/datasheets/2315442.pdf" H 6900 3450 50  0001 C CNN
 F 4 "1463389" H 0   0   50  0001 C CNN "Farnell"
-F 5 "" H 0   0   50  0001 C CNN "Mouser"
 	1    6900 3450
 	0    1    1    0
@@
 F 2 "" H 2700 7250 50  0001 C CNN
 F 3 "http://www.farnell.com/datasheets/2028669.pdf" H 2700 7250 50  0001 C CNN
-F 4 "" H 0   0   50  0001 C CNN "Mouser"
-F 5 "1459134" H 2700 7250 60  0001 C CNN "Farnell"
+F 4 "1459134" H 2700 7250 60  0001 C CNN "Farnell"
 	1    2700 7250
 	0    -1   -1   0
@@
 F 2 "agg:SIL-254P-02" H 2850 1700 50  0001 C CNN
 F 3 "" H 2850 1700 50  0001 C CNN
-F 4 "" H 0   0   50  0001 C CNN "Mouser"
 	1    2850 1700
 	1    0    0    -1
@@
 F 2 "agg:SIL-254P-02" H 2850 3200 50  0001 C CNN
 F 3 "" H 2850 3200 50  0001 C CNN
-F 4 "" H 0   0   50  0001 C CNN "Mouser"
 	1    2850 3200
 	1    0    0    -1
@@
 F 3 "" H 7550 3500 50  0001 C CNN
 F 4 "1593411" H 7550 3500 60  0001 C CNN "Farnell"
-F 5 "" H 0   0   50  0001 C CNN "Mouser"
 	1    7550 3500
 	-1   0    0    1
@@
 F 3 "http://www.farnell.com/datasheets/2007092.pdf" H 7400 3700 50  0001 C CNN
 F 4 "2476361" H 7400 3700 60  0001 C CNN "Farnell"
-F 5 "" H 0   0   50  0001 C CNN "Mouser"
 	1    7400 3700
 	0    1    1    0
@@
 P 5300 3400
 F 0 "R1" H 5350 3222 50  0000 C CNN
-F 1 "R" H 5350 3313 50  0000 C CNN
+F 1 "30k" H 5350 3313 50  0000 C CNN
 F 2 "agg:0603" H 5300 3400 50  0001 C CNN
-F 3 "" H 5300 3400 50  0001 C CNN
-F 4 "Value" H 5300 3400 60  0001 C CNN "Farnell"
+F 3 "http://www.farnell.com/datasheets/2563624.pdf" H 5300 3400 50  0001 C CNN
+F 4 "2447333" H 5300 3400 60  0001 C CNN "Farnell"
 	1    5300 3400
 	-1   0    0    1
@@
 F 3 "http://www.farnell.com/datasheets/2238474.pdf" H 3450 1770 50  0001 C CNN
 F 4 "1843668" H 3400 1700 60  0001 C CNN "Farnell"
-F 5 "" H 0   0   50  0001 C CNN "Mouser"
 	1    3400 1700
 	-1   0    0    1
@@
 F 3 "http://www.farnell.com/datasheets/2238474.pdf" H 3450 3270 50  0001 C CNN
 F 4 "1843668" H 3400 3200 60  0001 C CNN "Farnell"
-F 5 "" H 0   0   50  0001 C CNN "Mouser"
 	1    3400 3200
 	-1   0    0    1
@@
 F 2 "agg:SIL-254P-02" H 4550 3650 50  0001 C CNN
 F 3 "" H 4550 3650 50  0001 C CNN
-F 4 "" H 0   0   50  0001 C CNN "Mouser"
 	1    4550 3650
 	1    0    0    -1
@@
 F 3 "" H 7250 1900 50  0001 C CNN
 F 4 "1593411" H 7250 1900 60  0001 C CNN "Farnell"
-F 5 "" H 0   0   50  0001 C CNN "Mouser"
 	1    7250 1900
 	1    0    0    -1

Commit message: Make the baord smaller and fix power lines
Parts:
- R1: value 30k -> 76.8k; Farnell 2447333 -> 2670896
Changed lines of the file:
@@
 P 5300 3400
 F 0 "R1" H 5350 3222 50  0000 C CNN
-F 1 "30k" H 5350 3313 50  0000 C CNN
+F 1 "76.8k" H 5350 3313 50  0000 C CNN
 F 2 "agg:0603" H 5300 3400 50  0001 C CNN
-F 3 "http://www.farnell.com/datasheets/2563624.pdf" H 5300 3400 50  0001 C CNN
-F 4 "2447333" H 5300 3400 60  0001 C CNN "Farnell"
+F 3 "http://www.farnell.com/datasheets/1960319.pdf" H 5300 3400 50  0001 C CNN
+F 4 "2670896" H 5300 3400 60  0001 C CNN "Farnell"
 	1    5300 3400
 	-1   0    0    1

Commit message: Forgot to save file
Parts:
- R1: Farnell 2670896 -> 2694941
Changed lines of the file:
@@
 F 1 "76.8k" H 5350 3313 50  0000 C CNN
 F 2 "agg:0603" H 5300 3400 50  0001 C CNN
-F 3 "http://www.farnell.com/datasheets/1960319.pdf" H 5300 3400 50  0001 C CNN
-F 4 "2670896" H 5300 3400 60  0001 C CNN "Farnell"
+F 3 "http://www.farnell.com/datasheets/2189593.pdf" H 5300 3400 50  0001 C CNN
+F 4 "2694941" H 5300 3400 60  0001 C CNN "Farnell"
 	1    5300 3400
 	-1   0    0    1
